File: hardware/project/ETH1CPMU1/AC_Source.sch (KiCad schematic (older format))
At the start: 0 parts

Commit message: Schematic design
Parts:
- added C801, C802: 10u, symbol Device:C
- added C803, C806, C807, C923: 10n, symbol Device:C
- added C804, C805, C931: 100n, symbol Device:C
- added C924: 4p7, symbol Device:C
- added C925: 18p, symbol Device:C
- added C926: 12p, symbol Device:C
- added C927, C930: 22p, symbol Device:C
- added C928, C929: 56p, symbol Device:C
- added L901, L902, L903: 4u7, symbol Device:L
- added R801: 2k7, symbol Device:R
- added R802, R911: 3k9, symbol Device:R
- added R803, R824, R831, R835, R838: 3k, symbol Device:R
- added R804, R805, R807, R809, R819: 1k5, symbol Device:R
- added R806: 1k8, symbol Device:R
- added R808, R820, R830: 1k2, symbol Device:R
- added R810, R817: 7k5, symbol Device:R
- added R811, R818: 15k, symbol Device:R
- added R812: 56, symbol Device:R
- added R813, R814, R815, R816, R822, R908: 10k, symbol Device:R
- added R821: 8k2, symbol Device:R
- added R823: 5k1, symbol Device:R
- added R825: 47k, symbol Device:R
- added R826, R828, R829, R832, R833: 150, symbol Device:R
- added R827, R909, R910: 300, symbol Device:R
- added R834: 5k6, symbol Device:R
- added R836: 2k4, symbol Device:R
- added R837: 12k, symbol Device:R
- added U801: AD8039, symbol ETH1CPMU1:AD8039
- added U802: REF191, symbol Reference_Voltage:REF191
- added U803, U806: OPA2277, symbol Amplifier_Operational:OPA2277
- added U804: LM6172, symbol Amplifier_Operational:LM6172
- added U805: AD603, symbol ETH1CPMU1:AD603
- added U807: LMH6321, symbol ETH1CPMU1:LMH6321
- added U906: AD9835, symbol ETH1CPMU1:AD9835
- added U907: ECS-3225SMV-500-GP-TR, symbol ETH1CPMU1:ECS-3225SMV
- added U908: 74AHCT1G08, symbol 74xGxx:74AHCT1G08
Connections:
- net labels added: +15VF, +3.3VP, +5VF, -15V, -15VF, AC_FOURCE, AGNDF, CL, DDS_OUT, DGNDF, GAIN, NULL, NULL_FB, OFFSET, OFFSET_FB, REF, REF_DDS
- wire segments 0 -> 222
- no-connect marks 0 -> 2

Commit message: Schematic design
Parts:
- added R?: 10k, symbol Device:R
- added U?: AD5324, symbol ETH1CPMU1:AD5324
Connections:
- net labels added: DAC_DIN, DAC_SCLK, DAC_~SYNC
- wire segments 222 -> 231
- no-connect marks 2 -> 3
Changed lines of the file:
@@
 Wire Wire Line
 	9350 2850 9350 3750
+$Comp
+L ETH1CPMU1:AD5324 U?
+U 1 1 5DD338C9
+P 5500 7800
+F 0 "U?" H 5150 8200 50  0000 C CNN
+F 1 "AD5324" H 5750 8200 50  0000 C CNN
+F 2 "" H 5100 8100 50  0001 C CNN
+F 3 "" H 5100 8100 50  0001 C CNN
+	1    5500 7800
+	1    0    0    -1
+$EndComp
+$Comp
+L power:+3.3VP #PWR?
+U 1 1 5DD36258
+P 5500 7350
+F 0 "#PWR?" H 5650 7300 50  0001 C CNN
+F 1 "+3.3VP" H 5520 7493 50  0000 C CNN
+F 2 "" H 5500 7350 50  0001 C CNN
+F 3 "" H 5500 7350 50  0001 C CNN
+	1    5500 7350
+	1    0    0    -1
+$EndComp
+$Comp
+L ETH1CPMU1:DGNDF #PWR?
+U 1 1 5DD3887D
+P 5500 8350
+F 0 "#PWR?" H 5500 8100 50  0001 C CNN
+F 1 "DGNDF" H 5505 8177 50  0000 C CNN
+F 2 "" H 5500 8350 50  0001 C CNN
+F 3 "" H 5500 8350 50  0001 C CNN
+	1    5500 8350
+	1    0    0    -1
+$EndComp
+Text Label 4850 7950 0    50   ~ 0
+REF
+Wire Wire Line
+	5000 7950 4850 7950
+Wire Wire Line
+	6000 7550 6300 7550
+Text Label 6300 7550 2    50   ~ 0
+NULL
+Wire Wire Line
+	6000 7750 6300 7750
+Text Label 6300 7750 2    50   ~ 0
+GAIN
+Wire Wire Line
+	6000 7950 6300 7950
+Text Label 6300 7950 2    50   ~ 0
+OFFSET
+NoConn ~ 6000 8150
+$Comp
+L Device:R R?
+U 1 1 5DD94F93
+P 4750 7250
+F 0 "R?" H 4820 7296 50  0000 L CNN
+F 1 "10k" H 4820 7205 50  0000 L CNN
+F 2 "" V 4680 7250 50  0001 C CNN
+F 3 "~" H 4750 7250 50  0001 C CNN
+	1    4750 7250
+	1    0    0    -1
+$EndComp
+Wire Wire Line
+	5000 7550 4750 7550
+Wire Wire Line
+	4750 7550 4750 7400
+$Comp
+L power:+3.3VP #PWR?
+U 1 1 5DDA3823
+P 4750 7100
+F 0 "#PWR?" H 4900 7050 50  0001 C CNN
+F 1 "+3.3VP" H 4770 7243 50  0000 C CNN
+F 2 "" H 4750 7100 50  0001 C CNN
+F 3 "" H 4750 7100 50  0001 C CNN
+	1    4750 7100
+	1    0    0    -1
+$EndComp
+Wire Wire Line
+	4750 7550 4300 7550
+Connection ~ 4750 7550
+Text Label 4300 7550 0    50   ~ 0
+DAC_~SYNC
+Wire Wire Line
+	5000 7650 4300 7650
+Text Label 4300 7650 0    50   ~ 0
+DAC_SCLK
+Wire Wire Line
+	5000 7750 4300 7750
+Text Label 4300 7750 0    50   ~ 0
+DAC_DIN
 $EndSCHEMATC

Commit message: Function generator schematic design.
Parts:
- removed C931: 100n, symbol Device:C
- removed R821: 8k2, symbol Device:R
- removed R822: 10k, symbol Device:R
- removed R823: 5k1, symbol Device:R
- removed R824, R831, R835, R838: 3k, symbol Device:R
- removed R825: 47k, symbol Device:R
- removed R826, R828, R829, R832, R833: 150, symbol Device:R
- removed R827: 300, symbol Device:R
- removed R830: 1k2, symbol Device:R
- removed R834: 5k6, symbol Device:R
- removed R836: 2k4, symbol Device:R
- removed R837: 12k, symbol Device:R
- removed U801: AD8039, symbol ETH1CPMU1:AD8039
- removed U802: REF191, symbol Reference_Voltage:REF191
- removed U803, U806: OPA2277, symbol Amplifier_Operational:OPA2277
- removed U804: LM6172, symbol Amplifier_Operational:LM6172
- removed U805: AD603, symbol ETH1CPMU1:AD603
- removed U807: LMH6321, symbol ETH1CPMU1:LMH6321
- removed U?: AD5324, symbol ETH1CPMU1:AD5324
- added C808, C811, C812, C813, C814, C815, C816, C817, C818, C819, C820: 100n, symbol Device:C
- added C809: 220n, symbol Device:C
- added C810: 1n, symbol Device:C
- added U802: AD5453, symbol ETH1CPMU1:AD545x
- added U805, U807: LT1468, symbol ETH1CPMU1:LT1468
- added U808: REF192, symbol Reference_Voltage:REF192
- added U809, U811: TL071, symbol Amplifier_Operational:TL071
- added U810: AD5689BRUZ, Package_SO:TSSOP-16_4.4x5mm_P0.65mm, symbol Analog_DAC:AD5689BRUZ
- C801, C802: value 10u -> C
- C803: value 10n -> 10u
- C805: value 100n -> 10u
- C806: value 10n -> 1u
- C807: value 10n -> 100n
- C923, C924, C925, C926, C927, C928, C929, C930: footprint (none) -> Capacitor_SMD:C_0603_1608Metric_Pad1.05x0.95mm_HandSolder
- R801: value 2k7 -> R
- R802: value 3k9 -> R
- R803: value 3k -> R
- R804, R805: value 1k5 -> R
- R806: value 1k8 -> 0
- R807: value 1k5 -> 4k22
- R808: value 1k2 -> 3k9
- R809: value 1k5 -> 1k96
- R810: value 7k5 -> 1k96
- R811: value 15k -> 0
- R812: value 56 -> 10k
- R814: value 10k -> 1k
- R815, R816: value 10k -> R
- R817: value 7k5 -> R
- R818: value 15k -> 24k9
- R819: value 1k5 -> 100k
- R820: value 1k2 -> 33k2
- gave numbers to parts that had none: 1
Connections:
- net labels added: +3.3VF, DDS_DAC_RSTSEL, DDS_DAC_SCLK, DDS_DAC_SDIN, DDS_DAC_SDO, DDS_DAC_~LDAC, DDS_DAC_~RESET, DDS_DAC_~SYNC, DDS_FGEN_PSEL0, DDS_FGEN_PSEL1, DDS_FGEN_SCLK, DDS_FGEN_SDATA, DDS_FGEN_~FSYNC, DDS_MDAC_DIN, DDS_MDAC_SCLK, DDS_MDAC_~SYNC, MEAS_AMPL, REF_2V5, V_AMPL, V_OFFSET
- net labels removed: -15V, CL, DAC_DIN, DAC_SCLK, DAC_~SYNC, DDS_OUT, GAIN, NULL, NULL_FB, OFFSET, OFFSET_FB, REF, REF_DDS
- wire segments 231 -> 212
- no-connect marks 3 -> 9
Other:
- moved on the sheet: C923, C924, C925, C926, C927, C928, C929, C930, L901, L902, L903, R821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

Commit message: Function generator schematic development.
Parts:
- added C821, C826: 1n, symbol Device:C
- added C822, C831: 100n, symbol Device:C
- added C823, C824: 100n, Capacitor_SMD:C_0603_1608Metric_Pad1.05x0.95mm_HandSolder, symbol Device:C
- added C825: 220p, symbol Device:C
- added C827: 470p, symbol Device:C
- added C828: 330p, symbol Device:C
- added C829: 150p, symbol Device:C
- added C830: 4n7, symbol Device:C
- added C832: 2u2, symbol Device:C
- added D801: SD103ATW, Package_TO_SOT_SMD:SOT-363_SC-70-6, symbol Diode:SD103ATW
- added D802: 1N4148W, symbol Device:D
- added K801: TQ2SA-5V, symbol ETH1CPMU1:TQ2SA-5V
- added R822, R823, R824, R825, R826, R832, R833: 10k, symbol Device:R
- added R827: 619, symbol Device:R
- added R828, R829, R830: 6k81, symbol Device:R
- added R831: 237k, symbol Device:R
- added U801, U803: TL072, symbol Amplifier_Operational:TL072
- added U804: DG419LEUA, Package_SO:MSOP-8_3x3mm_P0.65mm, symbol Analog_Switch:DG419LEUA
- added U806: ADS7818, symbol ETH1CPMU1:ADS7818
- C801, C802, C804, C807, C808, C809, C810, C811, C812, C813, C814, C815, C816, C817, C818, C819, C820: footprint (none) -> Capacitor_SMD:C_0603_1608Metric_Pad1.05x0.95mm_HandSolder
- R801, R802, R803, R804, R805, R806, R807, R808, R809, R810, R811, R812, R813, R814, R815, R816, R817, R818, R819, R820, R821, R908, R909, R910, R911: footprint (none) -> Resistor_SMD:R_0603_1608Metric_Pad1.05x0.95mm_HandSolder
Connections:
- net +15VF: now also C823.1, U801.8 (V+), U803.8 (V+), U804.4 (V+)
- net +3.3VP: now also U804.5 (VL)
- net +5VF: now also C831.1, D802.1 (K), K801.1, R832.1, U806.8 (VDD)
- net -15VF: now also C824.1, U801.4 (V-), U803.4 (V-), U804.7 (V-)
- net AC_FOURCE: now also K801.4; no longer C801.1, R803.1, U807.6
- net AGNDF: now also C821.2, C823.2, C824.2, C827.2, C828.2, C829.2, C830.2, C831.2, C832.2, K801.7, K801.8, K801.9, U803.5 (+), U804.3 (GND), U806.3 (IN-), U806.4 (GND)
- net MEAS_AMPL: now also U804.2
- net REF_2V5: no longer C806.1, R807.2, U808.6 (Vout), U810.1 (VREF)
- net at C808.2, R810.1, U809.3 (+): now also D801.1 (K), D801.4 (A)
- net at R809.2, U810.3 (VOUTA): now also D801.3 (K), D801.6 (A)
- new net: K801.2, R822.2
- new net: C801.1, K801.3, R803.1, U807.6
- new net: R823.1, R828.2, U801.1
- new net: R823.2, R824.2, U801.2 (-)
- new net: U801.3 (+), U804.1
- new net: C829.1, R830.1, U801.5 (+)
- new net: C825.1, C826.1, R827.2, U801.6 (-), U801.7
- new net: C822.1, R824.1, R825.1, U803.7
- new net: C822.2, R825.2, R826.1, U803.6 (-)
- new net: R826.2, R831.2, U803.1, U803.2 (-)
- new net: C832.1, U803.3 (+), U806.1 (VREF)
- new net: C827.1, C828.1, R828.1, R829.2, R831.1
- new net: C825.2, C826.2, R829.1, R830.2
- new net: C830.1, R827.1, U806.2 (IN+)
- new net: R832.2, R833.2, U806.6 (DATA)
- new net +2V5REF: C806.1, R807.2, U808.6 (Vout), U810.1 (VREF)
- new net AC_RELAY: D802.2 (A), K801.10
- new net DDS_MEAS_CLK: U806.7 (CLK)
- new net DDS_MEAS_CONV: U806.5 (CONV)
- new net DDS_MEAS_DATA: R833.1
- new net DDS_MEAS_SELECT: U804.6
- new net MEAS_OUT: C821.1, R822.1, U804.8
- no-connect marks 9 -> 11
Other:
- moved on the sheet: C801, C802, C803, C804, C805, C806, C807, C808, C809, C810, C811, C812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

Commit message: New footprint development, changes in schematics.
Parts:
- C802: renamed from C821; footprint (none) -> Capacitor_SMD:C_0603_1608Metric_Pad1.05x0.95mm_HandSolder
- C808: renamed from C803; footprint (none) -> Capacitor_SMD:C_1206_3216Metric_Pad1.42x1.75mm_HandSolder
- C814: renamed from C831; footprint (none) -> Capacitor_SMD:C_0603_1608Metric_Pad1.05x0.95mm_HandSolder
- C815: renamed from C805; footprint (none) -> Capacitor_SMD:C_0805_2012Metric_Pad1.15x1.40mm_HandSolder
- C816: renamed from C806; footprint (none) -> Capacitor_SMD:C_0603_1608Metric_Pad1.05x0.95mm_HandSolder
- C817: renamed from C825; footprint (none) -> Capacitor_SMD:C_0603_1608Metric_Pad1.05x0.95mm_HandSolder
- C818: renamed from C826; footprint (none) -> Capacitor_SMD:C_0603_1608Metric_Pad1.05x0.95mm_HandSolder
- C821: renamed from C827; footprint (none) -> Capacitor_SMD:C_0603_1608Metric_Pad1.05x0.95mm_HandSolder
- C822: renamed from C828; footprint (none) -> Capacitor_SMD:C_0603_1608Metric_Pad1.05x0.95mm_HandSolder
- C823: renamed from C829; footprint (none) -> Capacitor_SMD:C_0603_1608Metric_Pad1.05x0.95mm_HandSolder
- C824: renamed from C830; footprint (none) -> Capacitor_SMD:C_0603_1608Metric_Pad1.05x0.95mm_HandSolder
- C825: renamed from C822; footprint (none) -> Capacitor_SMD:C_0603_1608Metric_Pad1.05x0.95mm_HandSolder
- C827: renamed from C832; footprint (none) -> Capacitor_SMD:C_0805_2012Metric_Pad1.15x1.40mm_HandSolder
- D801: renamed from D802; footprint (none) -> Diode_SMD:D_SOD-123
- K801: footprint (none) -> ETH1CPMU1:SA
- L801: renamed from L901; footprint (none) -> Inductor_SMD:L_0603_1608Metric_Pad1.05x0.95mm_HandSolder
- L802: renamed from L902; footprint (none) -> Inductor_SMD:L_0603_1608Metric_Pad1.05x0.95mm_HandSolder
- L803: renamed from L903; footprint (none) -> Inductor_SMD:L_0603_1608Metric_Pad1.05x0.95mm_HandSolder
- R802: renamed from R822; footprint (none) -> Resistor_SMD:R_0603_1608Metric_Pad1.05x0.95mm_HandSolder
- R813: renamed from R832; footprint (none) -> Resistor_SMD:R_0603_1608Metric_Pad1.05x0.95mm_HandSolder
- R818: renamed from R827; footprint (none) -> Resistor_SMD:R_0603_1608Metric_Pad1.05x0.95mm_HandSolder
- R819: renamed from R833; footprint (none) -> Resistor_SMD:R_0603_1608Metric_Pad1.05x0.95mm_HandSolder
- R820: renamed from R828; footprint (none) -> Resistor_SMD:R_0603_1608Metric_Pad1.05x0.95mm_HandSolder
- R821: renamed from R829; footprint (none) -> Resistor_SMD:R_0603_1608Metric_Pad1.05x0.95mm_HandSolder
- R822: renamed from R830; footprint (none) -> Resistor_SMD:R_0603_1608Metric_Pad1.05x0.95mm_HandSolder
- R823: renamed from R831; footprint (none) -> Resistor_SMD:R_0603_1608Metric_Pad1.05x0.95mm_HandSolder
- R827: renamed from R823; footprint (none) -> Resistor_SMD:R_0603_1608Metric_Pad1.05x0.95mm_HandSolder
- R828: renamed from R824; footprint (none) -> Resistor_SMD:R_0603_1608Metric_Pad1.05x0.95mm_HandSolder
- R830: renamed from R825; footprint (none) -> Resistor_SMD:R_0603_1608Metric_Pad1.05x0.95mm_HandSolder
- R832: renamed from R826; footprint (none) -> Resistor_SMD:R_0603_1608Metric_Pad1.05x0.95mm_HandSolder
- U801: renamed from U802; value AD5453 -> AD5453YRMZ; footprint (none) -> Package_SO:MSOP-8_3x3mm_P0.65mm
- U802: renamed from U805; footprint (none) -> Package_SO:SSOP-8_3.9x5.05mm_P1.27mm
- U803: renamed from U807; footprint (none) -> Package_SO:SSOP-8_3.9x5.05mm_P1.27mm
- U804: renamed from U906; footprint (none) -> Package_SO:TSSOP-16_4.4x5mm_P0.65mm
- U806: renamed from U908; footprint (none) -> Package_TO_SOT_SMD:SOT-23-5_HandSoldering
- U807: renamed from U808; footprint (none) -> Package_SO:SSOP-8_3.9x5.05mm_P1.27mm
- U808: renamed from U809; footprint (none) -> Package_SO:SOIC-8_3.9x4.9mm_P1.27mm
- U810: renamed from U801; footprint (none) -> Package_SO:SOIC-8_3.9x4.9mm_P1.27mm
- U811: renamed from U806; footprint (none) -> Package_SO:MSOP-8_3x3mm_P0.65mm
- U813: renamed from U811; footprint (none) -> Package_SO:SOIC-8_3.9x4.9mm_P1.27mm
- U814: renamed from U803; footprint (none) -> Package_SO:SOIC-8_3.9x4.9mm_P1.27mm
- renumbered C802 to C803, C923 to C804, C924 to C805, C925 to C806, C926 to C807, C927 to C809, C928 to C810, C929 to C811, C930 to C812, C804 to C813, C807 to C819, C808 to C820, C809 to C826, C810 to C828, C811 to C829, C812 to C830, C813 to C831, C814 to C832, C815 to C833, C816 to C834, C817 to C835, C818 to C836, C819 to C837, C820 to C838, C823 to C839, C824 to C840, D801 to D802, R802 to R803, R803 to R804, R908 to R805, R804 to R806, R805 to R807, R909 to R808, R910 to R809, R911 to R810, R806 to R811, R807 to R812, R808 to R814, R809 to R815, R810 to R816, R811 to R817, R821 to R824, R812 to R825, R813 to R826, R814 to R829, R815 to R831, R818 to R833, R819 to R834, R816 to R835, R817 to R836, R820 to R837, U907 to U805, U804 to U809, U810 to U812
Connections:
- net REF_2V5 is gone; now on net +2V5REF: R833.2
Other:
- moved on the sheet: C808, C814, C815, C816, C817, C818, C819, C820, C821, C822, C823, C824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

Commit message: Schematic and PCB design.
Parts:
- removed U806: 74AHCT1G08, Package_TO_SOT_SMD:SOT-23-5_HandSoldering, symbol 74xGxx:74AHCT1G08
- added U806: 74AHCT1G08, Package_TO_SOT_SMD:SOT-353_SC-70-5_Handsoldering, symbol ETH1CPMU1:74AHCT1G08
- U805: footprint (none) -> ETH1CPMU1:ECS
Connections:
- net +3.3VP: now also U806.5
- net DGNDF: now also U806.3
- net at R811.1, U804.6 (MCLK): now also U806.4
- net at R811.2, U805.3 (OUT): now also U806.1, U806.2
Other:
- moved on the sheet: R811
Changed lines of the file:
@@
 	5350 2200 4550 2200
 Connection ~ 5350 2200
-$Comp
-L 74xGxx:74AHCT1G08 U806
-U 1 1 5DD68372
-P 2400 2900
-F 0 "U806" H 2750 3100 50  0000 C CNN
-F 1 "74AHCT1G08" H 2750 3000 50  0000 C CNN
-F 2 "Package_TO_SOT_SMD:SOT-23-5_HandSoldering" H 2400 2900 50  0001 C CNN
-F 3 "http://www.ti.com/lit/sg/scyt129e/scyt129e.pdf" H 2400 2900 50  0001 C CNN
-	1    2400 2900
-	1    0    0    -1
-$EndComp
-Wire Wire Line
-	2650 2900 3050 2900
-$Comp
-L ETH1CPMU1:DGNDF #PWR0824
-U 1 1 5DD7B574
-P 2400 3000
-F 0 "#PWR0824" H 2400 2750 50  0001 C CNN
-F 1 "DGNDF" H 2405 2827 50  0000 C CNN
-F 2 "" H 2400 3000 50  0001 C CNN
-F 3 "" H 2400 3000 50  0001 C CNN
-	1    2400 3000
-	1    0    0    -1
-$EndComp
-Wire Wire Line
-	2100 2950 2050 2950
-Wire Wire Line
-	2050 2850 2100 2850
-Wire Wire Line
-	2050 2850 2050 2900
-Wire Wire Line
-	3050 2900 3050 2700
+Wire Wire Line
+	2650 2950 3050 2950
+Wire Wire Line
+	2100 3000 2050 3000
+Wire Wire Line
+	2050 2900 2100 2900
+Wire Wire Line
+	3050 2950 3050 2700
 Wire Wire Line
 	3050 2700 3250 2700
@@
 F 0 "U805" H 1400 3165 50  0000 C CNN
 F 1 "ECS-3225SMV-500-GP-TR" H 1400 3074 50  0000 C CNN
-F 2 "" H 1800 3350 50  0001 C CNN
+F 2 "ETH1CPMU1:ECS" H 1800 3350 50  0001 C CNN
 F 3 "" H 1800 3350 50  0001 C CNN
 	1    1400 2800
@@
 Connection ~ 2050 2900
 Wire Wire Line
-	2050 2900 2050 2950
+	2050 2900 2050 3000
 $Comp
 L ETH1CPMU1:DGNDF #PWR0823
@@
 	1    0    0    -1
 $EndComp
-$Comp
-L power:+3.3VP #PWR0822
-U 1 1 5F50A5E2
-P 2400 2800
-F 0 "#PWR0822" H 2550 2750 50  0001 C CNN
-F 1 "+3.3VP" H 2420 2943 50  0000 C CNN
-F 2 "" H 2400 2800 50  0001 C CNN
-F 3 "" H 2400 2800 50  0001 C CNN
-	1    2400 2800
-	1    0    0    -1
-$EndComp
 Text HLabel 15050 2400 2    50   Output ~ 0
 AC_FOURCE
@@
 L Device:R R811
 U 1 1 5DD89B99
-P 2550 3500
-F 0 "R811" V 2343 3500 50  0000 C CNN
-F 1 "0" V 2434 3500 50  0000 C CNN
-F 2 "Resistor_SMD:R_0603_1608Metric_Pad1.05x0.95mm_HandSolder" V 2480 3500 50  0001 C CNN
-F 3 "~" H 2550 3500 50  0001 C CNN
-	1    2550 3500
-	0    1    1    0
-$EndComp
-Wire Wire Line
-	2400 3500 2050 3500
-Wire Wire Line
-	2050 3500 2050 2950
-Connection ~ 2050 2950
-Wire Wire Line
-	2700 3500 3050 3500
-Wire Wire Line
-	3050 3500 3050 2900
-Connection ~ 3050 2900
+P 2750 3500
+F 0 "R811" V 2543 3500 50  0000 C CNN
+F 1 "0" V 2634 3500 50  0000 C CNN
+F 2 "Resistor_SMD:R_0603_1608Metric_Pad1.05x0.95mm_HandSolder" V 2680 3500 50  0001 C CNN
+F 3 "~" H 2750 3500 50  0001 C CNN
+	1    2750 3500
+	0    1    1    0
+$EndComp
+Wire Wire Line
+	2600 3500 2050 3500
+Wire Wire Line
+	2050 3500 2050 3000
+Connection ~ 2050 3000
+Wire Wire Line
+	2900 3500 3050 3500
+Wire Wire Line
+	3050 3500 3050 2950
+Connection ~ 3050 2950
 $Comp
 L Device:R R806
@@
 	13250 2300 12800 2300
 Connection ~ 12800 2300
-Wire Wire Line
-	13850 2400 15050 2400
 $Comp
 L Amplifier_Operational:TL072 U810
@@
 Text Label 4650 8000 0    50   ~ 0
 +2V5REF
+Wire Wire Line
+	13850 2400 15050 2400
+$Comp
+L ETH1CPMU1:74AHCT1G08 U806
+U 1 1 5E75FDEB
+P 2400 2950
+F 0 "U806" H 2650 3150 50  0000 L CNN
+F 1 "74AHCT1G08" H 2500 3050 50  0000 L CNN
+F 2 "Package_TO_SOT_SMD:SOT-353_SC-70-5_Handsoldering" H 2400 2950 50  0001 C CNN
+F 3 "http://www.ti.com/lit/sg/scyt129e/scyt129e.pdf" H 2400 2950 50  0001 C CNN
+	1    2400 2950
+	1    0    0    -1
+$EndComp
+$Comp
+L power:+3.3VP #PWR0822
+U 1 1 5E761278
+P 2400 2750
+F 0 "#PWR0822" H 2550 2700 50  0001 C CNN
+F 1 "+3.3VP" H 2420 2893 50  0000 C CNN
+F 2 "" H 2400 2750 50  0001 C CNN
+F 3 "" H 2400 2750 50  0001 C CNN
+	1    2400 2750
+	1    0    0    -1
+$EndComp
+$Comp
+L ETH1CPMU1:DGNDF #PWR0824
+U 1 1 5E7D5BEA
+P 2400 3150
+F 0 "#PWR0824" H 2400 2900 50  0001 C CNN
+F 1 "DGNDF" H 2405 2977 50  0000 C CNN
+F 2 "" H 2400 3150 50  0001 C CNN
+F 3 "" H 2400 3150 50  0001 C CNN
+	1    2400 3150
+	1    0    0    -1
+$EndComp
 $EndSCHEMATC

Commit message: Schematic design
Parts:
- removed U809: DG419LEUA, Package_SO:MSOP-8_3x3mm_P0.65mm, symbol Analog_Switch:DG419LEUA
- added C841, C842: 100n, Capacitor_SMD:C_0603_1608Metric_Pad1.05x0.95mm_HandSolder, symbol Device:C
- added R838, R839, R841, R842, R843: 10k, Resistor_SMD:R_0603_1608Metric_Pad1.05x0.95mm_HandSolder, symbol Device:R
- added R840: 70k, Resistor_SMD:R_0603_1608Metric_Pad1.05x0.95mm_HandSolder, symbol Device:R
- added U809: DG408DY, Package_SO:TSSOP-16_4.4x5mm_P0.65mm, symbol ETH1CPMU1:DG408DY
- added U815: TXB0104D, Package_SO:SOIC-14_3.9x8.7mm_P1.27mm, symbol Logic_LevelTranslator:TXB0104D
Connections:
- net +15VF: now also C841.1, U809.13 (V+)
- net +3.3VP: now also R839.1, U815.1 (VCCA)
- net +5VF: now also R838.2, U815.14 (VCCB)
- net -15VF: now also C842.1, U809.3 (V-)
- net AGNDF: now also C841.2, C842.2, R841.2, R843.2, U809.14 (GND), U809.4 (S0)
- net DGNDF: now also U815.7 (GND)
- net MEAS_AMPL: now also U809.5 (S1)
- net MEAS_OUT: now also R840.2
- net DDS_FGEN_FSELECT: now reaches U804.10 (FSELECT)
- net at U810.3 (+): now also U809.8 (D)
- net at R823.2, R832.2, U814.1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: now also R842.1
- new net: U809.1 (A0), U815.11 (B3)
- new net: U809.15 (A2), U815.13 (B1)
- new net: U809.16 (A1), U815.12 (B2)
- new net: R838.1, U809.2 (EN)
- new net: R840.1, R841.1, U809.6 (S2)
- new net: R842.2, R843.1, U809.7 (S3)
- new net: R839.2, U815.8 (OE)
- new net DDS_MEAS_A0: U815.4 (A3)
- new net DDS_MEAS_A1: U815.3 (A2)
- new net DDS_MEAS_A2: U815.2 (A1)
- no-connect marks 11 -> 17
Other:
- moved on the sheet: C801, C802, C803, C804, C805, C806, C807, C808, C809, C810, C811, C812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
