File: hardware/project/ETH1CPMU1/MCU_Second.sch (KiCad schematic (older format))
At the start: 26 parts, among them J1301 Conn_02x05, U1301 STM32H743ZI, U1302 24LC08, Y1301 NX3225GD-8MHZ-STD-CRA-3

Commit message: Schematic and PCB design.
Parts:
- U1302: value 24LC08 -> 24LC08B-E/MS; footprint (none) -> Package_SO:MSOP-8_3x3mm_P0.65mm
- renumbered R1303 to R1301, R1304 to R1302, R1301 to R1303, R1302 to R1304
Connections:
- net GND is gone; now on net DGNDF: C1305.2
Other:
- moved on the sheet: R1303, R1304, U1302
Changed lines of the file:
@@
 	8600 950  8600 900
 $Comp
-L ETH1CPMU1:DGNDF #PWR01312
+L ETH1CPMU1:DGNDF #PWR01308
 U 1 1 5DD30B8E
 P 8600 9200
-F 0 "#PWR01312" H 8600 8950 50  0001 C CNN
+F 0 "#PWR01308" H 8600 8950 50  0001 C CNN
 F 1 "DGNDF" H 8605 9027 50  0000 C CNN
 F 2 "" H 8600 9200 50  0001 C CNN
@@
 	8600 9200 8600 9150
 $Comp
-L Device:R R1304
+L Device:R R1302
 U 1 1 5DD38026
 P 14400 9000
-F 0 "R1304" H 14470 9046 50  0000 L CNN
+F 0 "R1302" H 14470 9046 50  0000 L CNN
 F 1 "10k" H 14470 8955 50  0000 L CNN
 F 2 "Resistor_SMD:R_0603_1608Metric_Pad1.05x0.95mm_HandSolder" V 14330 9000 50  0001 C CNN
@@
 	14400 8800 14300 8800
 $Comp
-L ETH1CPMU1:DGNDF #PWR01313
+L ETH1CPMU1:DGNDF #PWR01309
 U 1 1 5DD3A05C
 P 14400 9200
-F 0 "#PWR01313" H 14400 8950 50  0001 C CNN
+F 0 "#PWR01309" H 14400 8950 50  0001 C CNN
 F 1 "DGNDF" H 14405 9027 50  0000 C CNN
 F 2 "" H 14400 9200 50  0001 C CNN
@@
 MCU_NRST
 $Comp
-L ETH1CPMU1:DGNDF #PWR01316
+L ETH1CPMU1:DGNDF #PWR01314
 U 1 1 5DD90023
 P 10250 10700
-F 0 "#PWR01316" H 10250 10450 50  0001 C CNN
+F 0 "#PWR01314" H 10250 10450 50  0001 C CNN
 F 1 "DGNDF" H 10255 10527 50  0000 C CNN
 F 2 "" H 10250 10700 50  0001 C CNN
@@
 $EndComp
 $Comp
-L ETH1CPMU1:+3.3VF #PWR01314
+L ETH1CPMU1:+3.3VF #PWR01311
 U 1 1 5DD9082D
 P 10250 10150
-F 0 "#PWR01314" H 10250 10000 50  0001 C CNN
+F 0 "#PWR01311" H 10250 10000 50  0001 C CNN
 F 1 "+3.3VF" H 10265 10323 50  0000 C CNN
 F 2 "" H 10250 10150 50  0001 C CNN
@@
 L Memory_EEPROM:24LC08 U?
 U 1 1 5E237856
-P 1150 7350
+P 8200 10500
 AR Path="/5DCED281/5E237856" Ref="U?"  Part="1"
 AR Path="/5DF35BC8/5E237856" Ref="U1302"  Part="1"
-F 0 "U1302" H 1350 7700 50  0000 C CNN
-F 1 "24LC08" H 1350 7600 50  0000 C CNN
-F 2 "" H 1150 7350 50  0001 C CNN
-F 3 "http://ww1.microchip.com/downloads/en/DeviceDoc/21710J.pdf" H 1150 7350 50  0001 C CNN
-	1    1150 7350
-	1    0    0    -1
-$EndComp
-Wire Wire Line
-	750  7250 700  7250
-Wire Wire Line
-	700  7250 700  7350
-Wire Wire Line
-	700  7450 750  7450
-Wire Wire Line
-	700  7650 700  7450
-Connection ~ 700  7450
-Wire Wire Line
-	750  7350 700  7350
-Connection ~ 700  7350
-Wire Wire Line
-	700  7350 700  7450
-Wire Wire Line
-	1550 7450 2050 7450
-Text Label 2050 7450 2    50   ~ 0
+F 0 "U1302" H 8550 10850 50  0000 C CNN
+F 1 "24LC08B-E/MS" H 8600 10750 50  0000 C CNN
+F 2 "Package_SO:MSOP-8_3x3mm_P0.65mm" H 8200 10500 50  0001 C CNN
+F 3 "http://ww1.microchip.com/downloads/en/DeviceDoc/21710J.pdf" H 8200 10500 50  0001 C CNN
+	1    8200 10500
+	1    0    0    -1
+$EndComp
+Wire Wire Line
+	7800 10400 7750 10400
+Wire Wire Line
+	7750 10400 7750 10500
+Wire Wire Line
+	7750 10600 7800 10600
+Wire Wire Line
+	7750 10800 7750 10600
+Connection ~ 7750 10600
+Wire Wire Line
+	7800 10500 7750 10500
+Connection ~ 7750 10500
+Wire Wire Line
+	7750 10500 7750 10600
+Wire Wire Line
+	8600 10600 9100 10600
+Text Label 9100 10600 2    50   ~ 0
 EEPROM_WP
-Text Label 2050 7350 2    50   ~ 0
+Text Label 9100 10500 2    50   ~ 0
 EEPROM_SCL
-Text Label 2050 7250 2    50   ~ 0
+Text Label 9100 10400 2    50   ~ 0
 EEPROM_SDA
 $Comp
 L Device:R R?
 U 1 1 5E23787A
-P 2100 7050
+P 9150 10200
 AR Path="/5DCED281/5E23787A" Ref="R?"  Part="1"
-AR Path="/5DF35BC8/5E23787A" Ref="R1301"  Part="1"
-F 0 "R1301" H 2170 7096 50  0000 L CNN
-F 1 "4k7" H 2170 7005 50  0000 L CNN
-F 2 "Resistor_SMD:R_0603_1608Metric_Pad1.05x0.95mm_HandSolder" V 2030 7050 50  0001 C CNN
-F 3 "~" H 2100 7050 50  0001 C CNN
-	1    2100 7050
+AR Path="/5DF35BC8/5E23787A" Ref="R1303"  Part="1"
+F 0 "R1303" H 9220 10246 50  0000 L CNN
+F 1 "4k7" H 9220 10155 50  0000 L CNN
+F 2 "Resistor_SMD:R_0603_1608Metric_Pad1.05x0.95mm_HandSolder" V 9080 10200 50  0001 C CNN
+F 3 "~" H 9150 10200 50  0001 C CNN
+	1    9150 10200
 	1    0    0    -1
 $EndComp
@@
 L Device:R R?
 U 1 1 5E237880
-P 2450 7050
+P 9500 10200
 AR Path="/5DCED281/5E237880" Ref="R?"  Part="1"
-AR Path="/5DF35BC8/5E237880" Ref="R1302"  Part="1"
-F 0 "R1302" H 2520 7096 50  0000 L CNN
-F 1 "4k7" H 2520 7005 50  0000 L CNN
-F 2 "Resistor_SMD:R_0603_1608Metric_Pad1.05x0.95mm_HandSolder" V 2380 7050 50  0001 C CNN
-F 3 "~" H 2450 7050 50  0001 C CNN
-	1    2450 7050
-	1    0    0    -1
-$EndComp
-Wire Wire Line
-	2100 7250 2100 7200
-Wire Wire Line
-	1550 7250 2100 7250
-Wire Wire Line
-	2450 7350 2450 7200
-Wire Wire Line
-	1550 7350 2450 7350
-Wire Wire Line
-	2100 6900 2100 6850
-Wire Wire Line
-	2100 6850 2450 6850
-Wire Wire Line
-	2450 6850 2450 6900
-Wire Wire Line
-	2450 6800 2450 6850
-Connection ~ 2450 6850
-$Comp
-L ETH1CPMU1:DGNDF #PWR01306
+AR Path="/5DF35BC8/5E237880" Ref="R1304"  Part="1"
+F 0 "R1304" H 9570 10246 50  0000 L CNN
+F 1 "4k7" H 9570 10155 50  0000 L CNN
+F 2 "Resistor_SMD:R_0603_1608Metric_Pad1.05x0.95mm_HandSolder" V 9430 10200 50  0001 C CNN
+F 3 "~" H 9500 10200 50  0001 C CNN
+	1    9500 10200
+	1    0    0    -1
+$EndComp
+Wire Wire Line
+	9150 10400 9150 10350
+Wire Wire Line
+	8600 10400 9150 10400
+Wire Wire Line
+	9500 10500 9500 10350
+Wire Wire Line
+	8600 10500 9500 10500
+Wire Wire Line
+	9150 10050 9150 10000
+Wire Wire Line
+	9150 10000 9500 10000
+Wire Wire Line
+	9500 10000 9500 10050
+Wire Wire Line
+	9500 9950 9500 10000
+Connection ~ 9500 10000
+$Comp
+L ETH1CPMU1:DGNDF #PWR01316
 U 1 1 5E23BC5E
-P 1150 7650
-F 0 "#PWR01306" H 1150 7400 50  0001 C CNN
-F 1 "DGNDF" H 1155 7477 50  0000 C CNN
-F 2 "" H 1150 7650 50  0001 C CNN
-F 3 "" H 1150 7650 50  0001 C CNN
-	1    1150 7650
-	1    0    0    -1
-$EndComp
-$Comp
-L ETH1CPMU1:DGNDF #PWR01305
+P 8200 10800
+F 0 "#PWR01316" H 8200 10550 50  0001 C CNN
+F 1 "DGNDF" H 8205 10627 50  0000 C CNN
+F 2 "" H 8200 10800 50  0001 C CNN
+F 3 "" H 8200 10800 50  0001 C CNN
+	1    8200 10800
+	1    0    0    -1
+$EndComp
+$Comp
+L ETH1CPMU1:DGNDF #PWR01315
 U 1 1 5E23BDCF
-P 700 7650
-F 0 "#PWR01305" H 700 7400 50  0001 C CNN
-F 1 "DGNDF" H 705 7477 50  0000 C CNN
-F 2 "" H 700 7650 50  0001 C CNN
-F 3 "" H 700 7650 50  0001 C CNN
-	1    700  7650
-	1    0    0    -1
-$EndComp
-$Comp
-L ETH1CPMU1:+3.3VF #PWR01304
+P 7750 10800
+F 0 "#PWR01315" H 7750 10550 50  0001 C CNN
+F 1 "DGNDF" H 7755 10627 50  0000 C CNN
+F 2 "" H 7750 10800 50  0001 C CNN
+F 3 "" H 7750 10800 50  0001 C CNN
+	1    7750 10800
+	1    0    0    -1
+$EndComp
+$Comp
+L ETH1CPMU1:+3.3VF #PWR01312
 U 1 1 5E23D8BE
-P 1150 7050
-F 0 "#PWR01304" H 1150 6900 50  0001 C CNN
-F 1 "+3.3VF" H 1165 7223 50  0000 C CNN
-F 2 "" H 1150 7050 50  0001 C CNN
-F 3 "" H 1150 7050 50  0001 C CNN
-	1    1150 7050
-	1    0    0    -1
-$EndComp
-$Comp
-L ETH1CPMU1:+3.3VF #PWR01303
+P 8200 10200
+F 0 "#PWR01312" H 8200 10050 50  0001 C CNN
+F 1 "+3.3VF" H 8215 10373 50  0000 C CNN
+F 2 "" H 8200 10200 50  0001 C CNN
+F 3 "" H 8200 10200 50  0001 C CNN
+	1    8200 10200
+	1    0    0    -1
+$EndComp
+$Comp
+L ETH1CPMU1:+3.3VF #PWR01310
 U 1 1 5E23DAAC
-P 2450 6800
-F 0 "#PWR01303" H 2450 6650 50  0001 C CNN
-F 1 "+3.3VF" H 2465 6973 50  0000 C CNN
-F 2 "" H 2450 6800 50  0001 C CNN
-F 3 "" H 2450 6800 50  0001 C CNN
-	1    2450 6800
+P 9500 9950
+F 0 "#PWR01310" H 9500 9800 50  0001 C CNN
+F 1 "+3.3VF" H 9515 10123 50  0000 C CNN
+F 2 "" H 9500 9950 50  0001 C CNN
+F 3 "" H 9500 9950 50  0001 C CNN
+	1    9500 9950
 	1    0    0    -1
 $EndComp
@@
 	2850 8800 2900 8800
 $Comp
-L ETH1CPMU1:+3.3VF #PWR01310
+L ETH1CPMU1:+3.3VF #PWR01306
 U 1 1 5E2661C9
 P 2800 8800
-F 0 "#PWR01310" H 2800 8650 50  0001 C CNN
+F 0 "#PWR01306" H 2800 8650 50  0001 C CNN
 F 1 "+3.3VF" V 2800 8950 50  0000 L CNN
 F 2 "" H 2800 8800 50  0001 C CNN
@@
 	3400 10450 3650 10450
 $Comp
-L ETH1CPMU1:+3.3VF #PWR01315
+L ETH1CPMU1:+3.3VF #PWR01313
 U 1 1 5DFCC179
 P 3400 10400
-F 0 "#PWR01315" H 3400 10250 50  0001 C CNN
+F 0 "#PWR01313" H 3400 10250 50  0001 C CNN
 F 1 "+3.3VF" H 3415 10573 50  0000 C CNN
 F 2 "" H 3400 10400 50  0001 C CNN
@@
 $EndComp
 $Comp
-L ETH1CPMU1:DGNDF #PWR01311
+L ETH1CPMU1:DGNDF #PWR01307
 U 1 1 5DFCF40C
 P 2850 9200
-F 0 "#PWR01311" H 2850 8950 50  0001 C CNN
+F 0 "#PWR01307" H 2850 8950 50  0001 C CNN
 F 1 "DGNDF" H 2855 9027 50  0000 C CNN
 F 2 "" H 2850 9200 50  0001 C CNN
@@
 $EndComp
 $Comp
-L ETH1CPMU1:DGNDF #PWR01308
+L ETH1CPMU1:DGNDF #PWR01304
 U 1 1 5DFCF998
 P 1950 8450
-F 0 "#PWR01308" H 1950 8200 50  0001 C CNN
+F 0 "#PWR01304" H 1950 8200 50  0001 C CNN
 F 1 "DGNDF" H 1955 8277 50  0000 C CNN
 F 2 "" H 1950 8450 50  0001 C CNN
@@
 P 15200 8200
 AR Path="/5DCED281/5E806B33" Ref="R?"  Part="1"
-AR Path="/5DF35BC8/5E806B33" Ref="R1303"  Part="1"
-F 0 "R1303" H 15270 8246 50  0000 L CNN
+AR Path="/5DF35BC8/5E806B33" Ref="R1301"  Part="1"
+F 0 "R1301" H 15270 8246 50  0000 L CNN
 F 1 "10k" H 15270 8155 50  0000 L CNN
 F 2 "Resistor_SMD:R_0603_1608Metric_Pad1.05x0.95mm_HandSolder" V 15130 8200 50  0001 C CNN
@@
 	15200 8350 15200 8400
 Connection ~ 15200 8400
-$Comp
-L power:GND #PWR?
-U 1 1 5E806B42
-P 15200 8750
-AR Path="/5DCED281/5E806B42" Ref="#PWR?"  Part="1"
-AR Path="/5DF35BC8/5E806B42" Ref="#PWR01309"  Part="1"
-F 0 "#PWR01309" H 15200 8500 50  0001 C CNN
-F 1 "GND" H 15205 8577 50  0000 C CNN
-F 2 "" H 15200 8750 50  0001 C CNN
-F 3 "" H 15200 8750 50  0001 C CNN
-	1    15200 8750
-	1    0    0    -1
-$EndComp
 Wire Wire Line
 	15700 8400 15200 8400
@@
 	14350 7800 14300 7800
 $Comp
-L ETH1CPMU1:+3.3VF #PWR01307
+L ETH1CPMU1:+3.3VF #PWR01303
 U 1 1 5E8AA48C
 P 15200 8050
-F 0 "#PWR01307" H 15200 7900 50  0001 C CNN
+F 0 "#PWR01303" H 15200 7900 50  0001 C CNN
 F 1 "+3.3VF" H 15215 8223 50  0000 C CNN
 F 2 "" H 15200 8050 50  0001 C CNN
@@
 NoConn ~ 14300 7600
 NoConn ~ 14300 7700
+$Comp
+L ETH1CPMU1:DGNDF #PWR01305
+U 1 1 5E492D3A
+P 15200 8750
+F 0 "#PWR01305" H 15200 8500 50  0001 C CNN
+F 1 "DGNDF" H 15205 8577 50  0000 C CNN
+F 2 "" H 15200 8750 50  0001 C CNN
+F 3 "" H 15200 8750 50  0001 C CNN
+	1    15200 8750
+	1    0    0    -1
+$EndComp
 $EndSCHEMATC

Commit message: Schematic design
Connections:
- net DAC_DIN renamed DAC_SDIN
Changed lines of the file:
@@
 	14300 3700 14350 3700
 Text HLabel 2850 6200 0    50   Output ~ 0
-DAC_DIN
+DAC_SDIN
 Text HLabel 2850 6000 0    50   Output ~ 0
 DAC_SCLK

Commit message: Schematic design
Parts:
- added C1519: 1u, Capacitor_SMD:C_0603_1608Metric_Pad1.05x0.95mm_HandSolder, symbol Device:C
- added FB1501: 742792031, Inductor_SMD:L_0805_2012Metric_Pad1.15x1.40mm_HandSolder, symbol Device:Ferrite_Bead
- renumbered C1301 to C1501, C1302 to C1502, C1303 to C1503, C1304 to C1504, C1305 to C1505, C1306 to C1506, C1307 to C1507, C1308 to C1508, C1309 to C1509, C1310 to C1510, C1311 to C1511, C1312 to C1512, C1313 to C1513, C1314 to C1514, C1315 to C1515, C1316 to C1516, C1317 to C1517, C1318 to C1518, J1301 to J1501, R1301 to R1501, R1302 to R1502, R1303 to R1503, R1304 to R1504, U1301 to U1501, U1302 to U1502, Y1301 to Y1501
Connections:
- net +3.3VF: now also FB1501.2
- net ADC_MUX_~SYNC: now also U1501.73 (PB12,TIM1_BKIN,I2C2_SMBA,SPI2_NSS,I2S2_WS,DFSDM1_DATIN1,USART3_CK,UART5_RX,CAN2_RX,OTG_HS_ULPI_D5,ETH_MII_TXD0,ETH_RMII_TXD0,OTG_HS_ID,EVENTOUT); no longer U1501.140 (PB9,I2C4_SDA,TIM4_CH4,TIM11_CH1,I2C1_SDA,SPI2_NSS,I2S2_WS,DFSDM1_DATIN7,UART5_TX,CAN1_TX,SDMMC2_D5,I2C4_SMBA,SDMMC1_D5,DCMI_D7,LCD_B7,EVENTOUT)
- net DAC_~LDAC: now also U1501.103 (PA11,TIM1_CH4,SPI2_NSS,I2S2_WS,UART4_RX,USART1_CTS,CAN1_RX,OTG_FS_DM,LCD_R4,EVENTOUT); no longer U1501.114 (PD0,DFSDM1_CKIN6,DFSDM1_DATIN7,UART4_RX,CAN1_RX,FMC_D2,EVENTOUT)
- net DGNDF: now also U1501.31 (VSSA), C1519.2
- net DAC_RSTSEL: now reaches U1501.102 (PA10,TIM1_CH3,USART1_RX,LCD_B4,OTG_FS_ID,MDIOS_MDIO,DCMI_D1,LCD_B1,EVENTOUT)
- net DAC_~RESET: now reaches U1501.104 (PA12,TIM1_ETR,SPI2_SCK,I2S2_CK,UART4_TX,USART1_RTS,SAI2_FS_B,CAN1_TX,OTG_FS_DP,LCD_R5,EVENTOUT)
- net DAC_SDO: now reaches U1501.112 (PC11,DFSDM1_DATIN5,SPI3_MISO,USART3_RX,UART4_RX,QUADSPI_BK2_NCS,SDMMC1_D3,DCMI_D4,EVENTOUT)
- net MCU3_MOSI: now reaches U1501.123 (PD7,DFSDM1_DATIN4,SPI1_MOSI,I2S1_SD,DFSDM1_CKIN1,USART2_CK,SPDIF_RX0,SDMMC2_CMD,FMC_NE1,EVENTOUT)
- net MCU3_MISO: now reaches U1501.124 (PG9,SPI1_MISO,SPDIF_RX3,USART6_RX,QUADSPI_BK2_IO2,SAI2_FS_B,SDMMC2_D0,FMC_NE2,FMC_NCE,DCMI_VSYNC,EVENTOUT)
- net MCU3_NSS: now reaches U1501.125 (PG10,SPI1_NSS,I2S1_WS,LCD_G3,SAI2_SD_B,SDMMC2_D1,FMC_NE3,DCMI_D2,LCD_B2,EVENTOUT)
- net MCU3_SCLK: now reaches U1501.126 (PG11,SPI1_SCK,I2S1_CK,SPDIF_RX0,SDMMC2_D2,ETH_MII_TX_EN,ETH_RMII_TX_EN,DCMI_D3,LCD_B3,EVENTOUT)
- net MCU_VDDA: now reaches U1501.32 (VREF+)
- net MCU_VDDA: now also U1501.33 (VDDA), C1519.1, FB1501.1; no longer U1501.31 (VSSA)
- net DAC_~CLR: no longer names the net of U1501.115 (PD1,DFSDM1_DATIN6,DFSDM1_CKIN7,UART4_TX,CAN1_TX,FMC_D3,EVENTOUT)
- no-connect marks 56 -> 54
Other:
- moved on the sheet: J1501, R1503, R1504, U1502
