File: hardware/project/ETH1CPMU1/MCU_Second.sch (KiCad schematic (older format))
At the start: 28 parts, among them J1501 Conn_02x05, U1501 STM32H743ZI, U1502 24LC08B-E/MS, Y1501 NX3225GD-8MHZ-STD-CRA-3

Commit message: PCB design.
Parts:
- renumbered C1519 to C1507, C1507 to C1508, C1508 to C1509, C1509 to C1510, C1510 to C1511, C1511 to C1512, C1512 to C1513, C1513 to C1514, C1514 to C1515, C1515 to C1516, C1516 to C1517, C1517 to C1518, C1518 to C1519
Connections:
- net ADC_CONVST: now reaches U1501.46 (PB0,TIM1_CH2N,TIM3_CH3,TIM8_CH2N,DFSDM1_CKOUT,UART4_CTS,_LCD_R3,OTG_HS_ULPI_D1,ETH_MII_RXD2,LCD_G1,EVENTOUT,ADC1_IN8,ADC2_IN8)
- no-connect marks 54 -> 53
Changed lines of the file:
@@
 	8600 950  8600 900
 $Comp
-L ETH1CPMU1:DGNDF #PWR01508
+L ETH1CPMU1:DGNDF #PWR01509
 U 1 1 5DD30B8E
 P 8600 9200
-F 0 "#PWR01508" H 8600 8950 50  0001 C CNN
+F 0 "#PWR01509" H 8600 8950 50  0001 C CNN
 F 1 "DGNDF" H 8605 9027 50  0000 C CNN
 F 2 "" H 8600 9200 50  0001 C CNN
@@
 	14400 8800 14300 8800
 $Comp
-L ETH1CPMU1:DGNDF #PWR01509
+L ETH1CPMU1:DGNDF #PWR01510
 U 1 1 5DD3A05C
 P 14400 9200
-F 0 "#PWR01509" H 14400 8950 50  0001 C CNN
+F 0 "#PWR01510" H 14400 8950 50  0001 C CNN
 F 1 "DGNDF" H 14405 9027 50  0000 C CNN
 F 2 "" H 14400 9200 50  0001 C CNN
@@
 MCU_NRST
 $Comp
-L ETH1CPMU1:DGNDF #PWR01514
+L ETH1CPMU1:DGNDF #PWR01516
 U 1 1 5DD90023
 P 10550 10700
-F 0 "#PWR01514" H 10550 10450 50  0001 C CNN
+F 0 "#PWR01516" H 10550 10450 50  0001 C CNN
 F 1 "DGNDF" H 10555 10527 50  0000 C CNN
 F 2 "" H 10550 10700 50  0001 C CNN
@@
 $EndComp
 $Comp
-L ETH1CPMU1:+3.3VF #PWR01511
+L ETH1CPMU1:+3.3VF #PWR01512
 U 1 1 5DD9082D
 P 10550 10150
-F 0 "#PWR01511" H 10550 10000 50  0001 C CNN
+F 0 "#PWR01512" H 10550 10000 50  0001 C CNN
 F 1 "+3.3VF" H 10565 10323 50  0000 C CNN
 F 2 "" H 10550 10150 50  0001 C CNN
@@
 Connection ~ 9800 10000
 $Comp
-L ETH1CPMU1:DGNDF #PWR01516
+L ETH1CPMU1:DGNDF #PWR01519
 U 1 1 5E23BC5E
 P 8500 10800
-F 0 "#PWR01516" H 8500 10550 50  0001 C CNN
+F 0 "#PWR01519" H 8500 10550 50  0001 C CNN
 F 1 "DGNDF" H 8505 10627 50  0000 C CNN
 F 2 "" H 8500 10800 50  0001 C CNN
@@
 $EndComp
 $Comp
-L ETH1CPMU1:DGNDF #PWR01515
+L ETH1CPMU1:DGNDF #PWR01518
 U 1 1 5E23BDCF
 P 8050 10800
-F 0 "#PWR01515" H 8050 10550 50  0001 C CNN
+F 0 "#PWR01518" H 8050 10550 50  0001 C CNN
 F 1 "DGNDF" H 8055 10627 50  0000 C CNN
 F 2 "" H 8050 10800 50  0001 C CNN
@@
 $EndComp
 $Comp
-L ETH1CPMU1:+3.3VF #PWR01512
+L ETH1CPMU1:+3.3VF #PWR01513
 U 1 1 5E23D8BE
 P 8500 10200
-F 0 "#PWR01512" H 8500 10050 50  0001 C CNN
+F 0 "#PWR01513" H 8500 10050 50  0001 C CNN
 F 1 "+3.3VF" H 8515 10373 50  0000 C CNN
 F 2 "" H 8500 10200 50  0001 C CNN
@@
 $EndComp
 $Comp
-L ETH1CPMU1:+3.3VF #PWR01510
+L ETH1CPMU1:+3.3VF #PWR01511
 U 1 1 5E23DAAC
 P 9800 9950
-F 0 "#PWR01510" H 9800 9800 50  0001 C CNN
+F 0 "#PWR01511" H 9800 9800 50  0001 C CNN
 F 1 "+3.3VF" H 9815 10123 50  0000 C CNN
 F 2 "" H 9800 9950 50  0001 C CNN
@@
 	2850 8800 2900 8800
 $Comp
-L ETH1CPMU1:+3.3VF #PWR01506
+L ETH1CPMU1:+3.3VF #PWR01507
 U 1 1 5E2661C9
 P 2800 8800
-F 0 "#PWR01506" H 2800 8650 50  0001 C CNN
+F 0 "#PWR01507" H 2800 8650 50  0001 C CNN
 F 1 "+3.3VF" V 2800 8950 50  0000 L CNN
 F 2 "" H 2800 8800 50  0001 C CNN
@@
 $EndComp
 $Comp
-L Device:C C1507
+L Device:C C1508
 U 1 1 5DFC30F8
 P 650 10650
-F 0 "C1507" H 765 10696 50  0000 L CNN
+F 0 "C1508" H 765 10696 50  0000 L CNN
 F 1 "100n" H 765 10605 50  0000 L CNN
 F 2 "Capacitor_SMD:C_0603_1608Metric_Pad1.05x0.95mm_HandSolder" H 688 10500 50  0001 C CNN
@@
 $EndComp
 $Comp
-L Device:C C1508
+L Device:C C1509
 U 1 1 5DFC30FE
 P 1150 10650
-F 0 "C1508" H 1265 10696 50  0000 L CNN
+F 0 "C1509" H 1265 10696 50  0000 L CNN
 F 1 "100n" H 1265 10605 50  0000 L CNN
 F 2 "Capacitor_SMD:C_0603_1608Metric_Pad1.05x0.95mm_HandSolder" H 1188 10500 50  0001 C CNN
@@
 $EndComp
 $Comp
-L Device:C C1509
+L Device:C C1510
 U 1 1 5DFC3104
 P 1650 10650
-F 0 "C1509" H 1765 10696 50  0000 L CNN
+F 0 "C1510" H 1765 10696 50  0000 L CNN
 F 1 "100n" H 1765 10605 50  0000 L CNN
 F 2 "Capacitor_SMD:C_0603_1608Metric_Pad1.05x0.95mm_HandSolder" H 1688 10500 50  0001 C CNN
@@
 $EndComp
 $Comp
-L Device:C C1510
+L Device:C C1511
 U 1 1 5DFC310A
 P 2150 10650
-F 0 "C1510" H 2265 10696 50  0000 L CNN
+F 0 "C1511" H 2265 10696 50  0000 L CNN
 F 1 "100n" H 2265 10605 50  0000 L CNN
 F 2 "Capacitor_SMD:C_0603_1608Metric_Pad1.05x0.95mm_HandSolder" H 2188 10500 50  0001 C CNN
@@
 $EndComp
 $Comp
-L Device:C C1511
+L Device:C C1512
 U 1 1 5DFC3110
 P 2650 10650
-F 0 "C1511" H 2765 10696 50  0000 L CNN
+F 0 "C1512" H 2765 10696 50  0000 L CNN
 F 1 "100n" H 2765 10605 50  0000 L CNN
 F 2 "Capacitor_SMD:C_0603_1608Metric_Pad1.05x0.95mm_HandSolder" H 2688 10500 50  0001 C CNN
@@
 $EndComp
 $Comp
-L Device:C C1512
+L Device:C C1513
 U 1 1 5DFC3116
 P 3150 10650
-F 0 "C1512" H 3265 10696 50  0000 L CNN
+F 0 "C1513" H 3265 10696 50  0000 L CNN
 F 1 "100n" H 3265 10605 50  0000 L CNN
 F 2 "Capacitor_SMD:C_0603_1608Metric_Pad1.05x0.95mm_HandSolder" H 3188 10500 50  0001 C CNN
@@
 $EndComp
 $Comp
-L Device:C C1513
+L Device:C C1514
 U 1 1 5DFC311C
 P 3650 10650
-F 0 "C1513" H 3765 10696 50  0000 L CNN
+F 0 "C1514" H 3765 10696 50  0000 L CNN
 F 1 "100n" H 3765 10605 50  0000 L CNN
 F 2 "Capacitor_SMD:C_0603_1608Metric_Pad1.05x0.95mm_HandSolder" H 3688 10500 50  0001 C CNN
@@
 $EndComp
 $Comp
-L Device:C C1514
+L Device:C C1515
 U 1 1 5DFC3122
 P 4150 10650
-F 0 "C1514" H 4265 10696 50  0000 L CNN
+F 0 "C1515" H 4265 10696 50  0000 L CNN
 F 1 "100n" H 4265 10605 50  0000 L CNN
 F 2 "Capacitor_SMD:C_0603_1608Metric_Pad1.05x0.95mm_HandSolder" H 4188 10500 50  0001 C CNN
@@
 $EndComp
 $Comp
-L Device:C C1515
+L Device:C C1516
 U 1 1 5DFC3128
 P 4650 10650
-F 0 "C1515" H 4765 10696 50  0000 L CNN
+F 0 "C1516" H 4765 10696 50  0000 L CNN
 F 1 "100n" H 4765 10605 50  0000 L CNN
 F 2 "Capacitor_SMD:C_0603_1608Metric_Pad1.05x0.95mm_HandSolder" H 4688 10500 50  0001 C CNN
@@
 $EndComp
 $Comp
-L Device:C C1516
+L Device:C C1517
 U 1 1 5DFC312E
 P 5150 10650
-F 0 "C1516" H 5265 10696 50  0000 L CNN
+F 0 "C1517" H 5265 10696 50  0000 L CNN
 F 1 "100n" H 5265 10605 50  0000 L CNN
 F 2 "Capacitor_SMD:C_0603_1608Metric_Pad1.05x0.95mm_HandSolder" H 5188 10500 50  0001 C CNN
@@
 $EndComp
 $Comp
-L Device:C C1517
+L Device:C C1518
 U 1 1 5DFC3134
 P 5650 10650
-F 0 "C1517" H 5765 10696 50  0000 L CNN
+F 0 "C1518" H 5765 10696 50  0000 L CNN
 F 1 "100n" H 5765 10605 50  0000 L CNN
 F 2 "Capacitor_SMD:C_0603_1608Metric_Pad1.05x0.95mm_HandSolder" H 5688 10500 50  0001 C CNN
@@
 $EndComp
 $Comp
-L Device:C C1518
+L Device:C C1519
 U 1 1 5DFC313A
 P 6150 10650
-F 0 "C1518" H 6265 10696 50  0000 L CNN
+F 0 "C1519" H 6265 10696 50  0000 L CNN
 F 1 "100n" H 6265 10605 50  0000 L CNN
 F 2 "Capacitor_SMD:C_0603_1608Metric_Pad1.05x0.95mm_HandSolder" H 6188 10500 50  0001 C CNN
@@
 	3400 10450 3650 10450
 $Comp
-L ETH1CPMU1:+3.3VF #PWR01513
+L ETH1CPMU1:+3.3VF #PWR01515
 U 1 1 5DFCC179
 P 3400 10400
-F 0 "#PWR01513" H 3400 10250 50  0001 C CNN
+F 0 "#PWR01515" H 3400 10250 50  0001 C CNN
 F 1 "+3.3VF" H 3415 10573 50  0000 C CNN
 F 2 "" H 3400 10400 50  0001 C CNN
@@
 $EndComp
 $Comp
-L ETH1CPMU1:DGNDF #PWR01517
+L ETH1CPMU1:DGNDF #PWR01520
 U 1 1 5DFCC68D
 P 3400 10900
-F 0 "#PWR01517" H 3400 10650 50  0001 C CNN
+F 0 "#PWR01520" H 3400 10650 50  0001 C CNN
 F 1 "DGNDF" H 3405 10727 50  0000 C CNN
 F 2 "" H 3400 10900 50  0001 C CNN
@@
 $EndComp
 $Comp
-L ETH1CPMU1:DGNDF #PWR01507
+L ETH1CPMU1:DGNDF #PWR01508
 U 1 1 5DFCF40C
 P 2850 9200
-F 0 "#PWR01507" H 2850 8950 50  0001 C CNN
+F 0 "#PWR01508" H 2850 8950 50  0001 C CNN
 F 1 "DGNDF" H 2855 9027 50  0000 C CNN
 F 2 "" H 2850 9200 50  0001 C CNN
@@
 NoConn ~ 14300 4700
 NoConn ~ 14300 4800
-NoConn ~ 14300 6400
-NoConn ~ 14300 6500
 NoConn ~ 14300 6600
 NoConn ~ 14300 6700
@@
 NoConn ~ 14300 7700
 $Comp
-L ETH1CPMU1:DGNDF #PWR01505
+L ETH1CPMU1:DGNDF #PWR01506
 U 1 1 5E492D3A
 P 15200 8750
-F 0 "#PWR01505" H 15200 8500 50  0001 C CNN
+F 0 "#PWR01506" H 15200 8500 50  0001 C CNN
 F 1 "DGNDF" H 15205 8577 50  0000 C CNN
 F 2 "" H 15200 8750 50  0001 C CNN
@@
 P 7250 10600
 AR Path="/5DCED281/5E2DFE17" Ref="C?"  Part="1"
-AR Path="/5DF35BC8/5E2DFE17" Ref="C1519"  Part="1"
-F 0 "C1519" H 7365 10646 50  0000 L CNN
+AR Path="/5DF35BC8/5E2DFE17" Ref="C1507"  Part="1"
+F 0 "C1507" H 7365 10646 50  0000 L CNN
 F 1 "1u" H 7365 10555 50  0000 L CNN
 F 2 "Capacitor_SMD:C_0603_1608Metric_Pad1.05x0.95mm_HandSolder" H 7288 10450 50  0001 C CNN
@@
 MCU_VDDA
 $Comp
-L ETH1CPMU1:+3.3VF #PWR0101
+L ETH1CPMU1:+3.3VF #PWR01514
 U 1 1 5E2EEABF
 P 6600 10350
-F 0 "#PWR0101" H 6600 10200 50  0001 C CNN
+F 0 "#PWR01514" H 6600 10200 50  0001 C CNN
 F 1 "+3.3VF" H 6615 10523 50  0000 C CNN
 F 2 "" H 6600 10350 50  0001 C CNN
@@
 $EndComp
 $Comp
-L ETH1CPMU1:DGNDF #PWR0102
+L ETH1CPMU1:DGNDF #PWR01517
 U 1 1 5E2F2EC2
 P 7250 10800
-F 0 "#PWR0102" H 7250 10550 50  0001 C CNN
+F 0 "#PWR01517" H 7250 10550 50  0001 C CNN
 F 1 "DGNDF" H 7255 10627 50  0000 C CNN
 F 2 "" H 7250 10800 50  0001 C CNN
@@
 $EndComp
 $Comp
-L ETH1CPMU1:DGNDF #PWR0103
+L ETH1CPMU1:DGNDF #PWR01505
 U 1 1 5E306998
 P 2850 8600
-F 0 "#PWR0103" H 2850 8350 50  0001 C CNN
+F 0 "#PWR01505" H 2850 8350 50  0001 C CNN
 F 1 "DGNDF" V 2855 8473 50  0000 R CNN
 F 2 "" H 2850 8600 50  0001 C CNN
@@
 Wire Wire Line
 	2850 8600 2900 8600
+Text HLabel 14350 6400 2    50   Output ~ 0
+ADC_CONVST
+Wire Wire Line
+	14350 6400 14300 6400
+NoConn ~ 14300 6500
 $EndSCHEMATC

Commit message: PCB design
Parts:
- renumbered C1508 to C1601, C1501 to C1602, C1509 to C1603, C1502 to C1604, C1510 to C1605, C1503 to C1606, C1504 to C1607, C1511 to C1608, C1512 to C1609, C1506 to C1610, C1513 to C1611, C1514 to C1612, C1515 to C1613, C1516 to C1614, C1517 to C1615, C1518 to C1616, C1519 to C1617, C1507 to C1618, C1505 to C1619, FB1501 to FB1601, J1501 to J1601, R1503 to R1601, R1504 to R1602, R1502 to R1603, R1501 to R1604, U1502 to U1601, U1501 to U1602, Y1501 to Y1601
Connections:
- net G1A0_CTR: now reaches U1602.114 (PD0,DFSDM1_CKIN6,DFSDM1_DATIN7,UART4_RX,CAN1_RX,FMC_D2,EVENTOUT)
- net G1A1_CTR: now reaches U1602.115 (PD1,DFSDM1_DATIN6,DFSDM1_CKIN7,UART4_TX,CAN1_TX,FMC_D3,EVENTOUT)
- net G2A0_CTR: now reaches U1602.116 (PD2,TRACED2,TIM3_ETR,UART5_RX,SDMMC1_CMD,DCMI_D11,EVENTOUT)
- net G2A1_CTR: now reaches U1602.117 (PD3,DFSDM1_CKOUT,SPI2_SCK,I2S2_CK,DFSDM1_DATIN0,USART2_CTS,FMC_CLK,DCMI_D5,LCD_G7,EVENTOUT)
- net G3A0_CTR: now reaches U1602.118 (PD4,DFSDM1_CKIN0,USART2_RTS,FMC_NOE,EVENTOUT)
- net G3A1_CTR: now reaches U1602.119 (PD5,USART2_TX,FMC_NWE,EVENTOUT)
- net DAC_RSTSEL: no longer names the net of U1602.102 (PA10,TIM1_CH3,USART1_RX,LCD_B4,OTG_FS_ID,MDIOS_MDIO,DCMI_D1,LCD_B1,EVENTOUT)
- net DAC_SDIN renamed DAC_DIN
- net DAC_SDO: no longer names the net of U1602.112 (PC11,DFSDM1_DATIN5,SPI3_MISO,USART3_RX,UART4_RX,QUADSPI_BK2_NCS,SDMMC1_D3,DCMI_D4,EVENTOUT)
- net DAC_~LDAC: no longer names the net of U1602.103 (PA11,TIM1_CH4,SPI2_NSS,I2S2_WS,UART4_RX,USART1_CTS,CAN1_RX,OTG_FS_DM,LCD_R4,EVENTOUT)
- net DAC_~RESET: no longer names the net of U1602.104 (PA12,TIM1_ETR,SPI2_SCK,I2S2_CK,UART4_TX,USART1_RTS,SAI2_FS_B,CAN1_TX,OTG_FS_DP,LCD_R5,EVENTOUT)
- no-connect marks 53 -> 51

Commit message: PCB designed
Parts:
- added C1620, C1621: 100n, Capacitor_SMD:C_0603_1608Metric_Pad1.05x0.95mm_HandSolder, symbol Device:C
- added R1605: 10k, Resistor_SMD:R_0603_1608Metric_Pad1.05x0.95mm_HandSolder, symbol Device:R
- added U1603: MCP23S17_ML, Package_DFN_QFN:QFN-28-1EP_6x6mm_P0.65mm_EP4.25x4.25mm, symbol Interface_Expansion:MCP23S17_ML
Connections:
- net DGNDF: now also C1620.2, C1621.2, U1603.11 (A0), U1603.12 (A1), U1603.13 (A2), U1603.29 (EP), U1603.6 (VSS)
- net G1A0_CTR: now also U1603.2 (GPB5); no longer U1602.114 (PD0,DFSDM1_CKIN6,DFSDM1_DATIN7,UART4_RX,CAN1_RX,FMC_D2,EVENTOUT)
- net G1A1_CTR: now also U1603.1 (GPB4); no longer U1602.115 (PD1,DFSDM1_DATIN6,DFSDM1_CKIN7,UART4_TX,CAN1_TX,FMC_D3,EVENTOUT)
- net G2A0_CTR: now also U1603.28 (GPB3); no longer U1602.116 (PD2,TRACED2,TIM3_ETR,UART5_RX,SDMMC1_CMD,DCMI_D11,EVENTOUT)
- net G2A1_CTR: now also U1603.27 (GPB2); no longer U1602.117 (PD3,DFSDM1_CKOUT,SPI2_SCK,I2S2_CK,DFSDM1_DATIN0,USART2_CTS,FMC_CLK,DCMI_D5,LCD_G7,EVENTOUT)
- net G3A0_CTR: now also U1603.4 (GPB7); no longer U1602.118 (PD4,DFSDM1_CKIN0,USART2_RTS,FMC_NOE,EVENTOUT)
- net G3A1_CTR: now also U1603.3 (GPB6); no longer U1602.119 (PD5,USART2_TX,FMC_NWE,EVENTOUT)
- net R_GND: now also U1603.20 (GPA3); no longer U1602.90 (PG5,FMC_A15,FMC_BA1,EVENTOUT)
- net R_GUARD: now also U1603.19 (GPA2); no longer U1602.93 (PG8,SPI6_NSS,SPDIF_RX2,USART6_RTS,ETH_PPS_OUT,FMC_SDCLK,LCD_G7,EVENTOUT)
- net R_GUARDIN: now also U1603.22 (GPA5); no longer U1602.89 (PG4,FMC_A14,FMC_BA0,EVENTOUT)
- net R_MEASHV: now also U1603.17 (GPA0); no longer U1602.88 (PG3,FMC_A13,EVENTOUT)
- net R_MEASIL: now also U1603.21 (GPA4); no longer U1602.91 (PG6,FMC_NE3,DCMI_D12,LCD_R7,EVENTOUT)
- net R_MEASVL: now also U1603.18 (GPA1); no longer U1602.92 (PG7,SAI1_MCLK_A,USART6_CK,FMC_INT,DCMI_D13,LCD_CLK,EVENTOUT)
- net GPIO_SO: now reaches U1602.127 (PG12,LPTIM1_IN1,SPI6_MISO,SPDIF_RX1,USART6_RTS,LCD_B4,SDMMC2_D3,FMC_NE4,LCD_B1,EVENTOUT)
- net GPIO_SO: now also U1603.10 (SO)
- net GPIO_SCK: now reaches U1602.128 (PG13,TRACED0,LPTIM1_OUT,SPI6_SCK,USART6_CTS,ETH_MII_TXD0,ETH_RMII_TXD0,FMC_A24,LCD_R0,EVENTOUT)
- net GPIO_SCK: now also U1603.8 (SCK)
- net GPIO_SI: now reaches U1602.129 (PG14,TRACED1,LPTIM1_ETR,SPI6_MOSI,USART6_TX,QUADSPI_BK2_IO3,ETH_MII_TXD1,ETH_RMII_TXD1,FMC_A25,LCD_B0,EVENTOUT)
- net GPIO_SI: now also U1603.9 (SI)
- net GPIO_~CS: now reaches U1602.132 (PG15,USART6_CTS,FMC_SDNCAS,DCMI_D13,EVENTOUT)
- net GPIO_~CS: now also U1603.7 (~CS~)
- new net: C1621.1, R1605.2, U1603.14 (~RESET~)
- new net +3.3VP: C1620.1, R1605.1, U1603.5 (VDD)
- no-connect marks 51 -> 65
Other:
- moved on the sheet: C1602, C1604, C1606, C1607, C1610, C1619, R1603, R1604, U1602, Y1601
