File: hardware/project/ETH1CPMU1/Power_Float.sch (KiCad schematic (older format))
At the start: 57 parts, among them U601 THL15-2415WI, U602 LM1117IMP-3.3/NOPB, U603 MC7815BD2TG, U604 LM1117IMP-3.3/NOPB, U605 TSR2-2450, U606 LT8330_S6, U607 MC7915BD2TG, U608 LM1117IMP-5.0/NOPB, U609 TSR1-2490, U610 LT8330_S6

Commit message: Schematic and PCB design.
Parts:
- added TP601: 5006, TestPoint:TestPoint_Loop_D2.60mm_Drill1.6mm_Beaded, symbol Connector:TestPoint
- C605, C612, C613, C623, C624: value 22u/16V -> 10u/16V; footprint Capacitor_SMD:C_2220_5650Metric_Pad1.97x5.40mm_HandSolder -> Capacitor_SMD:C_1206_3216Metric_Pad1.42x1.75mm_HandSolder
- C607, C620: footprint (none) -> Capacitor_SMD:C_1206_3216Metric_Pad1.42x1.75mm_HandSolder
- C608, C609, C610, C611, C621, C622: footprint Capacitor_SMD:C_1210_3225Metric_Pad1.42x2.65mm_HandSolder -> Capacitor_SMD:C_1206_3216Metric_Pad1.42x1.75mm_HandSolder
- L601: footprint (none) -> ETH1CPMU1:7448013501
- U601: footprint (none) -> ETH1CPMU1:THL15
- U605: footprint (none) -> ETH1CPMU1:TSR2
- U609: footprint (none) -> ETH1CPMU1:TSR1
Connections:
- net +24VDD: now also L601.2; no longer L601.1
- net AGNDF: now also TP601.1
- net GND: now also L601.1; no longer L601.2
- net at C606.2, U601.2 (-VIN): now also L601.4; no longer L601.3
- net at C601.2, U601.1 (+VIN): now also L601.3; no longer L601.4
Other:
- moved on the sheet: C615, C616, C617, C618, C626, C627, C628, C629, FB601, FB602, U603, U607

Commit message: Schematic design
Changed lines of the file:
@@
 	10700 3850 10700 3900
 $Comp
-L ETH1CPMU1:+3.3VF #PWR0611
+L ETH1CPMU1:+3.3VF #PWR0612
 U 1 1 5E155843
 P 10700 3100
-F 0 "#PWR0611" H 10700 2950 50  0001 C CNN
+F 0 "#PWR0612" H 10700 2950 50  0001 C CNN
 F 1 "+3.3VF" H 10715 3273 50  0000 C CNN
 F 2 "" H 10700 3100 50  0001 C CNN
@@
 	2200 4750 2200 4700
 $Comp
-L ETH1CPMU1:+24VF #PWR0608
+L ETH1CPMU1:+24VF #PWR0609
 U 1 1 5DD94C6F
 P 650 3100
-F 0 "#PWR0608" H 650 2950 50  0001 C CNN
+F 0 "#PWR0609" H 650 2950 50  0001 C CNN
 F 1 "+24VF" H 665 3273 50  0000 C CNN
 F 2 "" H 650 3100 50  0001 C CNN
@@
 Connection ~ 5750 3250
 $Comp
-L ETH1CPMU1:+15VF #PWR0609
+L ETH1CPMU1:+15VF #PWR0610
 U 1 1 5DDB9470
 P 6250 3100
-F 0 "#PWR0609" H 6250 2950 50  0001 C CNN
+F 0 "#PWR0610" H 6250 2950 50  0001 C CNN
 F 1 "+15VF" H 6265 3273 50  0000 C CNN
 F 2 "" H 6250 3100 50  0001 C CNN
@@
 	2200 6900 2200 6850
 $Comp
-L ETH1CPMU1:+24VF #PWR0616
+L ETH1CPMU1:+24VF #PWR0617
 U 1 1 5DE720EA
 P 650 5250
-F 0 "#PWR0616" H 650 5100 50  0001 C CNN
+F 0 "#PWR0617" H 650 5100 50  0001 C CNN
 F 1 "+24VF" H 665 5423 50  0000 C CNN
 F 2 "" H 650 5250 50  0001 C CNN
@@
 	10700 6000 10700 6050
 $Comp
-L ETH1CPMU1:+5VF #PWR0619
+L ETH1CPMU1:+5VF #PWR0620
 U 1 1 5DEE4B5F
 P 10700 5250
-F 0 "#PWR0619" H 10700 5100 50  0001 C CNN
+F 0 "#PWR0620" H 10700 5100 50  0001 C CNN
 F 1 "+5VF" H 10715 5423 50  0000 C CNN
 F 2 "" H 10700 5250 50  0001 C CNN
@@
 $EndComp
 $Comp
-L ETH1CPMU1:-15VF #PWR0617
+L ETH1CPMU1:-15VF #PWR0618
 U 1 1 5DF2FE99
 P 6250 5250
-F 0 "#PWR0617" H 6250 5100 50  0001 C CNN
+F 0 "#PWR0618" H 6250 5100 50  0001 C CNN
 F 1 "-15VF" H 6265 5423 50  0000 C CNN
 F 2 "" H 6250 5250 50  0001 C CNN
@@
 $EndComp
 $Comp
-L ETH1CPMU1:DGNDF #PWR0603
+L ETH1CPMU1:DGNDF #PWR0604
 U 1 1 5DF45BA9
 P 4200 1900
-F 0 "#PWR0603" H 4200 1650 50  0001 C CNN
+F 0 "#PWR0604" H 4200 1650 50  0001 C CNN
 F 1 "DGNDF" H 4205 1727 50  0000 C CNN
 F 2 "" H 4200 1900 50  0001 C CNN
@@
 $EndComp
 $Comp
-L ETH1CPMU1:DGNDF #PWR0615
+L ETH1CPMU1:DGNDF #PWR0616
 U 1 1 5DF46A7A
 P 2200 4750
-F 0 "#PWR0615" H 2200 4500 50  0001 C CNN
+F 0 "#PWR0616" H 2200 4500 50  0001 C CNN
 F 1 "DGNDF" H 2205 4577 50  0000 C CNN
 F 2 "" H 2200 4750 50  0001 C CNN
@@
 $EndComp
 $Comp
-L ETH1CPMU1:DGNDF #PWR0612
+L ETH1CPMU1:DGNDF #PWR0613
 U 1 1 5DF487C8
 P 2700 3700
-F 0 "#PWR0612" H 2700 3450 50  0001 C CNN
+F 0 "#PWR0613" H 2700 3450 50  0001 C CNN
 F 1 "DGNDF" H 2705 3527 50  0000 C CNN
 F 2 "" H 2700 3700 50  0001 C CNN
@@
 $EndComp
 $Comp
-L ETH1CPMU1:DGNDF #PWR0623
+L ETH1CPMU1:DGNDF #PWR0624
 U 1 1 5DF49793
 P 2200 6900
-F 0 "#PWR0623" H 2200 6650 50  0001 C CNN
+F 0 "#PWR0624" H 2200 6650 50  0001 C CNN
 F 1 "DGNDF" H 2205 6727 50  0000 C CNN
 F 2 "" H 2200 6900 50  0001 C CNN
@@
 $EndComp
 $Comp
-L ETH1CPMU1:DGNDF #PWR0622
+L ETH1CPMU1:DGNDF #PWR0623
 U 1 1 5DF4DCC7
 P 10700 6050
-F 0 "#PWR0622" H 10700 5800 50  0001 C CNN
+F 0 "#PWR0623" H 10700 5800 50  0001 C CNN
 F 1 "DGNDF" H 10705 5877 50  0000 C CNN
 F 2 "" H 10700 6050 50  0001 C CNN
@@
 $EndComp
 $Comp
-L ETH1CPMU1:DGNDF #PWR0614
+L ETH1CPMU1:DGNDF #PWR0615
 U 1 1 5DF4E402
 P 10700 3900
-F 0 "#PWR0614" H 10700 3650 50  0001 C CNN
+F 0 "#PWR0615" H 10700 3650 50  0001 C CNN
 F 1 "DGNDF" H 10705 3727 50  0000 C CNN
 F 2 "" H 10700 3900 50  0001 C CNN
@@
 $EndComp
 $Comp
-L ETH1CPMU1:DGNDF #PWR0606
+L ETH1CPMU1:DGNDF #PWR0607
 U 1 1 5E4E760E
 P 10200 2550
-F 0 "#PWR0606" H 10200 2300 50  0001 C CNN
+F 0 "#PWR0607" H 10200 2300 50  0001 C CNN
 F 1 "DGNDF" H 10205 2377 50  0000 C CNN
 F 2 "" H 10200 2550 50  0001 C CNN
@@
 	10200 2550 10200 2350
 $Comp
-L ETH1CPMU1:DGNDF #PWR0607
+L ETH1CPMU1:DGNDF #PWR0608
 U 1 1 5E4F37FA
 P 10700 2550
-F 0 "#PWR0607" H 10700 2300 50  0001 C CNN
+F 0 "#PWR0608" H 10700 2300 50  0001 C CNN
 F 1 "DGNDF" H 10705 2377 50  0000 C CNN
 F 2 "" H 10700 2550 50  0001 C CNN
@@
 Connection ~ 10700 2050
 $Comp
-L ETH1CPMU1:DGNDF #PWR0620
+L ETH1CPMU1:DGNDF #PWR0621
 U 1 1 5F7AA41C
 P 2700 5850
-F 0 "#PWR0620" H 2700 5600 50  0001 C CNN
+F 0 "#PWR0621" H 2700 5600 50  0001 C CNN
 F 1 "DGNDF" H 2705 5677 50  0000 C CNN
 F 2 "" H 2700 5850 50  0001 C CNN
@@
 	7100 3100 7100 3250
 $Comp
-L ETH1CPMU1:+24VF #PWR0610
+L ETH1CPMU1:+24VF #PWR0611
 U 1 1 5E1C68D9
 P 7100 3100
-F 0 "#PWR0610" H 7100 2950 50  0001 C CNN
+F 0 "#PWR0611" H 7100 2950 50  0001 C CNN
 F 1 "+24VF" H 7115 3273 50  0000 C CNN
 F 2 "" H 7100 3100 50  0001 C CNN
@@
 $EndComp
 $Comp
-L ETH1CPMU1:DGNDF #PWR0613
+L ETH1CPMU1:DGNDF #PWR0614
 U 1 1 5DF4F662
 P 7100 3900
-F 0 "#PWR0613" H 7100 3650 50  0001 C CNN
+F 0 "#PWR0614" H 7100 3650 50  0001 C CNN
 F 1 "DGNDF" H 7105 3727 50  0000 C CNN
 F 2 "" H 7100 3900 50  0001 C CNN
@@
 $EndComp
 $Comp
-L ETH1CPMU1:DGNDF #PWR0624
+L ETH1CPMU1:DGNDF #PWR0625
 U 1 1 5E1AEE0F
 P 650 7450
-F 0 "#PWR0624" H 650 7200 50  0001 C CNN
+F 0 "#PWR0625" H 650 7200 50  0001 C CNN
 F 1 "DGNDF" H 655 7277 50  0000 C CNN
 F 2 "" H 650 7450 50  0001 C CNN
@@
 Connection ~ 8150 5400
 $Comp
-L ETH1CPMU1:DGNDF #PWR0621
+L ETH1CPMU1:DGNDF #PWR0622
 U 1 1 5DF4AD33
 P 7950 6050
-F 0 "#PWR0621" H 7950 5800 50  0001 C CNN
+F 0 "#PWR0622" H 7950 5800 50  0001 C CNN
 F 1 "DGNDF" H 7955 5877 50  0000 C CNN
 F 2 "" H 7950 6050 50  0001 C CNN
@@
 	7950 5250 7950 5400
 $Comp
-L ETH1CPMU1:+24VF #PWR0618
+L ETH1CPMU1:+24VF #PWR0619
 U 1 1 5DED3D95
 P 7950 5250
-F 0 "#PWR0618" H 7950 5100 50  0001 C CNN
+F 0 "#PWR0619" H 7950 5100 50  0001 C CNN
 F 1 "+24VF" H 7965 5423 50  0000 C CNN
 F 2 "" H 7950 5250 50  0001 C CNN
@@
 AR Path="/5DC846AF/5DCFB9B5" Ref="#PWR?"  Part="1"
 AR Path="/5DCE1F8B/5DCFB9B5" Ref="#PWR?"  Part="1"
-AR Path="/5DD0DBE6/5DCFB9B5" Ref="#PWR0605"  Part="1"
-F 0 "#PWR0605" H 650 1700 50  0001 C CNN
+AR Path="/5DD0DBE6/5DCFB9B5" Ref="#PWR0606"  Part="1"
+F 0 "#PWR0606" H 650 1700 50  0001 C CNN
 F 1 "GND" H 655 1777 50  0000 C CNN
 F 2 "" H 650 1950 50  0001 C CNN
@@
 $EndComp
 $Comp
-L power:+3.3VP #PWR0604
+L power:+3.3VP #PWR0605
 U 1 1 5E73326F
 P 10700 1900
-F 0 "#PWR0604" H 10850 1850 50  0001 C CNN
+F 0 "#PWR0605" H 10850 1850 50  0001 C CNN
 F 1 "+3.3VP" H 10720 2043 50  0000 C CNN
 F 2 "" H 10700 1900 50  0001 C CNN
@@
 $EndComp
 $Comp
-L ETH1CPMU1:AGNDF #PWR0625
+L ETH1CPMU1:AGNDF #PWR0603
 U 1 1 5E7FA273
 P 3850 1900
-F 0 "#PWR0625" H 3850 1650 50  0001 C CNN
+F 0 "#PWR0603" H 3850 1650 50  0001 C CNN
 F 1 "AGNDF" H 3855 1727 50  0000 C CNN
 F 2 "" H 3850 1900 50  0001 C CNN
@@
 Wire Wire Line
 	3850 1850 4200 1850
+$Comp
+L ETH1CPMU1:+24VF #PWR0626
+U 1 1 5DE107B6
+P 1250 7450
+F 0 "#PWR0626" H 1250 7300 50  0001 C CNN
+F 1 "+24VF" H 1265 7623 50  0000 C CNN
+F 2 "" H 1250 7450 50  0001 C CNN
+F 3 "" H 1250 7450 50  0001 C CNN
+	1    1250 7450
+	1    0    0    -1
+$EndComp
+$Comp
+L power:PWR_FLAG #FLG0605
+U 1 1 5DE10F55
+P 1250 7450
+F 0 "#FLG0605" H 1250 7525 50  0001 C CNN
+F 1 "PWR_FLAG" H 1250 7623 50  0000 C CNN
+F 2 "" H 1250 7450 50  0001 C CNN
+F 3 "~" H 1250 7450 50  0001 C CNN
+	1    1250 7450
+	-1   0    0    1
+$EndComp
+$Comp
+L power:PWR_FLAG #FLG0606
+U 1 1 5DE489FC
+P 1700 7450
+F 0 "#FLG0606" H 1700 7525 50  0001 C CNN
+F 1 "PWR_FLAG" H 1700 7623 50  0000 C CNN
+F 2 "" H 1700 7450 50  0001 C CNN
+F 3 "~" H 1700 7450 50  0001 C CNN
+	1    1700 7450
+	-1   0    0    1
+$EndComp
+$Comp
+L ETH1CPMU1:+15VF #PWR0627
+U 1 1 5DE48F13
+P 1700 7450
+F 0 "#PWR0627" H 1700 7300 50  0001 C CNN
+F 1 "+15VF" H 1715 7623 50  0000 C CNN
+F 2 "" H 1700 7450 50  0001 C CNN
+F 3 "" H 1700 7450 50  0001 C CNN
+	1    1700 7450
+	1    0    0    -1
+$EndComp
+$Comp
+L power:PWR_FLAG #FLG0607
+U 1 1 5DE4A092
+P 2150 7450
+F 0 "#FLG0607" H 2150 7525 50  0001 C CNN
+F 1 "PWR_FLAG" H 2150 7623 50  0000 C CNN
+F 2 "" H 2150 7450 50  0001 C CNN
+F 3 "~" H 2150 7450 50  0001 C CNN
+	1    2150 7450
+	-1   0    0    1
+$EndComp
+$Comp
+L ETH1CPMU1:-15VF #PWR0628
+U 1 1 5DE5688B
+P 2150 7450
+F 0 "#PWR0628" H 2150 7300 50  0001 C CNN
+F 1 "-15VF" H 2165 7623 50  0000 C CNN
+F 2 "" H 2150 7450 50  0001 C CNN
+F 3 "" H 2150 7450 50  0001 C CNN
+	1    2150 7450
+	1    0    0    -1
+$EndComp
+$Comp
+L power:PWR_FLAG #FLG0608
+U 1 1 5DE65EAA
+P 2600 7450
+F 0 "#FLG0608" H 2600 7525 50  0001 C CNN
+F 1 "PWR_FLAG" H 2600 7623 50  0000 C CNN
+F 2 "" H 2600 7450 50  0001 C CNN
+F 3 "~" H 2600 7450 50  0001 C CNN
+	1    2600 7450
+	-1   0    0    1
+$EndComp
+$Comp
+L ETH1CPMU1:DGNDF #PWR0629
+U 1 1 5DE6634D
+P 2600 7450
+F 0 "#PWR0629" H 2600 7200 50  0001 C CNN
+F 1 "DGNDF" H 2605 7277 50  0000 C CNN
+F 2 "" H 2600 7450 50  0001 C CNN
+F 3 "" H 2600 7450 50  0001 C CNN
+	1    2600 7450
+	-1   0    0    1
+$EndComp
 $EndSCHEMATC
