File: hardware/project/ETH1CPMU1/Power_Float.sch (KiCad schematic (older format))
At the start: 58 parts, among them U601 THL15-2415WI, U602 LM1117IMP-3.3/NOPB, U603 MC7815BD2TG, U604 LM1117IMP-3.3/NOPB, U605 TSR2-2450, U606 LT8330_S6, U607 MC7915BD2TG, U608 LM1117IMP-5.0/NOPB, U609 TSR1-2490, U610 LT8330_S6

Commit message: PCB design.
Parts:
- removed FB601, FB602: 742792031, Inductor_SMD:L_0805_2012Metric_Pad1.15x1.40mm_HandSolder, symbol Device:Ferrite_Bead
- C627, C628: footprint Capacitor_SMD:C_0805_2012Metric_Pad1.15x1.40mm_HandSolder -> Capacitor_SMD:C_1206_3216Metric_Pad1.42x1.75mm_HandSolder
Connections:
- net +15VF: now also C618.1, U603.3 (OUT)
- net -15VF: now also C629.1, U607.3 (VO)
Changed lines of the file:
@@
 	5750 4700 5400 4700
 Connection ~ 5400 4700
-$Comp
-L Device:Ferrite_Bead FB601
-U 1 1 5DDB2389
-P 5950 3250
-F 0 "FB601" V 5676 3250 50  0000 C CNN
-F 1 "742792031" V 5767 3250 50  0000 C CNN
-F 2 "Inductor_SMD:L_0805_2012Metric_Pad1.15x1.40mm_HandSolder" V 5880 3250 50  0001 C CNN
-F 3 "~" H 5950 3250 50  0001 C CNN
-	1    5950 3250
-	0    1    1    0
-$EndComp
-Wire Wire Line
-	5800 3250 5750 3250
 Connection ~ 5750 3250
 $Comp
 L ETH1CPMU1:+15VF #PWR0610
 U 1 1 5DDB9470
-P 6250 3100
-F 0 "#PWR0610" H 6250 2950 50  0001 C CNN
-F 1 "+15VF" H 6265 3273 50  0000 C CNN
-F 2 "" H 6250 3100 50  0001 C CNN
-F 3 "" H 6250 3100 50  0001 C CNN
-	1    6250 3100
-	1    0    0    -1
-$EndComp
-Wire Wire Line
-	6250 3100 6250 3250
-Wire Wire Line
-	6250 3250 6100 3250
+P 5950 3100
+F 0 "#PWR0610" H 5950 2950 50  0001 C CNN
+F 1 "+15VF" H 5965 3273 50  0000 C CNN
+F 2 "" H 5950 3100 50  0001 C CNN
+F 3 "" H 5950 3100 50  0001 C CNN
+	1    5950 3100
+	1    0    0    -1
+$EndComp
+Wire Wire Line
+	5950 3100 5950 3250
 Connection ~ 2700 3250
 Wire Wire Line
@@
 F 0 "C627" H 4415 5896 50  0000 L CNN
 F 1 "2u2/50V" H 4415 5805 50  0000 L CNN
-F 2 "Capacitor_SMD:C_0805_2012Metric_Pad1.15x1.40mm_HandSolder" H 4338 5700 50  0001 C CNN
+F 2 "Capacitor_SMD:C_1206_3216Metric_Pad1.42x1.75mm_HandSolder" H 4338 5700 50  0001 C CNN
 F 3 "~" H 4300 5850 50  0001 C CNN
 	1    4300 5850
@@
 F 0 "C628" H 5015 5896 50  0000 L CNN
 F 1 "2u2/50V" H 5015 5805 50  0000 L CNN
-F 2 "Capacitor_SMD:C_0805_2012Metric_Pad1.15x1.40mm_HandSolder" H 4938 5700 50  0001 C CNN
+F 2 "Capacitor_SMD:C_1206_3216Metric_Pad1.42x1.75mm_HandSolder" H 4938 5700 50  0001 C CNN
 F 3 "~" H 4900 5850 50  0001 C CNN
 	1    4900 5850
@@
 	5750 6850 5400 6850
 Connection ~ 5400 6850
-$Comp
-L Device:Ferrite_Bead FB602
-U 1 1 5DE72108
-P 5950 5400
-F 0 "FB602" V 5676 5400 50  0000 C CNN
-F 1 "742792031" V 5767 5400 50  0000 C CNN
-F 2 "Inductor_SMD:L_0805_2012Metric_Pad1.15x1.40mm_HandSolder" V 5880 5400 50  0001 C CNN
-F 3 "~" H 5950 5400 50  0001 C CNN
-	1    5950 5400
-	0    1    1    0
-$EndComp
-Wire Wire Line
-	5800 5400 5750 5400
 Connection ~ 5750 5400
 Wire Wire Line
-	6250 5250 6250 5400
-Wire Wire Line
-	6250 5400 6100 5400
+	5950 5250 5950 5400
 Connection ~ 2700 5400
 Wire Wire Line
@@
 L ETH1CPMU1:-15VF #PWR0618
 U 1 1 5DF2FE99
-P 6250 5250
-F 0 "#PWR0618" H 6250 5100 50  0001 C CNN
-F 1 "-15VF" H 6265 5423 50  0000 C CNN
-F 2 "" H 6250 5250 50  0001 C CNN
-F 3 "" H 6250 5250 50  0001 C CNN
-	1    6250 5250
+P 5950 5250
+F 0 "#PWR0618" H 5950 5100 50  0001 C CNN
+F 1 "-15VF" H 5965 5423 50  0000 C CNN
+F 2 "" H 5950 5250 50  0001 C CNN
+F 3 "" H 5950 5250 50  0001 C CNN
+	1    5950 5250
 	1    0    0    -1
 $EndComp
@@
 	-1   0    0    1
 $EndComp
+Wire Wire Line
+	5750 3250 5950 3250
+Wire Wire Line
+	5750 5400 5950 5400
 $EndSCHEMATC

Commit message: PCB design
Changed lines of the file:
@@
 $EndComp
 $Comp
-L power:PWR_FLAG #FLG0606
-U 1 1 5DE489FC
+L power:PWR_FLAG #FLG0608
+U 1 1 5DE65EAA
 P 1700 7450
-F 0 "#FLG0606" H 1700 7525 50  0001 C CNN
+F 0 "#FLG0608" H 1700 7525 50  0001 C CNN
 F 1 "PWR_FLAG" H 1700 7623 50  0000 C CNN
 F 2 "" H 1700 7450 50  0001 C CNN
@@
 $EndComp
 $Comp
-L ETH1CPMU1:+15VF #PWR0627
-U 1 1 5DE48F13
+L ETH1CPMU1:DGNDF #PWR0629
+U 1 1 5DE6634D
 P 1700 7450
-F 0 "#PWR0627" H 1700 7300 50  0001 C CNN
-F 1 "+15VF" H 1715 7623 50  0000 C CNN
+F 0 "#PWR0629" H 1700 7200 50  0001 C CNN
+F 1 "DGNDF" H 1705 7277 50  0000 C CNN
 F 2 "" H 1700 7450 50  0001 C CNN
 F 3 "" H 1700 7450 50  0001 C CNN
 	1    1700 7450
-	1    0    0    -1
-$EndComp
-$Comp
-L power:PWR_FLAG #FLG0607
-U 1 1 5DE4A092
-P 2150 7450
-F 0 "#FLG0607" H 2150 7525 50  0001 C CNN
-F 1 "PWR_FLAG" H 2150 7623 50  0000 C CNN
-F 2 "" H 2150 7450 50  0001 C CNN
-F 3 "~" H 2150 7450 50  0001 C CNN
-	1    2150 7450
 	-1   0    0    1
 $EndComp
-$Comp
-L ETH1CPMU1:-15VF #PWR0628
-U 1 1 5DE5688B
-P 2150 7450
-F 0 "#PWR0628" H 2150 7300 50  0001 C CNN
-F 1 "-15VF" H 2165 7623 50  0000 C CNN
-F 2 "" H 2150 7450 50  0001 C CNN
-F 3 "" H 2150 7450 50  0001 C CNN
-	1    2150 7450
-	1    0    0    -1
-$EndComp
-$Comp
-L power:PWR_FLAG #FLG0608
-U 1 1 5DE65EAA
-P 2600 7450
-F 0 "#FLG0608" H 2600 7525 50  0001 C CNN
-F 1 "PWR_FLAG" H 2600 7623 50  0000 C CNN
-F 2 "" H 2600 7450 50  0001 C CNN
-F 3 "~" H 2600 7450 50  0001 C CNN
-	1    2600 7450
-	-1   0    0    1
-$EndComp
-$Comp
-L ETH1CPMU1:DGNDF #PWR0629
-U 1 1 5DE6634D
-P 2600 7450
-F 0 "#PWR0629" H 2600 7200 50  0001 C CNN
-F 1 "DGNDF" H 2605 7277 50  0000 C CNN
-F 2 "" H 2600 7450 50  0001 C CNN
-F 3 "" H 2600 7450 50  0001 C CNN
-	1    2600 7450
-	-1   0    0    1
-$EndComp

Commit message: PCB design
Parts:
- renumbered C602 to C601, C614 to C602, C625 to C603, C603 to C604, C619 to C605, C630 to C606, C620 to C608, C601 to C609, C606 to C610, C615 to C611, C626 to C612, C604 to C613, C616 to C614, C627 to C615, C617 to C616, C628 to C617, C629 to C619, C608 to C620, C609 to C621, C621 to C622, C610 to C623, C622 to C624, C611 to C625, C612 to C626, C623 to C627, C605 to C628, C613 to C629, C624 to C630, D602 to D601, D601 to D602, L604 to L603, L603 to L604, R603 to R602, R605 to R603, R607 to R604, R602 to R605, R604 to R606, R606 to R607, U606 to U601, U610 to U602, U601 to U603, U603 to U604, U607 to U605, U605 to U606, U609 to U607, U602 to U608, U604 to U609, U608 to U610
