File: hardware/project/ETH1CPMU1/DAC.sch (KiCad schematic (older format))
At the start: 0 parts

Commit message: Schematic design
Parts:
- added C1005, C1006, C1007: 100n, symbol Device:C
- added R1005, R1006, R1007, R1008, R1009, R1010, R1011: R, symbol Device:R
- added U1006: OPA2140, symbol ETH1CPMU1:OPA2140
- added U1007: DAC8563, symbol ETH1CPMU1:DAC8562T
Connections:
- net labels added: +15VF, +3.3VF, -15VF, AGNDF, DAC_DIN, DAC_SCLK, DAC_~CLR, DAC_~LDAC, DAC_~SYNC
- wire segments 0 -> 37

Commit message: Function generator schematic design.
Parts:
- C1005, C1006, C1007: footprint (none) -> Capacitor_SMD:C_0603_1608Metric_Pad1.05x0.95mm_HandSolder
Changed lines of the file:
@@
 $Descr A4 11693 8268
 encoding utf-8
-Sheet 9 14
+Sheet 9 15
 Title ""
 Date ""
@@
 F 0 "C1005" H 1715 7146 50  0000 L CNN
 F 1 "100n" H 1715 7055 50  0000 L CNN
-F 2 "" H 1638 6950 50  0001 C CNN
+F 2 "Capacitor_SMD:C_0603_1608Metric_Pad1.05x0.95mm_HandSolder" H 1638 6950 50  0001 C CNN
 F 3 "~" H 1600 7100 50  0001 C CNN
 	1    1600 7100
@@
 F 0 "C1006" H 2215 7146 50  0000 L CNN
 F 1 "100n" H 2215 7055 50  0000 L CNN
-F 2 "" H 2138 6950 50  0001 C CNN
+F 2 "Capacitor_SMD:C_0603_1608Metric_Pad1.05x0.95mm_HandSolder" H 2138 6950 50  0001 C CNN
 F 3 "~" H 2100 7100 50  0001 C CNN
 	1    2100 7100
@@
 F 0 "C1007" H 2765 7146 50  0000 L CNN
 F 1 "100n" H 2765 7055 50  0000 L CNN
-F 2 "" H 2688 6950 50  0001 C CNN
+F 2 "Capacitor_SMD:C_0603_1608Metric_Pad1.05x0.95mm_HandSolder" H 2688 6950 50  0001 C CNN
 F 3 "~" H 2650 7100 50  0001 C CNN
 	1    2650 7100

Commit message: Function generator schematic development.
Parts:
- R1005, R1006, R1007, R1008, R1009, R1010, R1011: footprint (none) -> Resistor_SMD:R_0603_1608Metric_Pad1.05x0.95mm_HandSolder
Changed lines of the file:
@@
 EESchema Schematic File Version 4
-LIBS:ETH1CPMU1-cache
 EELAYER 30 0
 EELAYER END
@@
 F 0 "R1007" V 5393 2950 50  0000 C CNN
 F 1 "R" V 5484 2950 50  0000 C CNN
-F 2 "" V 5530 2950 50  0001 C CNN
+F 2 "Resistor_SMD:R_0603_1608Metric_Pad1.05x0.95mm_HandSolder" V 5530 2950 50  0001 C CNN
 F 3 "~" H 5600 2950 50  0001 C CNN
 	1    5600 2950
@@
 F 0 "R1009" V 5393 3600 50  0000 C CNN
 F 1 "R" V 5484 3600 50  0000 C CNN
-F 2 "" V 5530 3600 50  0001 C CNN
+F 2 "Resistor_SMD:R_0603_1608Metric_Pad1.05x0.95mm_HandSolder" V 5530 3600 50  0001 C CNN
 F 3 "~" H 5600 3600 50  0001 C CNN
 	1    5600 3600
@@
 F 0 "R1008" H 6020 3196 50  0000 L CNN
 F 1 "R" H 6020 3105 50  0000 L CNN
-F 2 "" V 5880 3150 50  0001 C CNN
+F 2 "Resistor_SMD:R_0603_1608Metric_Pad1.05x0.95mm_HandSolder" V 5880 3150 50  0001 C CNN
 F 3 "~" H 5950 3150 50  0001 C CNN
 	1    5950 3150
@@
 F 0 "R1010" H 6020 3846 50  0000 L CNN
 F 1 "R" H 6020 3755 50  0000 L CNN
-F 2 "" V 5880 3800 50  0001 C CNN
+F 2 "Resistor_SMD:R_0603_1608Metric_Pad1.05x0.95mm_HandSolder" V 5880 3800 50  0001 C CNN
 F 3 "~" H 5950 3800 50  0001 C CNN
 	1    5950 3800
@@
 F 0 "R1006" V 6543 2150 50  0000 C CNN
 F 1 "R" V 6634 2150 50  0000 C CNN
-F 2 "" V 6680 2150 50  0001 C CNN
+F 2 "Resistor_SMD:R_0603_1608Metric_Pad1.05x0.95mm_HandSolder" V 6680 2150 50  0001 C CNN
 F 3 "~" H 6750 2150 50  0001 C CNN
 	1    6750 2150
@@
 F 0 "R1011" V 6543 4000 50  0000 C CNN
 F 1 "R" V 6634 4000 50  0000 C CNN
-F 2 "" V 6680 4000 50  0001 C CNN
+F 2 "Resistor_SMD:R_0603_1608Metric_Pad1.05x0.95mm_HandSolder" V 6680 4000 50  0001 C CNN
 F 3 "~" H 6750 4000 50  0001 C CNN
 	1    6750 4000
@@
 F 0 "R1005" V 4743 2150 50  0000 C CNN
 F 1 "R" V 4834 2150 50  0000 C CNN
-F 2 "" V 4880 2150 50  0001 C CNN
+F 2 "Resistor_SMD:R_0603_1608Metric_Pad1.05x0.95mm_HandSolder" V 4880 2150 50  0001 C CNN
 F 3 "~" H 4950 2150 50  0001 C CNN
 	1    4950 2150

Commit message: New footprint development, changes in schematics.
Parts:
- removed R1005, R1006, R1007, R1008, R1009, R1010, R1011: R, Resistor_SMD:R_0603_1608Metric_Pad1.05x0.95mm_HandSolder, symbol Device:R
- removed U1006: OPA2140, symbol ETH1CPMU1:OPA2140
- removed U1007: DAC8563, symbol ETH1CPMU1:DAC8562T
- added C901, C905: 220n, Capacitor_SMD:C_0603_1608Metric_Pad1.05x0.95mm_HandSolder, symbol Device:C
- added C902: 10u, Capacitor_SMD:C_0805_2012Metric_Pad1.15x1.40mm_HandSolder, symbol Device:C
- added C903: 1u, Capacitor_SMD:C_0603_1608Metric_Pad1.05x0.95mm_HandSolder, symbol Device:C
- added C904, C906: 1n, Capacitor_SMD:C_0603_1608Metric_Pad1.05x0.95mm_HandSolder, symbol Device:C
- added C907, C908: 100n, Capacitor_SMD:C_0603_1608Metric_Pad1.05x0.95mm_HandSolder, symbol Device:C
- added R901, R907: 1k, Resistor_SMD:R_0603_1608Metric_Pad1.05x0.95mm_HandSolder, symbol Device:R
- added R902, R909: 24k9, Resistor_SMD:R_0603_1608Metric_Pad1.05x0.95mm_HandSolder, symbol Device:R
- added R903, R910: 100k, Resistor_SMD:R_0603_1608Metric_Pad1.05x0.95mm_HandSolder, symbol Device:R
- added R904, R905: 10k, Resistor_SMD:R_0603_1608Metric_Pad1.05x0.95mm_HandSolder, symbol Device:R
- added R906, R913: 33k2, Resistor_SMD:R_0603_1608Metric_Pad1.05x0.95mm_HandSolder, symbol Device:R
- added R908, R911, R912: R, Resistor_SMD:R_0603_1608Metric_Pad1.05x0.95mm_HandSolder, symbol Device:R
- added U901: REF192, Package_SO:SSOP-8_3.9x5.05mm_P1.27mm, symbol Reference_Voltage:REF192
- added U902, U904: TL071, Package_SO:SOIC-8_3.9x4.9mm_P1.27mm, symbol Amplifier_Operational:TL071
- added U903: AD5689BRUZ, Package_SO:TSSOP-16_4.4x5mm_P0.65mm, symbol Analog_DAC:AD5689BRUZ
- renumbered C1005 to C909, C1006 to C910, C1007 to C911
Connections:
- net labels added: +2V5REF, +5VF, DAC_RSTSEL, DAC_SDIN, DAC_SDO, DAC_~RESET
- net labels removed: DAC_DIN, DAC_~CLR
- wire segments 37 -> 95
- no-connect marks 0 -> 4
Other:
- moved on the sheet: C909, C910, C911

Commit message: Schematic design
Parts:
- renumbered C901 to C1101, C902 to C1102, C903 to C1103, C904 to C1104, C905 to C1105, C906 to C1106, C907 to C1107, C908 to C1108, C909 to C1109, C910 to C1110, C911 to C1111, R901 to R1101, R902 to R1102, R903 to R1103, R904 to R1104, R905 to R1105, R906 to R1106, R907 to R1107, R908 to R1108, R909 to R1109, R910 to R1110, R911 to R1111, R912 to R1112, R913 to R1113, U901 to U1101, U902 to U1102, U903 to U1103, U904 to U1104
Connections:
- net PMU_CPH: now reaches C1104.1, R1103.1, U1102.6
- net PMU_CLH: now reaches C1106.1, R1110.1, U1104.6

Commit message: PCB design.
Parts:
- removed C1107, C1108: 100n, Capacitor_SMD:C_0603_1608Metric_Pad1.05x0.95mm_HandSolder, symbol Device:C
- removed U1102, U1104: TL071, Package_SO:SOIC-8_3.9x4.9mm_P1.27mm, symbol Amplifier_Operational:TL071
- added C1110: 100n, Capacitor_SMD:C_0603_1608Metric_Pad1.05x0.95mm_HandSolder, symbol Device:C
- added U1102: TL072, Package_SO:SOIC-8_3.9x4.9mm_P1.27mm, symbol Amplifier_Operational:TL072
- renumbered C1109 to C1107, C1110 to C1108, C1111 to C1109
Connections:
- net +15VF: now also U1102.8 (V+)
- net +5VF: now also C1110.1
- net -15VF: now also U1102.4 (V-)
- net AGNDF: now also C1110.2
- net PMU_CLH: now also U1102.7
- net PMU_CPH: now also U1102.1
- net at C1104.2, R1102.1, R1103.2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: now also U1102.2 (-)
- net at C1101.1, R1101.1: now also U1102.3 (+)
- net at C1106.2, R1109.1, R1110.2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: now also U1102.6 (-)
- net at C1105.1, R1107.1: now also U1102.5 (+)
- no-connect marks 4 -> 0
Other:
- moved on the sheet: C1107, C1108, C1109

Commit message: PCB design
Parts:
- removed C1110: 100n, Capacitor_SMD:C_0603_1608Metric_Pad1.05x0.95mm_HandSolder, symbol Device:C
- removed R1104, R1105: 10k, Resistor_SMD:R_0603_1608Metric_Pad1.05x0.95mm_HandSolder, symbol Device:R
- removed R1108, R1111, R1112: R, Resistor_SMD:R_0603_1608Metric_Pad1.05x0.95mm_HandSolder, symbol Device:R
- removed U1102: TL072, Package_SO:SOIC-8_3.9x4.9mm_P1.27mm, symbol Amplifier_Operational:TL072
- removed U1103: AD5689BRUZ, Package_SO:TSSOP-16_4.4x5mm_P0.65mm, symbol Analog_DAC:AD5689BRUZ
- added C1508, C1509: 220n, Capacitor_SMD:C_0603_1608Metric_Pad1.05x0.95mm_HandSolder, symbol Device:C
- added C1512, C1513: 1n, Capacitor_SMD:C_0603_1608Metric_Pad1.05x0.95mm_HandSolder, symbol Device:C
- added R1503, R1504: 1k, Resistor_SMD:R_0603_1608Metric_Pad1.05x0.95mm_HandSolder, symbol Device:R
- added R1509, R1511: 24k9, Resistor_SMD:R_0603_1608Metric_Pad1.05x0.95mm_HandSolder, symbol Device:R
- added R1510, R1512: 33k2, Resistor_SMD:R_0603_1608Metric_Pad1.05x0.95mm_HandSolder, symbol Device:R
- added R1515, R1516: 100k, Resistor_SMD:R_0603_1608Metric_Pad1.05x0.95mm_HandSolder, symbol Device:R
- added U1502: TL074, Package_SO:SOIC-14_3.9x8.7mm_P1.27mm, symbol Amplifier_Operational:TL074
- added U1503: AD5324, Package_SO:MSOP-10_3x3mm_P0.5mm, symbol ETH1CPMU1:AD5324
- renumbered C1107 to C1501, C1102 to C1502, C1108 to C1503, C1109 to C1504, C1103 to C1505, C1101 to C1506, C1105 to C1507, C1104 to C1510, C1106 to C1511, R1101 to R1501, R1107 to R1502, R1102 to R1505, R1106 to R1506, R1109 to R1507, R1113 to R1508, R1103 to R1513, R1110 to R1514, U1101 to U1501
Connections:
- net +15VF: now also U1502.4 (V+)
- net +2V5REF: now also R1509.2, R1511.2, U1503.5 (REFIN)
- net +3.3VF: now also U1503.1 (VDD)
- net -15VF: now also U1502.11 (V-)
- net AGNDF: now also C1508.2, C1509.2, R1510.2, R1512.2, U1503.7 (GND)
- net DAC_SCLK: now also U1503.9 (SCLK)
- net DAC_~SYNC: now also U1503.10 (~SYNC)
- net PMU_CLH: now also U1502.7
- net PMU_CPH: now also U1502.1
- net at R1501.2: now also U1503.2 (VOUTA)
- net at R1502.2: now also U1503.3 (VOUTB)
- net at C1511.2, R1507.1, R1508.1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: now also U1502.6 (-)
- net at C1507.1, R1502.1: now also U1502.5 (+)
- net at C1510.2, R1505.1, R1506.1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: now also U1502.2 (-)
- net at C1506.1, R1501.1: now also U1502.3 (+)
- new net: R1503.2, U1503.4 (VOUTC)
- new net: R1504.2, U1503.6 (VOUTD)
- new net: C1508.1, R1503.1, U1502.10 (+)
- new net: C1512.2, R1509.1, R1510.1, R1515.2, U1502.9 (-)
- new net: C1509.1, R1504.1, U1502.12 (+)
- new net: C1513.2, R1511.1, R1512.1, R1516.2, U1502.13 (-)
- new net DAC_DIN: U1503.8 (DIN)
- new net OFFSET1: C1512.1, R1515.1, U1502.8
- new net OFFSET2: C1513.1, R1516.1, U1502.14
Other:
- moved on the sheet: C1502, C1505, C1506, C1507, C1510, C1511, R1501, R1502, R1505, R1506, R1507, R1508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
