File: hardware/project/ETH1CPMU1/DAC.sch (KiCad schematic (older format))
At the start: 32 parts, among them U1501 REF192, U1502 TL074, U1503 AD5324

Commit message: PCB design
Connections:
- net +3.3VF renamed +3.3VP
Changed lines of the file:
@@
 Wire Wire Line
 	1850 7350 1850 7200
-$Comp
-L ETH1CPMU1:+3.3VF #PWR01507
-U 1 1 5EB96AA1
-P 1850 6750
-F 0 "#PWR01507" H 1850 6600 50  0001 C CNN
-F 1 "+3.3VF" H 1865 6923 50  0000 C CNN
-F 2 "" H 1850 6750 50  0001 C CNN
-F 3 "" H 1850 6750 50  0001 C CNN
-	1    1850 6750
-	1    0    0    -1
-$EndComp
 Wire Wire Line
 	3300 2100 3300 2050
@@
 Text Label 2550 3300 2    50   ~ 0
 +2V5REF
-$Comp
-L ETH1CPMU1:+3.3VF #PWR01511
-U 1 1 5E5BE512
-P 3300 2050
-F 0 "#PWR01511" H 3300 1900 50  0001 C CNN
-F 1 "+3.3VF" H 3315 2223 50  0000 C CNN
-F 2 "" H 3300 2050 50  0001 C CNN
-F 3 "" H 3300 2050 50  0001 C CNN
-	1    3300 2050
-	1    0    0    -1
-$EndComp
 Text HLabel 6950 2600 2    50   Output ~ 0
 PMU_CLH
@@
 Wire Wire Line
 	900  3700 1600 3700
+$Comp
+L power:+3.3VP #PWR0112
+U 1 1 5E0D6265
+P 1850 6750
+F 0 "#PWR0112" H 2000 6700 50  0001 C CNN
+F 1 "+3.3VP" H 1870 6893 50  0000 C CNN
+F 2 "" H 1850 6750 50  0001 C CNN
+F 3 "" H 1850 6750 50  0001 C CNN
+	1    1850 6750
+	1    0    0    -1
+$EndComp
+$Comp
+L power:+3.3VP #PWR0113
+U 1 1 5E0D675D
+P 3300 2050
+F 0 "#PWR0113" H 3450 2000 50  0001 C CNN
+F 1 "+3.3VP" H 3320 2193 50  0000 C CNN
+F 2 "" H 3300 2050 50  0001 C CNN
+F 3 "" H 3300 2050 50  0001 C CNN
+	1    3300 2050
+	1    0    0    -1
+$EndComp
 $EndSCHEMATC
