File: hardware/project/ETH1CPMU1/DC_Source.sch (KiCad schematic (older format))
At the start: 36 parts, among them U901 AD8676, U902 AD8676, U903 AD8675, U904 AD5791, U905 REF02AU

Commit message: Schematic design
Connections:
- net +15VF: now also C910.1
- net AGNDF: now also C910.2
Other:
- moved on the sheet: C910
Changed lines of the file:
@@
 $Descr A4 11693 8268
 encoding utf-8
-Sheet 9 14
+Sheet 8 14
 Title ""
 Date ""
@@
 	4200 3450 4250 3450
 Wire Wire Line
-	750  6100 750  6050
-Wire Wire Line
-	750  6400 750  6450
+	750  6000 750  5950
+Wire Wire Line
+	750  6300 750  6350
 $Comp
 L ETH1CPMU1:-15VF #PWR0916
@@
 L Device:C C910
 U 1 1 5DFDE3EA
-P 750 6250
-F 0 "C910" H 865 6296 50  0000 L CNN
-F 1 "10u" H 865 6205 50  0000 L CNN
-F 2 "" H 788 6100 50  0001 C CNN
-F 3 "~" H 750 6250 50  0001 C CNN
-	1    750  6250
+P 750 6150
+F 0 "C910" H 865 6196 50  0000 L CNN
+F 1 "10u" H 865 6105 50  0000 L CNN
+F 2 "" H 788 6000 50  0001 C CNN
+F 3 "~" H 750 6150 50  0001 C CNN
+	1    750  6150
 	1    0    0    -1
 $EndComp
@@
 Wire Wire Line
 	5200 7450 5450 7450
-NoConn ~ 1900 1700
+NoConn ~ 2150 1700
 $Comp
 L Device:R_POT_TRIM RV901

Commit message: Function generator schematic design.
Parts:
- C901, C904, C906, C908, C910, C911, C913, C915, C917, C919, C921: footprint (none) -> Capacitor_SMD:C_1206_3216Metric_Pad1.42x1.75mm_HandSolder
- C902, C903, C905, C907, C909, C912, C914, C916, C918, C920, C922: footprint (none) -> Capacitor_SMD:C_0603_1608Metric_Pad1.05x0.95mm_HandSolder
- RV901: footprint (none) -> Resistor_SMD:R_0603_1608Metric_Pad1.05x0.95mm_HandSolder
Changed lines of the file:
@@
 $Descr A4 11693 8268
 encoding utf-8
-Sheet 8 14
+Sheet 7 15
 Title ""
 Date ""
@@
 F 0 "C911" H 865 7296 50  0000 L CNN
 F 1 "10u" H 865 7205 50  0000 L CNN
-F 2 "" H 788 7100 50  0001 C CNN
+F 2 "Capacitor_SMD:C_1206_3216Metric_Pad1.42x1.75mm_HandSolder" H 788 7100 50  0001 C CNN
 F 3 "~" H 750 7250 50  0001 C CNN
 	1    750  7250
@@
 F 0 "C912" H 1365 7296 50  0000 L CNN
 F 1 "100n" H 1365 7205 50  0000 L CNN
-F 2 "" H 1288 7100 50  0001 C CNN
+F 2 "Capacitor_SMD:C_0603_1608Metric_Pad1.05x0.95mm_HandSolder" H 1288 7100 50  0001 C CNN
 F 3 "~" H 1250 7250 50  0001 C CNN
 	1    1250 7250
@@
 F 0 "C913" H 1915 7296 50  0000 L CNN
 F 1 "10u" H 1915 7205 50  0000 L CNN
-F 2 "" H 1838 7100 50  0001 C CNN
+F 2 "Capacitor_SMD:C_1206_3216Metric_Pad1.42x1.75mm_HandSolder" H 1838 7100 50  0001 C CNN
 F 3 "~" H 1800 7250 50  0001 C CNN
 	1    1800 7250
@@
 F 0 "C914" H 2415 7296 50  0000 L CNN
 F 1 "100n" H 2415 7205 50  0000 L CNN
-F 2 "" H 2338 7100 50  0001 C CNN
+F 2 "Capacitor_SMD:C_0603_1608Metric_Pad1.05x0.95mm_HandSolder" H 2338 7100 50  0001 C CNN
 F 3 "~" H 2300 7250 50  0001 C CNN
 	1    2300 7250
@@
 F 0 "C919" H 6115 7296 50  0000 L CNN
 F 1 "10u" H 6115 7205 50  0000 L CNN
-F 2 "" H 6038 7100 50  0001 C CNN
+F 2 "Capacitor_SMD:C_1206_3216Metric_Pad1.42x1.75mm_HandSolder" H 6038 7100 50  0001 C CNN
 F 3 "~" H 6000 7250 50  0001 C CNN
 	1    6000 7250
@@
 F 0 "C920" H 6615 7296 50  0000 L CNN
 F 1 "100n" H 6615 7205 50  0000 L CNN
-F 2 "" H 6538 7100 50  0001 C CNN
+F 2 "Capacitor_SMD:C_0603_1608Metric_Pad1.05x0.95mm_HandSolder" H 6538 7100 50  0001 C CNN
 F 3 "~" H 6500 7250 50  0001 C CNN
 	1    6500 7250
@@
 F 0 "C902" H 4765 3696 50  0000 L CNN
 F 1 "100n" H 4765 3605 50  0000 L CNN
-F 2 "" H 4688 3500 50  0001 C CNN
+F 2 "Capacitor_SMD:C_0603_1608Metric_Pad1.05x0.95mm_HandSolder" H 4688 3500 50  0001 C CNN
 F 3 "~" H 4650 3650 50  0001 C CNN
 	1    4650 3650
@@
 F 0 "C905" H 2415 6196 50  0000 L CNN
 F 1 "100n" H 2415 6105 50  0000 L CNN
-F 2 "" H 2338 6000 50  0001 C CNN
+F 2 "Capacitor_SMD:C_0603_1608Metric_Pad1.05x0.95mm_HandSolder" H 2338 6000 50  0001 C CNN
 F 3 "~" H 2300 6150 50  0001 C CNN
 	1    2300 6150
@@
 F 0 "C904" H 1915 6196 50  0000 L CNN
 F 1 "10u" H 1915 6105 50  0000 L CNN
-F 2 "" H 1838 6000 50  0001 C CNN
+F 2 "Capacitor_SMD:C_1206_3216Metric_Pad1.42x1.75mm_HandSolder" H 1838 6000 50  0001 C CNN
 F 3 "~" H 1800 6150 50  0001 C CNN
 	1    1800 6150
@@
 F 0 "C903" H 1365 6196 50  0000 L CNN
 F 1 "100n" H 1365 6105 50  0000 L CNN
-F 2 "" H 1288 6000 50  0001 C CNN
+F 2 "Capacitor_SMD:C_0603_1608Metric_Pad1.05x0.95mm_HandSolder" H 1288 6000 50  0001 C CNN
 F 3 "~" H 1250 6150 50  0001 C CNN
 	1    1250 6150
@@
 F 0 "C910" H 865 6196 50  0000 L CNN
 F 1 "10u" H 865 6105 50  0000 L CNN
-F 2 "" H 788 6000 50  0001 C CNN
+F 2 "Capacitor_SMD:C_1206_3216Metric_Pad1.42x1.75mm_HandSolder" H 788 6000 50  0001 C CNN
 F 3 "~" H 750 6150 50  0001 C CNN
 	1    750  6150
@@
 F 0 "C915" H 2965 7296 50  0000 L CNN
 F 1 "10u" H 2965 7205 50  0000 L CNN
-F 2 "" H 2888 7100 50  0001 C CNN
+F 2 "Capacitor_SMD:C_1206_3216Metric_Pad1.42x1.75mm_HandSolder" H 2888 7100 50  0001 C CNN
 F 3 "~" H 2850 7250 50  0001 C CNN
 	1    2850 7250
@@
 F 0 "C916" H 3465 7296 50  0000 L CNN
 F 1 "100n" H 3465 7205 50  0000 L CNN
-F 2 "" H 3388 7100 50  0001 C CNN
+F 2 "Capacitor_SMD:C_0603_1608Metric_Pad1.05x0.95mm_HandSolder" H 3388 7100 50  0001 C CNN
 F 3 "~" H 3350 7250 50  0001 C CNN
 	1    3350 7250
@@
 F 0 "C917" H 4015 7296 50  0000 L CNN
 F 1 "10u" H 4015 7205 50  0000 L CNN
-F 2 "" H 3938 7100 50  0001 C CNN
+F 2 "Capacitor_SMD:C_1206_3216Metric_Pad1.42x1.75mm_HandSolder" H 3938 7100 50  0001 C CNN
 F 3 "~" H 3900 7250 50  0001 C CNN
 	1    3900 7250
@@
 F 0 "C918" H 4515 7296 50  0000 L CNN
 F 1 "100n" H 4515 7205 50  0000 L CNN
-F 2 "" H 4438 7100 50  0001 C CNN
+F 2 "Capacitor_SMD:C_0603_1608Metric_Pad1.05x0.95mm_HandSolder" H 4438 7100 50  0001 C CNN
 F 3 "~" H 4400 7250 50  0001 C CNN
 	1    4400 7250
@@
 F 0 "C909" H 4515 6196 50  0000 L CNN
 F 1 "100n" H 4515 6105 50  0000 L CNN
-F 2 "" H 4438 6000 50  0001 C CNN
+F 2 "Capacitor_SMD:C_0603_1608Metric_Pad1.05x0.95mm_HandSolder" H 4438 6000 50  0001 C CNN
 F 3 "~" H 4400 6150 50  0001 C CNN
 	1    4400 6150
@@
 F 0 "C908" H 4015 6196 50  0000 L CNN
 F 1 "10u" H 4015 6105 50  0000 L CNN
-F 2 "" H 3938 6000 50  0001 C CNN
+F 2 "Capacitor_SMD:C_1206_3216Metric_Pad1.42x1.75mm_HandSolder" H 3938 6000 50  0001 C CNN
 F 3 "~" H 3900 6150 50  0001 C CNN
 	1    3900 6150
@@
 F 0 "C907" H 3465 6196 50  0000 L CNN
 F 1 "100n" H 3465 6105 50  0000 L CNN
-F 2 "" H 3388 6000 50  0001 C CNN
+F 2 "Capacitor_SMD:C_0603_1608Metric_Pad1.05x0.95mm_HandSolder" H 3388 6000 50  0001 C CNN
 F 3 "~" H 3350 6150 50  0001 C CNN
 	1    3350 6150
@@
 F 0 "C906" H 2965 6196 50  0000 L CNN
 F 1 "10u" H 2965 6105 50  0000 L CNN
-F 2 "" H 2888 6000 50  0001 C CNN
+F 2 "Capacitor_SMD:C_1206_3216Metric_Pad1.42x1.75mm_HandSolder" H 2888 6000 50  0001 C CNN
 F 3 "~" H 2850 6150 50  0001 C CNN
 	1    2850 6150
@@
 F 0 "C901" H 4715 1846 50  0000 L CNN
 F 1 "10u" H 4715 1755 50  0000 L CNN
-F 2 "" H 4638 1650 50  0001 C CNN
+F 2 "Capacitor_SMD:C_1206_3216Metric_Pad1.42x1.75mm_HandSolder" H 4638 1650 50  0001 C CNN
 F 3 "~" H 4600 1800 50  0001 C CNN
 	1    4600 1800
@@
 F 0 "C921" H 5065 7296 50  0000 L CNN
 F 1 "10u" H 5065 7205 50  0000 L CNN
-F 2 "" H 4988 7100 50  0001 C CNN
+F 2 "Capacitor_SMD:C_1206_3216Metric_Pad1.42x1.75mm_HandSolder" H 4988 7100 50  0001 C CNN
 F 3 "~" H 4950 7250 50  0001 C CNN
 	1    4950 7250
@@
 F 0 "C922" H 5565 7296 50  0000 L CNN
 F 1 "100n" H 5565 7205 50  0000 L CNN
-F 2 "" H 5488 7100 50  0001 C CNN
+F 2 "Capacitor_SMD:C_0603_1608Metric_Pad1.05x0.95mm_HandSolder" H 5488 7100 50  0001 C CNN
 F 3 "~" H 5450 7250 50  0001 C CNN
 	1    5450 7250
@@
 F 0 "RV901" H 2980 1846 50  0000 R CNN
 F 1 "10k" H 2980 1755 50  0000 R CNN
-F 2 "" H 3050 1800 50  0001 C CNN
+F 2 "Resistor_SMD:R_0603_1608Metric_Pad1.05x0.95mm_HandSolder" H 3050 1800 50  0001 C CNN
 F 3 "~" H 3050 1800 50  0001 C CNN
 	1    3050 1800

Commit message: Function generator schematic development.
Parts:
- R904, R905: footprint (none) -> Resistor_SMD:R_0603_1608Metric_Pad1.05x0.95mm_HandSolder
Changed lines of the file:
@@
 EESchema Schematic File Version 4
-LIBS:ETH1CPMU1-cache
 EELAYER 30 0
 EELAYER END
@@
 F 0 "R904" H 4720 3296 50  0000 L CNN
 F 1 "10k" H 4720 3205 50  0000 L CNN
-F 2 "" V 4580 3250 50  0001 C CNN
+F 2 "Resistor_SMD:R_0603_1608Metric_Pad1.05x0.95mm_HandSolder" V 4580 3250 50  0001 C CNN
 F 3 "~" H 4650 3250 50  0001 C CNN
 	1    4650 3250
@@
 F 0 "R905" V 4193 3450 50  0000 C CNN
 F 1 "0" V 4284 3450 50  0000 C CNN
-F 2 "" V 4330 3450 50  0001 C CNN
+F 2 "Resistor_SMD:R_0603_1608Metric_Pad1.05x0.95mm_HandSolder" V 4330 3450 50  0001 C CNN
 F 3 "~" H 4400 3450 50  0001 C CNN
 	1    4400 3450

Commit message: New footprint development, changes in schematics.
Parts:
- R701: renamed from R901; footprint (none) -> Resistor_SMD:R_0805_2012Metric_Pad1.15x1.40mm_HandSolder
- R702: renamed from R902; footprint (none) -> Resistor_SMD:R_0805_2012Metric_Pad1.15x1.40mm_HandSolder
- R703: renamed from R903; footprint (none) -> Resistor_SMD:R_0805_2012Metric_Pad1.15x1.40mm_HandSolder
- R706: renamed from R906; footprint (none) -> Resistor_SMD:R_0805_2012Metric_Pad1.15x1.40mm_HandSolder
- R707: renamed from R907; footprint (none) -> Resistor_SMD:R_0805_2012Metric_Pad1.15x1.40mm_HandSolder
- U702: renamed from U901; footprint (none) -> Package_SO:SOIC-8_3.9x4.9mm_P1.27mm
- U703: renamed from U902; footprint (none) -> Package_SO:SOIC-8_3.9x4.9mm_P1.27mm
- U704: renamed from U903; footprint (none) -> Package_SO:SOIC-8_3.9x4.9mm_P1.27mm
- U705: renamed from U904; footprint (none) -> Package_SO:TSSOP-20_4.4x6.5mm_P0.65mm
- renumbered C901 to C701, C902 to C702, C910 to C703, C903 to C704, C904 to C705, C905 to C706, C906 to C707, C907 to C708, C908 to C709, C909 to C710, C911 to C711, C912 to C712, C913 to C713, C914 to C714, C915 to C715, C916 to C716, C917 to C717, C918 to C718, C921 to C719, C922 to C720, C919 to C721, C920 to C722, R904 to R704, R905 to R705, RV901 to RV701, TP901 to TP701, U905 to U701

Commit message: Schematic and PCB design.
Parts:
- RV701: value 10k -> 3314J-1-103E; footprint Resistor_SMD:R_0603_1608Metric_Pad1.05x0.95mm_HandSolder -> Potentiometer_SMD:Potentiometer_Bourns_3314J_Vertical
- TP701: value TestPoint -> 5006; footprint (none) -> TestPoint:TestPoint_Loop_D2.60mm_Drill1.6mm_Beaded
Other:
- moved on the sheet: RV701, TP701, U701
Changed lines of the file:
@@
 	1    0    0    -1
 $EndComp
-Wire Wire Line
-	8550 3050 8850 3050
 Connection ~ 8550 3050
-Text HLabel 8850 3050 2    50   Output ~ 0
+Text HLabel 9000 3050 2    50   Output ~ 0
 DC_FOURCE
 Wire Wire Line
@@
 L Reference_Voltage:REF02AU U701
 U 1 1 5E1B845C
-P 2450 1700
-F 0 "U701" H 2700 2100 50  0000 C CNN
-F 1 "REF02AU" H 2700 2000 50  0000 C CNN
-F 2 "Package_SO:SOIC-8_3.9x4.9mm_P1.27mm" H 2400 1750 50  0001 C CIN
-F 3 "http://www.ti.com/lit/ds/symlink/ref02.pdf" H 2400 1700 50  0001 C CIN
-	1    2450 1700
-	1    0    0    -1
-$EndComp
-Connection ~ 3550 1600
+P 2250 1700
+F 0 "U701" H 2500 2100 50  0000 C CNN
+F 1 "REF02AU" H 2500 2000 50  0000 C CNN
+F 2 "Package_SO:SOIC-8_3.9x4.9mm_P1.27mm" H 2200 1750 50  0001 C CIN
+F 3 "http://www.ti.com/lit/ds/symlink/ref02.pdf" H 2200 1700 50  0001 C CIN
+	1    2250 1700
+	1    0    0    -1
+$EndComp
 $Comp
 L ETH1CPMU1:AGNDF #PWR0703
 U 1 1 5E1C1B35
-P 2450 2050
-F 0 "#PWR0703" H 2450 1800 50  0001 C CNN
-F 1 "AGNDF" H 2455 1877 50  0000 C CNN
-F 2 "" H 2450 2050 50  0001 C CNN
-F 3 "" H 2450 2050 50  0001 C CNN
-	1    2450 2050
-	1    0    0    -1
-$EndComp
-Wire Wire Line
-	2450 2050 2450 2000
+P 2250 2050
+F 0 "#PWR0703" H 2250 1800 50  0001 C CNN
+F 1 "AGNDF" H 2255 1877 50  0000 C CNN
+F 2 "" H 2250 2050 50  0001 C CNN
+F 3 "" H 2250 2050 50  0001 C CNN
+	1    2250 2050
+	1    0    0    -1
+$EndComp
+Wire Wire Line
+	2250 2050 2250 2000
 $Comp
 L ETH1CPMU1:+15VF #PWR0701
 U 1 1 5E1CDFAF
-P 2450 1350
-F 0 "#PWR0701" H 2450 1200 50  0001 C CNN
-F 1 "+15VF" H 2465 1523 50  0000 C CNN
-F 2 "" H 2450 1350 50  0001 C CNN
-F 3 "" H 2450 1350 50  0001 C CNN
-	1    2450 1350
-	1    0    0    -1
-$EndComp
-Wire Wire Line
-	2450 1350 2450 1400
+P 2250 1350
+F 0 "#PWR0701" H 2250 1200 50  0001 C CNN
+F 1 "+15VF" H 2265 1523 50  0000 C CNN
+F 2 "" H 2250 1350 50  0001 C CNN
+F 3 "" H 2250 1350 50  0001 C CNN
+	1    2250 1350
+	1    0    0    -1
+$EndComp
+Wire Wire Line
+	2250 1350 2250 1400
 $Comp
 L ETH1CPMU1:+15VF #PWR0732
@@
 Wire Wire Line
 	5200 7450 5450 7450
-NoConn ~ 2150 1700
+NoConn ~ 1950 1700
 $Comp
 L Device:R_POT_TRIM RV701
 U 1 1 5E236BDD
-P 3050 1800
-F 0 "RV701" H 2980 1846 50  0000 R CNN
-F 1 "10k" H 2980 1755 50  0000 R CNN
-F 2 "Resistor_SMD:R_0603_1608Metric_Pad1.05x0.95mm_HandSolder" H 3050 1800 50  0001 C CNN
-F 3 "~" H 3050 1800 50  0001 C CNN
-	1    3050 1800
+P 2850 1800
+F 0 "RV701" H 2780 1846 50  0000 R CNN
+F 1 "3314J-1-103E" H 2780 1755 50  0000 R CNN
+F 2 "Potentiometer_SMD:Potentiometer_Bourns_3314J_Vertical" H 2850 1800 50  0001 C CNN
+F 3 "~" H 2850 1800 50  0001 C CNN
+	1    2850 1800
 	-1   0    0    -1
 $EndComp
@@
 L ETH1CPMU1:AGNDF #PWR0704
 U 1 1 5E242161
-P 3050 2050
-F 0 "#PWR0704" H 3050 1800 50  0001 C CNN
-F 1 "AGNDF" H 3055 1877 50  0000 C CNN
-F 2 "" H 3050 2050 50  0001 C CNN
-F 3 "" H 3050 2050 50  0001 C CNN
-	1    3050 2050
-	1    0    0    -1
-$EndComp
-Wire Wire Line
-	2900 1800 2850 1800
-Wire Wire Line
-	3050 2050 3050 1950
-Wire Wire Line
-	2850 1600 3050 1600
-Wire Wire Line
-	3050 1600 3050 1650
-Connection ~ 3050 1600
-Wire Wire Line
-	3050 1600 3550 1600
+P 2850 2050
+F 0 "#PWR0704" H 2850 1800 50  0001 C CNN
+F 1 "AGNDF" H 2855 1877 50  0000 C CNN
+F 2 "" H 2850 2050 50  0001 C CNN
+F 3 "" H 2850 2050 50  0001 C CNN
+	1    2850 2050
+	1    0    0    -1
+$EndComp
+Wire Wire Line
+	2700 1800 2650 1800
+Wire Wire Line
+	2850 2050 2850 1950
+Wire Wire Line
+	2650 1600 2850 1600
+Wire Wire Line
+	2850 1600 2850 1650
+Connection ~ 2850 1600
 $Comp
 L Connector:TestPoint TP701
 U 1 1 5E276B52
-P 3050 1550
-F 0 "TP701" H 3108 1668 50  0000 L CNN
-F 1 "TestPoint" H 3108 1577 50  0000 L CNN
-F 2 "" H 3250 1550 50  0001 C CNN
-F 3 "~" H 3250 1550 50  0001 C CNN
-	1    3050 1550
-	1    0    0    -1
-$EndComp
-Wire Wire Line
-	3050 1550 3050 1600
+P 2850 1550
+F 0 "TP701" H 2908 1668 50  0000 L CNN
+F 1 "5006" H 2908 1577 50  0000 L CNN
+F 2 "TestPoint:TestPoint_Loop_D2.60mm_Drill1.6mm_Beaded" H 3050 1550 50  0001 C CNN
+F 3 "~" H 3050 1550 50  0001 C CNN
+	1    2850 1550
+	1    0    0    -1
+$EndComp
+Wire Wire Line
+	2850 1550 2850 1600
+Wire Wire Line
+	2850 1600 3550 1600
+Connection ~ 3550 1600
+Wire Wire Line
+	8550 3050 9000 3050
 $EndSCHEMATC

Commit message: PCB design.
Parts:
- C703, C705, C707, C709, C711, C713, C715, C717, C719, C721: footprint Capacitor_SMD:C_1206_3216Metric_Pad1.42x1.75mm_HandSolder -> Capacitor_SMD:C_0805_2012Metric_Pad1.15x1.40mm_HandSolder
Changed lines of the file:
@@
 F 0 "C711" H 865 7296 50  0000 L CNN
 F 1 "10u" H 865 7205 50  0000 L CNN
-F 2 "Capacitor_SMD:C_1206_3216Metric_Pad1.42x1.75mm_HandSolder" H 788 7100 50  0001 C CNN
+F 2 "Capacitor_SMD:C_0805_2012Metric_Pad1.15x1.40mm_HandSolder" H 788 7100 50  0001 C CNN
 F 3 "~" H 750 7250 50  0001 C CNN
 	1    750  7250
@@
 F 0 "C713" H 1915 7296 50  0000 L CNN
 F 1 "10u" H 1915 7205 50  0000 L CNN
-F 2 "Capacitor_SMD:C_1206_3216Metric_Pad1.42x1.75mm_HandSolder" H 1838 7100 50  0001 C CNN
+F 2 "Capacitor_SMD:C_0805_2012Metric_Pad1.15x1.40mm_HandSolder" H 1838 7100 50  0001 C CNN
 F 3 "~" H 1800 7250 50  0001 C CNN
 	1    1800 7250
@@
 F 0 "C721" H 6115 7296 50  0000 L CNN
 F 1 "10u" H 6115 7205 50  0000 L CNN
-F 2 "Capacitor_SMD:C_1206_3216Metric_Pad1.42x1.75mm_HandSolder" H 6038 7100 50  0001 C CNN
+F 2 "Capacitor_SMD:C_0805_2012Metric_Pad1.15x1.40mm_HandSolder" H 6038 7100 50  0001 C CNN
 F 3 "~" H 6000 7250 50  0001 C CNN
 	1    6000 7250
@@
 F 0 "C705" H 1915 6196 50  0000 L CNN
 F 1 "10u" H 1915 6105 50  0000 L CNN
-F 2 "Capacitor_SMD:C_1206_3216Metric_Pad1.42x1.75mm_HandSolder" H 1838 6000 50  0001 C CNN
+F 2 "Capacitor_SMD:C_0805_2012Metric_Pad1.15x1.40mm_HandSolder" H 1838 6000 50  0001 C CNN
 F 3 "~" H 1800 6150 50  0001 C CNN
 	1    1800 6150
@@
 F 0 "C703" H 865 6196 50  0000 L CNN
 F 1 "10u" H 865 6105 50  0000 L CNN
-F 2 "Capacitor_SMD:C_1206_3216Metric_Pad1.42x1.75mm_HandSolder" H 788 6000 50  0001 C CNN
+F 2 "Capacitor_SMD:C_0805_2012Metric_Pad1.15x1.40mm_HandSolder" H 788 6000 50  0001 C CNN
 F 3 "~" H 750 6150 50  0001 C CNN
 	1    750  6150
@@
 F 0 "C715" H 2965 7296 50  0000 L CNN
 F 1 "10u" H 2965 7205 50  0000 L CNN
-F 2 "Capacitor_SMD:C_1206_3216Metric_Pad1.42x1.75mm_HandSolder" H 2888 7100 50  0001 C CNN
+F 2 "Capacitor_SMD:C_0805_2012Metric_Pad1.15x1.40mm_HandSolder" H 2888 7100 50  0001 C CNN
 F 3 "~" H 2850 7250 50  0001 C CNN
 	1    2850 7250
@@
 F 0 "C717" H 4015 7296 50  0000 L CNN
 F 1 "10u" H 4015 7205 50  0000 L CNN
-F 2 "Capacitor_SMD:C_1206_3216Metric_Pad1.42x1.75mm_HandSolder" H 3938 7100 50  0001 C CNN
+F 2 "Capacitor_SMD:C_0805_2012Metric_Pad1.15x1.40mm_HandSolder" H 3938 7100 50  0001 C CNN
 F 3 "~" H 3900 7250 50  0001 C CNN
 	1    3900 7250
@@
 F 0 "C709" H 4015 6196 50  0000 L CNN
 F 1 "10u" H 4015 6105 50  0000 L CNN
-F 2 "Capacitor_SMD:C_1206_3216Metric_Pad1.42x1.75mm_HandSolder" H 3938 6000 50  0001 C CNN
+F 2 "Capacitor_SMD:C_0805_2012Metric_Pad1.15x1.40mm_HandSolder" H 3938 6000 50  0001 C CNN
 F 3 "~" H 3900 6150 50  0001 C CNN
 	1    3900 6150
@@
 F 0 "C707" H 2965 6196 50  0000 L CNN
 F 1 "10u" H 2965 6105 50  0000 L CNN
-F 2 "Capacitor_SMD:C_1206_3216Metric_Pad1.42x1.75mm_HandSolder" H 2888 6000 50  0001 C CNN
+F 2 "Capacitor_SMD:C_0805_2012Metric_Pad1.15x1.40mm_HandSolder" H 2888 6000 50  0001 C CNN
 F 3 "~" H 2850 6150 50  0001 C CNN
 	1    2850 6150
@@
 F 0 "C719" H 5065 7296 50  0000 L CNN
 F 1 "10u" H 5065 7205 50  0000 L CNN
-F 2 "Capacitor_SMD:C_1206_3216Metric_Pad1.42x1.75mm_HandSolder" H 4988 7100 50  0001 C CNN
+F 2 "Capacitor_SMD:C_0805_2012Metric_Pad1.15x1.40mm_HandSolder" H 4988 7100 50  0001 C CNN
 F 3 "~" H 4950 7250 50  0001 C CNN
 	1    4950 7250

Commit message: PCB design
Parts:
- renumbered C703 to C701, C711 to C702, C704 to C703, C712 to C704, C713 to C706, C706 to C707, C714 to C708, C707 to C709, C715 to C710, C708 to C711, C716 to C712, C709 to C713, C717 to C714, C710 to C715, C718 to C716, C701 to C717, C702 to C718, R707 to R702, R705 to R703, R703 to R705, R702 to R707, U703 to U702, U702 to U703, U705 to U704, U704 to U705
