File: hardware/project/ETH1CPMU1/DC_Source.sch (KiCad schematic (older format))
At the start: 36 parts, among them U701 REF02AU, U702 AD8676, U703 AD8676, U704 AD5791, U705 AD8675

Commit message: PCB design
Connections:
- net +3.3VF renamed +3.3VP
Changed lines of the file:
@@
 Wire Wire Line
 	5900 3700 5900 3750
-$Comp
-L ETH1CPMU1:+3.3VF #PWR0730
-U 1 1 5DF97F26
-P 6050 2550
-F 0 "#PWR0730" H 6050 2400 50  0001 C CNN
-F 1 "+3.3VF" H 6065 2723 50  0000 C CNN
-F 2 "" H 6050 2550 50  0001 C CNN
-F 3 "" H 6050 2550 50  0001 C CNN
-	1    6050 2550
-	1    0    0    -1
-$EndComp
 Wire Wire Line
 	6050 2550 6050 2600
@@
 F 3 "" H 6250 7500 50  0001 C CNN
 	1    6250 7500
-	1    0    0    -1
-$EndComp
-$Comp
-L ETH1CPMU1:+3.3VF #PWR0734
-U 1 1 5DFAA283
-P 6250 7000
-F 0 "#PWR0734" H 6250 6850 50  0001 C CNN
-F 1 "+3.3VF" H 6265 7173 50  0000 C CNN
-F 2 "" H 6250 7000 50  0001 C CNN
-F 3 "" H 6250 7000 50  0001 C CNN
-	1    6250 7000
 	1    0    0    -1
 $EndComp
@@
 	1    0    0    -1
 $EndComp
-$Comp
-L ETH1CPMU1:+3.3VF #PWR0721
-U 1 1 5DFCB46A
-P 4650 3050
-F 0 "#PWR0721" H 4650 2900 50  0001 C CNN
-F 1 "+3.3VF" H 4665 3223 50  0000 C CNN
-F 2 "" H 4650 3050 50  0001 C CNN
-F 3 "" H 4650 3050 50  0001 C CNN
-	1    4650 3050
-	1    0    0    -1
-$EndComp
 Wire Wire Line
 	4650 3050 4650 3100
@@
 Wire Wire Line
 	8550 3050 9000 3050
+$Comp
+L power:+3.3VP #PWR0105
+U 1 1 5E08FBF9
+P 6250 7000
+F 0 "#PWR0105" H 6400 6950 50  0001 C CNN
+F 1 "+3.3VP" H 6270 7143 50  0000 C CNN
+F 2 "" H 6250 7000 50  0001 C CNN
+F 3 "" H 6250 7000 50  0001 C CNN
+	1    6250 7000
+	1    0    0    -1
+$EndComp
+$Comp
+L power:+3.3VP #PWR0106
+U 1 1 5E090762
+P 4650 3050
+F 0 "#PWR0106" H 4800 3000 50  0001 C CNN
+F 1 "+3.3VP" H 4670 3193 50  0000 C CNN
+F 2 "" H 4650 3050 50  0001 C CNN
+F 3 "" H 4650 3050 50  0001 C CNN
+	1    4650 3050
+	1    0    0    -1
+$EndComp
+$Comp
+L power:+3.3VP #PWR0107
+U 1 1 5E091AC9
+P 6050 2550
+F 0 "#PWR0107" H 6200 2500 50  0001 C CNN
+F 1 "+3.3VP" H 6070 2693 50  0000 C CNN
+F 2 "" H 6050 2550 50  0001 C CNN
+F 3 "" H 6050 2550 50  0001 C CNN
+	1    6050 2550
+	1    0    0    -1
+$EndComp
 $EndSCHEMATC
