File: hardware/project/ETH1CPMU1/Isolation.sch (KiCad schematic (older format))
At the start: 3 parts, among them U1301 ADuM3151

Commit message: Function generator schematic design.
Parts:
- C1301, C1302: footprint (none) -> Capacitor_SMD:C_0603_1608Metric_Pad1.05x0.95mm_HandSolder
Connections:
- net MAIN_GPIO_OUT1 renamed MCU1_GPIO_OUT1
- net MAIN_GPIO_OUT2 renamed MCU1_GPIO_OUT2
- net MAIN_MCLK renamed MCU1_MCLK
- net MAIN_MISO renamed MCU1_MISO
- net MAIN_MOSI renamed MCU1_MOSI
- net MAIN_STATUS_IN renamed MCU1_STATUS_IN
- net MAIN_~MSS renamed MCU1_~MSS
- net SECOND_GPIO_OUT1 renamed MCU2_GPIO_OUT1
- net SECOND_GPIO_OUT2 renamed MCU2_GPIO_OUT2
- net SECOND_MISO renamed MCU2_MISO
- net SECOND_MOSI renamed MCU2_MOSI
- net SECOND_SCLK renamed MCU2_SCLK
- net SECOND_STATUS_IN renamed MCU2_STATUS_IN
- net SECOND_~SSS renamed MCU2_~SSS
Changed lines of the file:
@@
 $Descr A4 11693 8268
 encoding utf-8
-Sheet 13 14
+Sheet 15 15
 Title ""
 Date ""
@@
 F 0 "C1301" H 4865 1346 50  0000 L CNN
 F 1 "100n" H 4865 1255 50  0000 L CNN
-F 2 "" H 4788 1150 50  0001 C CNN
+F 2 "Capacitor_SMD:C_0603_1608Metric_Pad1.05x0.95mm_HandSolder" H 4788 1150 50  0001 C CNN
 F 3 "~" H 4750 1300 50  0001 C CNN
 	1    4750 1300
@@
 F 0 "C1302" H 6365 1396 50  0000 L CNN
 F 1 "100n" H 6365 1305 50  0000 L CNN
-F 2 "" H 6288 1200 50  0001 C CNN
+F 2 "Capacitor_SMD:C_0603_1608Metric_Pad1.05x0.95mm_HandSolder" H 6288 1200 50  0001 C CNN
 F 3 "~" H 6250 1350 50  0001 C CNN
 	1    6250 1350
@@
 $EndComp
 Text HLabel 4750 2900 0    50   Input ~ 0
-MAIN_GPIO_OUT1
+MCU1_GPIO_OUT1
 Text HLabel 4750 2700 0    50   Input ~ 0
-MAIN_~MSS
+MCU1_~MSS
 Text HLabel 4750 2600 0    50   Output ~ 0
-MAIN_MISO
+MCU1_MISO
 Text HLabel 4750 2500 0    50   Input ~ 0
-MAIN_MOSI
+MCU1_MOSI
 Text HLabel 4750 2400 0    50   Input ~ 0
-MAIN_MCLK
+MCU1_MCLK
 Text HLabel 4750 3100 0    50   Output ~ 0
-MAIN_STATUS_IN
+MCU1_STATUS_IN
 Text HLabel 4750 3000 0    50   Input ~ 0
-MAIN_GPIO_OUT2
+MCU1_GPIO_OUT2
 Wire Wire Line
 	4750 3100 4800 3100
@@
 	4750 2400 4800 2400
 Text HLabel 6250 2700 2    50   Output ~ 0
-SECOND_~SSS
+MCU2_~SSS
 Text HLabel 6250 2600 2    50   Input ~ 0
-SECOND_MISO
+MCU2_MISO
 Text HLabel 6250 2500 2    50   Output ~ 0
-SECOND_MOSI
+MCU2_MOSI
 Text HLabel 6250 2400 2    50   Output ~ 0
-SECOND_SCLK
+MCU2_SCLK
 Text HLabel 6250 2900 2    50   Output ~ 0
-SECOND_GPIO_OUT1
+MCU2_GPIO_OUT1
 Text HLabel 6250 3100 2    50   Input ~ 0
-SECOND_STATUS_IN
+MCU2_STATUS_IN
 Text HLabel 6250 3000 2    50   Output ~ 0
-SECOND_GPIO_OUT2
+MCU2_GPIO_OUT2
 Wire Wire Line
 	6250 2400 6200 2400

Commit message: New footprint development, changes in schematics.
Parts:
- U1501: renamed from U1301; footprint (none) -> Package_SO:SSOP-20_5.3x7.2mm_P0.65mm
- renumbered C1301 to C1501, C1302 to C1502
Changed lines of the file:
@@
 $EndDescr
 $Comp
-L ETH1CPMU1:ADuM3151 U1301
+L ETH1CPMU1:ADuM3151 U1501
 U 1 1 5DD9E9B5
 P 5500 2800
-F 0 "U1301" H 5500 3665 50  0000 C CNN
+F 0 "U1501" H 5500 3665 50  0000 C CNN
 F 1 "ADuM3151" H 5500 3574 50  0000 C CNN
-F 2 "" H 7400 3250 50  0001 C CNN
+F 2 "Package_SO:SSOP-20_5.3x7.2mm_P0.65mm" H 7400 3250 50  0001 C CNN
 F 3 "" H 7400 3250 50  0001 C CNN
 	1    5500 2800
@@
 	4750 2200 4800 2200
 $Comp
-L power:GND #PWR01307
+L power:GND #PWR01507
 U 1 1 5DDA742F
 P 4750 3500
-F 0 "#PWR01307" H 4750 3250 50  0001 C CNN
+F 0 "#PWR01507" H 4750 3250 50  0001 C CNN
 F 1 "GND" H 4755 3327 50  0000 C CNN
 F 2 "" H 4750 3500 50  0001 C CNN
@@
 	5500 3600 5500 7700
 $Comp
-L power:+3.3V #PWR01305
+L power:+3.3V #PWR01505
 U 1 1 5DDAF4AD
 P 4750 2100
-F 0 "#PWR01305" H 4750 1950 50  0001 C CNN
+F 0 "#PWR01505" H 4750 1950 50  0001 C CNN
 F 1 "+3.3V" H 4765 2273 50  0000 C CNN
 F 2 "" H 4750 2100 50  0001 C CNN
@@
 $EndComp
 $Comp
-L ETH1CPMU1:+3.3VF #PWR01306
+L ETH1CPMU1:+3.3VF #PWR01506
 U 1 1 5DDAFA37
 P 6250 2100
-F 0 "#PWR01306" H 6250 1950 50  0001 C CNN
+F 0 "#PWR01506" H 6250 1950 50  0001 C CNN
 F 1 "+3.3VF" H 6265 2273 50  0000 C CNN
 F 2 "" H 6250 2100 50  0001 C CNN
@@
 	6250 2200 6200 2200
 $Comp
-L ETH1CPMU1:DGNDF #PWR01308
+L ETH1CPMU1:DGNDF #PWR01508
 U 1 1 5DDB1D03
 P 6250 3500
-F 0 "#PWR01308" H 6250 3250 50  0001 C CNN
+F 0 "#PWR01508" H 6250 3250 50  0001 C CNN
 F 1 "DGNDF" H 6255 3327 50  0000 C CNN
 F 2 "" H 6250 3500 50  0001 C CNN
@@
 	6250 3400 6250 3300
 $Comp
-L power:+3.3V #PWR01301
+L power:+3.3V #PWR01501
 U 1 1 5DDB5B86
 P 4750 1150
-F 0 "#PWR01301" H 4750 1000 50  0001 C CNN
+F 0 "#PWR01501" H 4750 1000 50  0001 C CNN
 F 1 "+3.3V" H 4765 1323 50  0000 C CNN
 F 2 "" H 4750 1150 50  0001 C CNN
@@
 $EndComp
 $Comp
-L Device:C C1301
+L Device:C C1501
 U 1 1 5DDB7F1A
 P 4750 1300
-F 0 "C1301" H 4865 1346 50  0000 L CNN
+F 0 "C1501" H 4865 1346 50  0000 L CNN
 F 1 "100n" H 4865 1255 50  0000 L CNN
 F 2 "Capacitor_SMD:C_0603_1608Metric_Pad1.05x0.95mm_HandSolder" H 4788 1150 50  0001 C CNN
@@
 $EndComp
 $Comp
-L power:GND #PWR01303
+L power:GND #PWR01503
 U 1 1 5DDBBA7D
 P 4750 1450
-F 0 "#PWR01303" H 4750 1200 50  0001 C CNN
+F 0 "#PWR01503" H 4750 1200 50  0001 C CNN
 F 1 "GND" H 4755 1277 50  0000 C CNN
 F 2 "" H 4750 1450 50  0001 C CNN
@@
 $EndComp
 $Comp
-L Device:C C1302
+L Device:C C1502
 U 1 1 5DDC10CB
 P 6250 1350
-F 0 "C1302" H 6365 1396 50  0000 L CNN
+F 0 "C1502" H 6365 1396 50  0000 L CNN
 F 1 "100n" H 6365 1305 50  0000 L CNN
 F 2 "Capacitor_SMD:C_0603_1608Metric_Pad1.05x0.95mm_HandSolder" H 6288 1200 50  0001 C CNN
@@
 $EndComp
 $Comp
-L ETH1CPMU1:+3.3VF #PWR01302
+L ETH1CPMU1:+3.3VF #PWR01502
 U 1 1 5DDC1869
 P 6250 1200
-F 0 "#PWR01302" H 6250 1050 50  0001 C CNN
+F 0 "#PWR01502" H 6250 1050 50  0001 C CNN
 F 1 "+3.3VF" H 6265 1373 50  0000 C CNN
 F 2 "" H 6250 1200 50  0001 C CNN
@@
 $EndComp
 $Comp
-L ETH1CPMU1:DGNDF #PWR01304
+L ETH1CPMU1:DGNDF #PWR01504
 U 1 1 5DDC21F1
 P 6250 1500
-F 0 "#PWR01304" H 6250 1250 50  0001 C CNN
+F 0 "#PWR01504" H 6250 1250 50  0001 C CNN
 F 1 "DGNDF" H 6255 1327 50  0000 C CNN
 F 2 "" H 6250 1500 50  0001 C CNN

Commit message: Schematic and PCB design.
Other:
- moved on the sheet: C1502
Changed lines of the file:
@@
 L Device:C C1502
 U 1 1 5DDC10CB
-P 6250 1350
-F 0 "C1502" H 6365 1396 50  0000 L CNN
-F 1 "100n" H 6365 1305 50  0000 L CNN
-F 2 "Capacitor_SMD:C_0603_1608Metric_Pad1.05x0.95mm_HandSolder" H 6288 1200 50  0001 C CNN
-F 3 "~" H 6250 1350 50  0001 C CNN
-	1    6250 1350
+P 6250 1300
+F 0 "C1502" H 6365 1346 50  0000 L CNN
+F 1 "100n" H 6365 1255 50  0000 L CNN
+F 2 "Capacitor_SMD:C_0603_1608Metric_Pad1.05x0.95mm_HandSolder" H 6288 1150 50  0001 C CNN
+F 3 "~" H 6250 1300 50  0001 C CNN
+	1    6250 1300
 	1    0    0    -1
 $EndComp
@@
 L ETH1CPMU1:+3.3VF #PWR01502
 U 1 1 5DDC1869
-P 6250 1200
-F 0 "#PWR01502" H 6250 1050 50  0001 C CNN
-F 1 "+3.3VF" H 6265 1373 50  0000 C CNN
-F 2 "" H 6250 1200 50  0001 C CNN
-F 3 "" H 6250 1200 50  0001 C CNN
-	1    6250 1200
+P 6250 1150
+F 0 "#PWR01502" H 6250 1000 50  0001 C CNN
+F 1 "+3.3VF" H 6265 1323 50  0000 C CNN
+F 2 "" H 6250 1150 50  0001 C CNN
+F 3 "" H 6250 1150 50  0001 C CNN
+	1    6250 1150
 	1    0    0    -1
 $EndComp
@@
 L ETH1CPMU1:DGNDF #PWR01504
 U 1 1 5DDC21F1
-P 6250 1500
-F 0 "#PWR01504" H 6250 1250 50  0001 C CNN
-F 1 "DGNDF" H 6255 1327 50  0000 C CNN
-F 2 "" H 6250 1500 50  0001 C CNN
-F 3 "" H 6250 1500 50  0001 C CNN
-	1    6250 1500
+P 6250 1450
+F 0 "#PWR01504" H 6250 1200 50  0001 C CNN
+F 1 "DGNDF" H 6255 1277 50  0000 C CNN
+F 2 "" H 6250 1450 50  0001 C CNN
+F 3 "" H 6250 1450 50  0001 C CNN
+	1    6250 1450
 	1    0    0    -1
 $EndComp

Commit message: Schematic design
Parts:
- renumbered C1501 to C1001, C1502 to C1002, U1501 to U1001
Changed lines of the file:
@@
 $EndDescr
 $Comp
-L ETH1CPMU1:ADuM3151 U1501
+L ETH1CPMU1:ADuM3151 U1001
 U 1 1 5DD9E9B5
 P 5500 2800
-F 0 "U1501" H 5500 3665 50  0000 C CNN
+F 0 "U1001" H 5500 3665 50  0000 C CNN
 F 1 "ADuM3151" H 5500 3574 50  0000 C CNN
 F 2 "Package_SO:SSOP-20_5.3x7.2mm_P0.65mm" H 7400 3250 50  0001 C CNN
@@
 	4750 2200 4800 2200
 $Comp
-L power:GND #PWR01507
+L power:GND #PWR01007
 U 1 1 5DDA742F
 P 4750 3500
-F 0 "#PWR01507" H 4750 3250 50  0001 C CNN
+F 0 "#PWR01007" H 4750 3250 50  0001 C CNN
 F 1 "GND" H 4755 3327 50  0000 C CNN
 F 2 "" H 4750 3500 50  0001 C CNN
@@
 	5500 3600 5500 7700
 $Comp
-L power:+3.3V #PWR01505
+L power:+3.3V #PWR01005
 U 1 1 5DDAF4AD
 P 4750 2100
-F 0 "#PWR01505" H 4750 1950 50  0001 C CNN
+F 0 "#PWR01005" H 4750 1950 50  0001 C CNN
 F 1 "+3.3V" H 4765 2273 50  0000 C CNN
 F 2 "" H 4750 2100 50  0001 C CNN
@@
 $EndComp
 $Comp
-L ETH1CPMU1:+3.3VF #PWR01506
+L ETH1CPMU1:+3.3VF #PWR01006
 U 1 1 5DDAFA37
 P 6250 2100
-F 0 "#PWR01506" H 6250 1950 50  0001 C CNN
+F 0 "#PWR01006" H 6250 1950 50  0001 C CNN
 F 1 "+3.3VF" H 6265 2273 50  0000 C CNN
 F 2 "" H 6250 2100 50  0001 C CNN
@@
 	6250 2200 6200 2200
 $Comp
-L ETH1CPMU1:DGNDF #PWR01508
+L ETH1CPMU1:DGNDF #PWR01008
 U 1 1 5DDB1D03
 P 6250 3500
-F 0 "#PWR01508" H 6250 3250 50  0001 C CNN
+F 0 "#PWR01008" H 6250 3250 50  0001 C CNN
 F 1 "DGNDF" H 6255 3327 50  0000 C CNN
 F 2 "" H 6250 3500 50  0001 C CNN
@@
 	6250 3400 6250 3300
 $Comp
-L power:+3.3V #PWR01501
+L power:+3.3V #PWR01001
 U 1 1 5DDB5B86
 P 4750 1150
-F 0 "#PWR01501" H 4750 1000 50  0001 C CNN
+F 0 "#PWR01001" H 4750 1000 50  0001 C CNN
 F 1 "+3.3V" H 4765 1323 50  0000 C CNN
 F 2 "" H 4750 1150 50  0001 C CNN
@@
 $EndComp
 $Comp
-L Device:C C1501
+L Device:C C1001
 U 1 1 5DDB7F1A
 P 4750 1300
-F 0 "C1501" H 4865 1346 50  0000 L CNN
+F 0 "C1001" H 4865 1346 50  0000 L CNN
 F 1 "100n" H 4865 1255 50  0000 L CNN
 F 2 "Capacitor_SMD:C_0603_1608Metric_Pad1.05x0.95mm_HandSolder" H 4788 1150 50  0001 C CNN
@@
 $EndComp
 $Comp
-L power:GND #PWR01503
+L power:GND #PWR01003
 U 1 1 5DDBBA7D
 P 4750 1450
-F 0 "#PWR01503" H 4750 1200 50  0001 C CNN
+F 0 "#PWR01003" H 4750 1200 50  0001 C CNN
 F 1 "GND" H 4755 1277 50  0000 C CNN
 F 2 "" H 4750 1450 50  0001 C CNN
@@
 $EndComp
 $Comp
-L Device:C C1502
+L Device:C C1002
 U 1 1 5DDC10CB
 P 6250 1300
-F 0 "C1502" H 6365 1346 50  0000 L CNN
+F 0 "C1002" H 6365 1346 50  0000 L CNN
 F 1 "100n" H 6365 1255 50  0000 L CNN
 F 2 "Capacitor_SMD:C_0603_1608Metric_Pad1.05x0.95mm_HandSolder" H 6288 1150 50  0001 C CNN
@@
 $EndComp
 $Comp
-L ETH1CPMU1:+3.3VF #PWR01502
+L ETH1CPMU1:+3.3VF #PWR01002
 U 1 1 5DDC1869
 P 6250 1150
-F 0 "#PWR01502" H 6250 1000 50  0001 C CNN
+F 0 "#PWR01002" H 6250 1000 50  0001 C CNN
 F 1 "+3.3VF" H 6265 1323 50  0000 C CNN
 F 2 "" H 6250 1150 50  0001 C CNN
@@
 $EndComp
 $Comp
-L ETH1CPMU1:DGNDF #PWR01504
+L ETH1CPMU1:DGNDF #PWR01004
 U 1 1 5DDC21F1
 P 6250 1450
-F 0 "#PWR01504" H 6250 1200 50  0001 C CNN
+F 0 "#PWR01004" H 6250 1200 50  0001 C CNN
 F 1 "DGNDF" H 6255 1277 50  0000 C CNN
 F 2 "" H 6250 1450 50  0001 C CNN
