File: hardware/project/ETH1CPMU1/MCU_Third.sch (KiCad schematic (older format))
At the start: 0 parts

Commit message: Function generator schematic design.
Parts:
- added C1419, C1420: 8p, Capacitor_SMD:C_0603_1608Metric_Pad1.05x0.95mm_HandSolder, symbol Device:C
- added C1421: 2u2, Capacitor_SMD:C_0805_2012Metric_Pad1.15x1.40mm_HandSolder, symbol Device:C
- added C1422: 100n, Capacitor_SMD:C_0603_1608Metric_Pad1.05x0.95mm_HandSolder, symbol Device:C
- added J1401: Conn_02x05, symbol Connector_Generic:Conn_02x05_Odd_Even
- added R1418, R1419: 10k, Resistor_SMD:R_0603_1608Metric_Pad1.05x0.95mm_HandSolder, symbol Device:R
- added R1420, R1421: 4k7, Resistor_SMD:R_0603_1608Metric_Pad1.05x0.95mm_HandSolder, symbol Device:R
- added U1405: STM32F413RGT6Tx, symbol ETH1CPMU1-rescue:STM32F413RGT6Tx-ETH1CPMU1
- added U1406: 24LC08, symbol Memory_EEPROM:24LC08
- added Y1401: NX3225GD-8MHZ-STD-CRA-3, symbol Device:Crystal
Connections:
- net labels added: +3.3VP, DGNDF, EEPROM_SCL, EEPROM_SDA, EEPROM_WP, MCU_NRST, TCK_SWCLK, TMS_SWDIO
- wire segments 0 -> 75
- no-connect marks 0 -> 6

Commit message: Function generator schematic development.
Parts:
- removed U1405: STM32F413RGT6Tx, symbol ETH1CPMU1-rescue:STM32F413RGT6Tx-ETH1CPMU1
- added U1405: STM32F413RGT6Tx, symbol ETH1CPMU1:STM32F413RGT6Tx
Changed lines of the file:
@@
 EESchema Schematic File Version 4
-LIBS:ETH1CPMU1-cache
 EELAYER 30 0
 EELAYER END
@@
 Comment4 ""
 $EndDescr
-$Comp
-L ETH1CPMU1-rescue:STM32F413RGT6Tx-ETH1CPMU1 U?
-U 1 1 5E29D775
-P 7700 3650
-AR Path="/5DF36C25/5E29D775" Ref="U?"  Part="1"
-AR Path="/5E29C232/5E29D775" Ref="U1405"  Part="1"
-AR Path="/5E29D775" Ref="U1405"  Part="1"
-F 0 "U1405" H 2250 5450 50  0000 C CNN
-F 1 "STM32F413RGT6Tx" H 12850 5450 50  0000 C CNN
-F 2 "" H 1000 3050 50  0001 C CNN
-F 3 "" H 1000 3050 50  0001 C CNN
-	1    7700 3650
-	1    0    0    -1
-$EndComp
 Wire Wire Line
 	7500 5500 7500 5550
@@
 	1    0    0    -1
 $EndComp
+$Comp
+L ETH1CPMU1:STM32F413RGT6Tx U1405
+U 1 1 5DD8B08C
+P 7700 3650
+F 0 "U1405" H 2200 5450 50  0000 C CNN
+F 1 "STM32F413RGT6Tx" H 12900 5450 50  0000 C CNN
+F 2 "" H 1000 3050 50  0001 C CNN
+F 3 "" H 1000 3050 50  0001 C CNN
+	1    7700 3650
+	1    0    0    -1
+$EndComp

Commit message: New footprint development, changes in schematics.
Parts:
- J1401: footprint (none) -> Connector_PinHeader_1.27mm:PinHeader_2x05_P1.27mm_Vertical
- Y1401: footprint (none) -> ETH1CPMU1:NX3225GD
- renumbered C1419 to C1401, C1420 to C1402, C1421 to C1403, C1422 to C1404, R1418 to R1401, R1419 to R1402, R1420 to R1403, R1421 to R1404, U1405 to U1401, U1406 to U1402
Changed lines of the file:
@@
 P 7700 5600
 AR Path="/5DF36C25/5E29D787" Ref="#PWR?"  Part="1"
-AR Path="/5E29C232/5E29D787" Ref="#PWR01444"  Part="1"
-F 0 "#PWR01444" H 7700 5350 50  0001 C CNN
+AR Path="/5E29C232/5E29D787" Ref="#PWR01407"  Part="1"
+F 0 "#PWR01407" H 7700 5350 50  0001 C CNN
 F 1 "DGNDF" H 7705 5427 50  0000 C CNN
 F 2 "" H 7700 5600 50  0001 C CNN
@@
 P 7700 1700
 AR Path="/5DF36C25/5E29D79D" Ref="#PWR?"  Part="1"
-AR Path="/5E29C232/5E29D79D" Ref="#PWR01438"  Part="1"
-F 0 "#PWR01438" H 7850 1650 50  0001 C CNN
+AR Path="/5E29C232/5E29D79D" Ref="#PWR01401"  Part="1"
+F 0 "#PWR01401" H 7850 1650 50  0001 C CNN
 F 1 "+3.3VP" H 7720 1843 50  0000 C CNN
 F 2 "" H 7700 1700 50  0001 C CNN
@@
 P 13450 5100
 AR Path="/5DF36C25/5E29D7A6" Ref="R?"  Part="1"
-AR Path="/5E29C232/5E29D7A6" Ref="R1419"  Part="1"
-F 0 "R1419" H 13520 5146 50  0000 L CNN
+AR Path="/5E29C232/5E29D7A6" Ref="R1402"  Part="1"
+F 0 "R1402" H 13520 5146 50  0000 L CNN
 F 1 "10k" H 13520 5055 50  0000 L CNN
 F 2 "Resistor_SMD:R_0603_1608Metric_Pad1.05x0.95mm_HandSolder" V 13380 5100 50  0001 C CNN
@@
 P 13450 5300
 AR Path="/5DF36C25/5E29D7AE" Ref="#PWR?"  Part="1"
-AR Path="/5E29C232/5E29D7AE" Ref="#PWR01443"  Part="1"
-F 0 "#PWR01443" H 13450 5050 50  0001 C CNN
+AR Path="/5E29C232/5E29D7AE" Ref="#PWR01406"  Part="1"
+F 0 "#PWR01406" H 13450 5050 50  0001 C CNN
 F 1 "DGNDF" H 13455 5127 50  0000 C CNN
 F 2 "" H 13450 5300 50  0001 C CNN
@@
 F 0 "J1401" H 10300 10767 50  0000 C CNN
 F 1 "Conn_02x05" H 10300 10676 50  0000 C CNN
-F 2 "" H 10250 10350 50  0001 C CNN
+F 2 "Connector_PinHeader_1.27mm:PinHeader_2x05_P1.27mm_Vertical" H 10250 10350 50  0001 C CNN
 F 3 "~" H 10250 10350 50  0001 C CNN
 	1    10250 10350
@@
 P 9900 10600
 AR Path="/5DF35BC8/5E74C1B5" Ref="#PWR?"  Part="1"
-AR Path="/5E29C232/5E74C1B5" Ref="#PWR01450"  Part="1"
-F 0 "#PWR01450" H 9900 10350 50  0001 C CNN
+AR Path="/5E29C232/5E74C1B5" Ref="#PWR01413"  Part="1"
+F 0 "#PWR01413" H 9900 10350 50  0001 C CNN
 F 1 "DGNDF" H 9905 10427 50  0000 C CNN
 F 2 "" H 9900 10600 50  0001 C CNN
@@
 F 0 "Y1401" V 15104 3931 50  0000 L CNN
 F 1 "NX3225GD-8MHZ-STD-CRA-3" V 15195 3931 50  0000 L CNN
-F 2 "" H 15150 3800 50  0001 C CNN
+F 2 "ETH1CPMU1:NX3225GD" H 15150 3800 50  0001 C CNN
 F 3 "~" H 15150 3800 50  0001 C CNN
 	1    15150 3800
@@
 P 15150 4200
 AR Path="/5DCED281/5E7594BE" Ref="C?"  Part="1"
-AR Path="/5E29C232/5E7594BE" Ref="C1419"  Part="1"
-F 0 "C1419" H 15265 4246 50  0000 L CNN
+AR Path="/5E29C232/5E7594BE" Ref="C1401"  Part="1"
+F 0 "C1401" H 15265 4246 50  0000 L CNN
 F 1 "8p" H 15265 4155 50  0000 L CNN
 F 2 "Capacitor_SMD:C_0603_1608Metric_Pad1.05x0.95mm_HandSolder" H 15188 4050 50  0001 C CNN
@@
 P 15650 4200
 AR Path="/5DCED281/5E7594C4" Ref="C?"  Part="1"
-AR Path="/5E29C232/5E7594C4" Ref="C1420"  Part="1"
-F 0 "C1420" H 15765 4246 50  0000 L CNN
+AR Path="/5E29C232/5E7594C4" Ref="C1402"  Part="1"
+F 0 "C1402" H 15765 4246 50  0000 L CNN
 F 1 "8p" H 15765 4155 50  0000 L CNN
 F 2 "Capacitor_SMD:C_0603_1608Metric_Pad1.05x0.95mm_HandSolder" H 15688 4050 50  0001 C CNN
@@
 	13350 3700 13800 3700
 $Comp
-L Device:R R1418
+L Device:R R1401
 U 1 1 5E7616EE
 P 14300 4400
-F 0 "R1418" H 14230 4354 50  0000 R CNN
+F 0 "R1401" H 14230 4354 50  0000 R CNN
 F 1 "10k" H 14230 4445 50  0000 R CNN
 F 2 "Resistor_SMD:R_0603_1608Metric_Pad1.05x0.95mm_HandSolder" V 14230 4400 50  0001 C CNN
@@
 P 8000 10300
 AR Path="/5DCED281/5E76F022" Ref="U?"  Part="1"
-AR Path="/5E29C232/5E76F022" Ref="U1406"  Part="1"
-F 0 "U1406" H 8200 10650 50  0000 C CNN
+AR Path="/5E29C232/5E76F022" Ref="U1402"  Part="1"
+F 0 "U1402" H 8200 10650 50  0000 C CNN
 F 1 "24LC08" H 8200 10550 50  0000 C CNN
 F 2 "" H 8000 10300 50  0001 C CNN
@@
 P 8950 10000
 AR Path="/5DCED281/5E76F046" Ref="R?"  Part="1"
-AR Path="/5E29C232/5E76F046" Ref="R1420"  Part="1"
-F 0 "R1420" H 9020 10046 50  0000 L CNN
+AR Path="/5E29C232/5E76F046" Ref="R1403"  Part="1"
+F 0 "R1403" H 9020 10046 50  0000 L CNN
 F 1 "4k7" H 9020 9955 50  0000 L CNN
 F 2 "Resistor_SMD:R_0603_1608Metric_Pad1.05x0.95mm_HandSolder" V 8880 10000 50  0001 C CNN
@@
 P 9300 10000
 AR Path="/5DCED281/5E76F04C" Ref="R?"  Part="1"
-AR Path="/5E29C232/5E76F04C" Ref="R1421"  Part="1"
-F 0 "R1421" H 9370 10046 50  0000 L CNN
+AR Path="/5E29C232/5E76F04C" Ref="R1404"  Part="1"
+F 0 "R1404" H 9370 10046 50  0000 L CNN
 F 1 "4k7" H 9370 9955 50  0000 L CNN
 F 2 "Resistor_SMD:R_0603_1608Metric_Pad1.05x0.95mm_HandSolder" V 9230 10000 50  0001 C CNN
@@
 Connection ~ 9300 9800
 $Comp
-L power:+3.3VP #PWR01447
+L power:+3.3VP #PWR01410
 U 1 1 5E770710
 P 9900 10050
-F 0 "#PWR01447" H 10050 10000 50  0001 C CNN
+F 0 "#PWR01410" H 10050 10000 50  0001 C CNN
 F 1 "+3.3VP" H 9920 10193 50  0000 C CNN
 F 2 "" H 9900 10050 50  0001 C CNN
@@
 $EndComp
 $Comp
-L ETH1CPMU1:DGNDF #PWR01449
+L ETH1CPMU1:DGNDF #PWR01412
 U 1 1 5E77122F
 P 8000 10600
-F 0 "#PWR01449" H 8000 10350 50  0001 C CNN
+F 0 "#PWR01412" H 8000 10350 50  0001 C CNN
 F 1 "DGNDF" H 8005 10427 50  0000 C CNN
 F 2 "" H 8000 10600 50  0001 C CNN
@@
 $EndComp
 $Comp
-L ETH1CPMU1:DGNDF #PWR01448
+L ETH1CPMU1:DGNDF #PWR01411
 U 1 1 5E7714DB
 P 7550 10600
-F 0 "#PWR01448" H 7550 10350 50  0001 C CNN
+F 0 "#PWR01411" H 7550 10350 50  0001 C CNN
 F 1 "DGNDF" H 7555 10427 50  0000 C CNN
 F 2 "" H 7550 10600 50  0001 C CNN
@@
 $EndComp
 $Comp
-L power:+3.3VP #PWR01446
+L power:+3.3VP #PWR01409
 U 1 1 5E7718B5
 P 8000 9950
-F 0 "#PWR01446" H 8150 9900 50  0001 C CNN
+F 0 "#PWR01409" H 8150 9900 50  0001 C CNN
 F 1 "+3.3VP" H 8020 10093 50  0000 C CNN
 F 2 "" H 8000 9950 50  0001 C CNN
@@
 	8000 9950 8000 10000
 $Comp
-L power:+3.3VP #PWR01445
+L power:+3.3VP #PWR01408
 U 1 1 5E772DFA
 P 9300 9750
-F 0 "#PWR01445" H 9450 9700 50  0001 C CNN
+F 0 "#PWR01408" H 9450 9700 50  0001 C CNN
 F 1 "+3.3VP" H 9320 9893 50  0000 C CNN
 F 2 "" H 9300 9750 50  0001 C CNN
@@
 $EndComp
 $Comp
-L Device:C C1421
+L Device:C C1403
 U 1 1 5E776A2B
 P 13550 4300
-F 0 "C1421" V 13298 4300 50  0000 C CNN
+F 0 "C1403" V 13298 4300 50  0000 C CNN
 F 1 "2u2" V 13389 4300 50  0000 C CNN
 F 2 "Capacitor_SMD:C_0805_2012Metric_Pad1.15x1.40mm_HandSolder" H 13588 4150 50  0001 C CNN
@@
 	13400 4300 13350 4300
 $Comp
-L ETH1CPMU1:DGNDF #PWR01441
+L ETH1CPMU1:DGNDF #PWR01404
 U 1 1 5E77E2A8
 P 15400 4450
-F 0 "#PWR01441" H 15400 4200 50  0001 C CNN
+F 0 "#PWR01404" H 15400 4200 50  0001 C CNN
 F 1 "DGNDF" H 15405 4277 50  0000 C CNN
 F 2 "" H 15400 4450 50  0001 C CNN
@@
 $EndComp
 $Comp
-L ETH1CPMU1:DGNDF #PWR01440
+L ETH1CPMU1:DGNDF #PWR01403
 U 1 1 5E77E4B3
 P 13750 4300
-F 0 "#PWR01440" H 13750 4050 50  0001 C CNN
+F 0 "#PWR01403" H 13750 4050 50  0001 C CNN
 F 1 "DGNDF" V 13755 4172 50  0000 R CNN
 F 2 "" H 13750 4300 50  0001 C CNN
@@
 	13800 3700 13800 4000
 $Comp
-L Device:C C1422
+L Device:C C1404
 U 1 1 5E7B49DC
 P 14300 4800
-F 0 "C1422" H 14415 4846 50  0000 L CNN
+F 0 "C1404" H 14415 4846 50  0000 L CNN
 F 1 "100n" H 14415 4755 50  0000 L CNN
 F 2 "Capacitor_SMD:C_0603_1608Metric_Pad1.05x0.95mm_HandSolder" H 14338 4650 50  0001 C CNN
@@
 P 14300 4950
 AR Path="/5DF36C25/5E7BFF4D" Ref="#PWR?"  Part="1"
-AR Path="/5E29C232/5E7BFF4D" Ref="#PWR01442"  Part="1"
-F 0 "#PWR01442" H 14300 4700 50  0001 C CNN
+AR Path="/5E29C232/5E7BFF4D" Ref="#PWR01405"  Part="1"
+F 0 "#PWR01405" H 14300 4700 50  0001 C CNN
 F 1 "DGNDF" H 14305 4777 50  0000 C CNN
 F 2 "" H 14300 4950 50  0001 C CNN
@@
 $EndComp
 $Comp
-L power:+3.3VP #PWR01439
+L power:+3.3VP #PWR01402
 U 1 1 5E7C0507
 P 14300 4250
-F 0 "#PWR01439" H 14450 4200 50  0001 C CNN
+F 0 "#PWR01402" H 14450 4200 50  0001 C CNN
 F 1 "+3.3VP" H 14320 4393 50  0000 C CNN
 F 2 "" H 14300 4250 50  0001 C CNN
@@
 $EndComp
 $Comp
-L ETH1CPMU1:STM32F413RGT6Tx U1405
+L ETH1CPMU1:STM32F413RGT6Tx U1401
 U 1 1 5DD8B08C
 P 7700 3650
-F 0 "U1405" H 2200 5450 50  0000 C CNN
+F 0 "U1401" H 2200 5450 50  0000 C CNN
 F 1 "STM32F413RGT6Tx" H 12900 5450 50  0000 C CNN
 F 2 "" H 1000 3050 50  0001 C CNN

Commit message: Schematic and PCB design.
Parts:
- U1401: footprint (none) -> Package_QFP:LQFP-64_10x10mm_P0.5mm
- U1402: value 24LC08 -> 24LC08B-E/MS; footprint (none) -> Package_SO:MSOP-8_3x3mm_P0.65mm
Changed lines of the file:
@@
 AR Path="/5DCED281/5E76F022" Ref="U?"  Part="1"
 AR Path="/5E29C232/5E76F022" Ref="U1402"  Part="1"
-F 0 "U1402" H 8200 10650 50  0000 C CNN
-F 1 "24LC08" H 8200 10550 50  0000 C CNN
-F 2 "" H 8000 10300 50  0001 C CNN
+F 0 "U1402" H 8350 10650 50  0000 C CNN
+F 1 "24LC08B-E/MS" H 8350 10550 50  0000 C CNN
+F 2 "Package_SO:MSOP-8_3x3mm_P0.65mm" H 8000 10300 50  0001 C CNN
 F 3 "http://ww1.microchip.com/downloads/en/DeviceDoc/21710J.pdf" H 8000 10300 50  0001 C CNN
 	1    8000 10300
@@
 F 0 "U1401" H 2200 5450 50  0000 C CNN
 F 1 "STM32F413RGT6Tx" H 12900 5450 50  0000 C CNN
-F 2 "" H 1000 3050 50  0001 C CNN
+F 2 "Package_QFP:LQFP-64_10x10mm_P0.5mm" H 1000 3050 50  0001 C CNN
 F 3 "" H 1000 3050 50  0001 C CNN
 	1    7700 3650

Commit message: Schematic design
Parts:
- added C1405, C1406, C1407, C1408, C1409, C1410: 100n, Capacitor_SMD:C_0603_1608Metric_Pad1.05x0.95mm_HandSolder, symbol Device:C
Connections:
- net labels added: DDS_DAC_RSTSEL, DDS_DAC_SCLK, DDS_DAC_SDIN, DDS_DAC_SDO, DDS_DAC_~LDAC, DDS_DAC_~RESET, DDS_DAC_~SYNC, DDS_FGEN_FSELECT, DDS_FGEN_PSEL0, DDS_FGEN_PSEL1, DDS_FGEN_SCLK, DDS_FGEN_SDATA, DDS_FGEN_~FSYNC, DDS_MDAC_DIN, DDS_MDAC_SCLK, DDS_MDAC_~SYNC, DDS_MEAS_A0, DDS_MEAS_A1, DDS_MEAS_A2, DDS_MEAS_CLK, DDS_MEAS_CONV, DDS_MEAS_DATA, MCU3_MISO, MCU3_MOSI, MCU3_NSS, MCU3_SCLK
- wire segments 75 -> 127
- no-connect marks 6 -> 21

Commit message: Schematic design
Parts:
- renumbered C1401 to C1201, C1402 to C1202, C1403 to C1203, C1404 to C1204, C1405 to C1205, C1406 to C1206, C1407 to C1207, C1408 to C1208, C1409 to C1209, C1410 to C1210, J1401 to J1201, R1401 to R1201, R1402 to R1202, R1403 to R1203, R1404 to R1204, U1401 to U1201, U1402 to U1202, Y1401 to Y1201

Commit message: PCB design.
Parts:
- added C1211: 100n, Capacitor_SMD:C_0603_1608Metric_Pad1.05x0.95mm_HandSolder, symbol Device:C
Connections:
- net +3.3VP: now also C1211.1
- net DGNDF: now also C1211.2
Changed lines of the file:
@@
 P 9900 10600
 AR Path="/5DF35BC8/5E74C1B5" Ref="#PWR?"  Part="1"
-AR Path="/5E29C232/5E74C1B5" Ref="#PWR01214"  Part="1"
-F 0 "#PWR01214" H 9900 10350 50  0001 C CNN
+AR Path="/5E29C232/5E74C1B5" Ref="#PWR01215"  Part="1"
+F 0 "#PWR01215" H 9900 10350 50  0001 C CNN
 F 1 "DGNDF" H 9905 10427 50  0000 C CNN
 F 2 "" H 9900 10600 50  0001 C CNN
@@
 $EndComp
 $Comp
-L ETH1CPMU1:DGNDF #PWR01213
+L ETH1CPMU1:DGNDF #PWR01214
 U 1 1 5E77122F
 P 8000 10600
-F 0 "#PWR01213" H 8000 10350 50  0001 C CNN
+F 0 "#PWR01214" H 8000 10350 50  0001 C CNN
 F 1 "DGNDF" H 8005 10427 50  0000 C CNN
 F 2 "" H 8000 10600 50  0001 C CNN
@@
 $EndComp
 $Comp
-L ETH1CPMU1:DGNDF #PWR01212
+L ETH1CPMU1:DGNDF #PWR01213
 U 1 1 5E7714DB
 P 7550 10600
-F 0 "#PWR01212" H 7550 10350 50  0001 C CNN
+F 0 "#PWR01213" H 7550 10350 50  0001 C CNN
 F 1 "DGNDF" H 7555 10427 50  0000 C CNN
 F 2 "" H 7550 10600 50  0001 C CNN
@@
 	1450 10700 1950 10700
 $Comp
-L ETH1CPMU1:DGNDF #PWR01215
+L ETH1CPMU1:DGNDF #PWR01216
 U 1 1 5E107792
 P 2200 10750
-F 0 "#PWR01215" H 2200 10500 50  0001 C CNN
+F 0 "#PWR01216" H 2200 10500 50  0001 C CNN
 F 1 "DGNDF" H 2205 10577 50  0000 C CNN
 F 2 "" H 2200 10750 50  0001 C CNN
@@
 Wire Wire Line
 	2200 10300 2450 10300
+$Comp
+L Device:C C1211
+U 1 1 5DEC46E0
+P 4100 10500
+F 0 "C1211" H 4215 10546 50  0000 L CNN
+F 1 "100n" H 4215 10455 50  0000 L CNN
+F 2 "Capacitor_SMD:C_0603_1608Metric_Pad1.05x0.95mm_HandSolder" H 4138 10350 50  0001 C CNN
+F 3 "~" H 4100 10500 50  0001 C CNN
+	1    4100 10500
+	1    0    0    -1
+$EndComp
+$Comp
+L power:+3.3VP #PWR01212
+U 1 1 5DEC5CD8
+P 4100 10250
+F 0 "#PWR01212" H 4250 10200 50  0001 C CNN
+F 1 "+3.3VP" H 4120 10393 50  0000 C CNN
+F 2 "" H 4100 10250 50  0001 C CNN
+F 3 "" H 4100 10250 50  0001 C CNN
+	1    4100 10250
+	1    0    0    -1
+$EndComp
+$Comp
+L ETH1CPMU1:DGNDF #PWR01217
+U 1 1 5DEC5F6E
+P 4100 10750
+F 0 "#PWR01217" H 4100 10500 50  0001 C CNN
+F 1 "DGNDF" H 4105 10577 50  0000 C CNN
+F 2 "" H 4100 10750 50  0001 C CNN
+F 3 "" H 4100 10750 50  0001 C CNN
+	1    4100 10750
+	1    0    0    -1
+$EndComp
+Wire Wire Line
+	4100 10750 4100 10650
+Wire Wire Line
+	4100 10250 4100 10350
 $EndSCHEMATC

Commit message: PCB design
Parts:
- renumbered C1205 to C1101, C1206 to C1102, C1207 to C1103, C1208 to C1104, C1209 to C1105, C1210 to C1106, C1211 to C1107, C1203 to C1108, C1204 to C1109, C1201 to C1110, C1202 to C1111, J1201 to J1101, R1203 to R1101, R1204 to R1102, R1202 to R1103, R1201 to R1104, U1201 to U1101, U1202 to U1102, Y1201 to Y1101
Connections:
- net AC_RELAY: now reaches U1101.37 (PC6,TIM3_CH1,TIM8_CH1,I2CFMP1_SCL,I2S2_MCK,DFSDM1_CKIN3,DFSDM2_DATIN6,USART6_TX,FSMC_D1,FSMC_DA1,SDIO_D6,EVENTOUT)
- no-connect marks 21 -> 20
