File: hardware/project/ETH1CPMU1/MCU_Third.sch (KiCad schematic (older format))
At the start: 19 parts, among them J1101 Conn_02x05, U1101 STM32F413RGT6Tx, U1102 24LC08B-E/MS, Y1101 NX3225GD-8MHZ-STD-CRA-3

Commit message: PCB designed
Connections:
- net MCU3_NSS: now also U1101.54 (PD2,TIM3_ETR,DFSDM2_CKOUT,UART5_RX,FSMC_NWE,SDIO_CMD,EVENTOUT); no longer U1101.20 (PA4,SPI1_NSS,I2S1_WS,SPI3_NSS,I2S3_WS,USART2_CK,DFSDM1_DATIN1,FSMC_D6,FSMC_DA6,EVENTOUT,ADC1_IN4,DAC_OUT1)
Changed lines of the file:
@@
 MCU3_MOSI
 Wire Wire Line
-	2050 2400 2000 2400
-Text HLabel 2000 2400 0    50   Input ~ 0
+	2050 5200 2000 5200
+Text HLabel 2000 5200 0    50   Input ~ 0
 MCU3_NSS
 Text HLabel 2000 2300 0    50   Output ~ 0
@@
 NoConn ~ 13350 3400
 NoConn ~ 2050 5000
-NoConn ~ 2050 5200
 NoConn ~ 2050 4200
 NoConn ~ 2050 4100
@@
 Wire Wire Line
 	2000 4300 2050 4300
+NoConn ~ 2050 2400
 $EndSCHEMATC
