File: hardware/project/ETH1CPMU1/Trigger.sch (KiCad schematic (older format))
At the start: 17 parts, among them U801 74AC125, U802 ADuM5402

Commit message: PCB design
Parts:
- renumbered D802 to D801, D801 to D802, R802 to R801, R803 to R802, R801 to R803, U802 to U801, U801 to U802
Changed lines of the file:
@@
 $Descr A4 11693 8268
 encoding utf-8
-Sheet 8 15
+Sheet 8 16
 Title ""
 Date ""
@@
 $EndDescr
 $Comp
-L Isolator:ADuM5402 U802
+L Isolator:ADuM5402 U801
 U 1 1 5D995D35
 P 4700 3350
-F 0 "U802" H 4300 4000 50  0000 C CNN
+F 0 "U801" H 4300 4000 50  0000 C CNN
 F 1 "ADuM5402" H 4300 3900 50  0000 C CNN
 F 2 "Package_SO:SOIC-16W_7.5x10.3mm_P1.27mm" H 4700 2400 50  0001 C CIN
@@
 	4800 2700 4800 2750
 $Comp
-L ETH1CPMU1:74AC125 U801
+L ETH1CPMU1:74AC125 U802
 U 3 1 5D9C7DE2
 P 7900 3250
-F 0 "U801" H 7900 3716 50  0000 C CNN
+F 0 "U802" H 7900 3716 50  0000 C CNN
 F 1 "74AC125" H 7900 3625 50  0000 C CNN
 F 2 "Package_SO:TSSOP-14_4.4x5mm_P0.65mm" H 7900 3250 50  0001 C CNN
@@
 	8450 5450 8650 5450
 $Comp
-L Device:D_Zener D801
+L Device:D_Zener D802
 U 1 1 5D1F1550
 P 8550 4800
-F 0 "D801" V 8504 4879 50  0000 L CNN
+F 0 "D802" V 8504 4879 50  0000 L CNN
 F 1 "SMBJ5.0A" V 8595 4879 50  0000 L CNN
 F 2 "Diode_SMD:D_SMB" H 8550 4800 50  0001 C CNN
@@
 	8550 4600 7950 4600
 $Comp
-L Device:R R801
+L Device:R R803
 U 1 1 5D1F8BEC
 P 7950 4400
-F 0 "R801" H 8020 4446 50  0000 L CNN
+F 0 "R803" H 8020 4446 50  0000 L CNN
 F 1 "1k" H 8020 4355 50  0000 L CNN
 F 2 "Resistor_SMD:R_0603_1608Metric_Pad1.05x0.95mm_HandSolder" V 7880 4400 50  0001 C CNN
@@
 	7950 4200 7950 4250
 $Comp
-L ETH1CPMU1:74AC125 U801
+L ETH1CPMU1:74AC125 U802
 U 4 1 5D218310
 P 6100 4600
-F 0 "U801" H 6500 4850 50  0000 C CNN
+F 0 "U802" H 6500 4850 50  0000 C CNN
 F 1 "74AC125" H 6500 4750 50  0000 C CNN
 F 2 "Package_SO:TSSOP-14_4.4x5mm_P0.65mm" H 6100 4600 50  0001 C CNN
@@
 $EndComp
 $Comp
-L ETH1CPMU1:74AC125 U801
+L ETH1CPMU1:74AC125 U802
 U 2 1 5D2189A9
 P 7900 2400
-F 0 "U801" H 7900 2866 50  0000 C CNN
+F 0 "U802" H 7900 2866 50  0000 C CNN
 F 1 "74AC125" H 7900 2775 50  0000 C CNN
 F 2 "Package_SO:TSSOP-14_4.4x5mm_P0.65mm" H 7900 2400 50  0001 C CNN
@@
 $EndComp
 $Comp
-L ETH1CPMU1:74AC125 U801
+L ETH1CPMU1:74AC125 U802
 U 1 1 5D21AD13
 P 7900 1550
-F 0 "U801" H 7900 2016 50  0000 C CNN
+F 0 "U802" H 7900 2016 50  0000 C CNN
 F 1 "74AC125" H 7900 1925 50  0000 C CNN
 F 2 "Package_SO:TSSOP-14_4.4x5mm_P0.65mm" H 7900 1550 50  0001 C CNN
@@
 Connection ~ 7350 3250
 $Comp
-L Device:R R803
+L Device:R R802
 U 1 1 5D25C5D7
 P 7050 5450
-F 0 "R803" V 6843 5450 50  0000 C CNN
+F 0 "R802" V 6843 5450 50  0000 C CNN
 F 1 "100" V 6934 5450 50  0000 C CNN
 F 2 "Resistor_SMD:R_0603_1608Metric_Pad1.05x0.95mm_HandSolder" V 6980 5450 50  0001 C CNN
@@
 	6650 5450 6900 5450
 $Comp
-L Device:R R802
+L Device:R R801
 U 1 1 5D27667C
 P 6100 5450
-F 0 "R802" V 5893 5450 50  0000 C CNN
+F 0 "R801" V 5893 5450 50  0000 C CNN
 F 1 "14k7" V 5984 5450 50  0000 C CNN
 F 2 "Resistor_SMD:R_0603_1608Metric_Pad1.05x0.95mm_HandSolder" V 6030 5450 50  0001 C CNN
@@
 NoConn ~ 4200 3550
 $Comp
-L power:+3.3V #PWR0807
+L power:+3.3V #PWR0804
 U 1 1 5EBBBCC5
 P 4500 2650
-F 0 "#PWR0807" H 4500 2500 50  0001 C CNN
+F 0 "#PWR0804" H 4500 2500 50  0001 C CNN
 F 1 "+3.3V" H 4515 2823 50  0000 C CNN
 F 2 "" H 4500 2650 50  0001 C CNN
@@
 $EndComp
 $Comp
-L power:GND #PWR0804
+L power:GND #PWR0802
 U 1 1 5EBCD574
 P 4100 1400
-F 0 "#PWR0804" H 4100 1150 50  0001 C CNN
+F 0 "#PWR0802" H 4100 1150 50  0001 C CNN
 F 1 "GND" H 4105 1227 50  0000 C CNN
 F 2 "" H 4100 1400 50  0001 C CNN
@@
 $EndComp
 $Comp
-L power:GND #PWR0810
+L power:GND #PWR0803
 U 1 1 5EBD53EB
 P 4400 4050
-F 0 "#PWR0810" H 4400 3800 50  0001 C CNN
+F 0 "#PWR0803" H 4400 3800 50  0001 C CNN
 F 1 "GND" H 4405 3877 50  0000 C CNN
 F 2 "" H 4400 4050 50  0001 C CNN
@@
 $EndComp
 $Comp
-L ETH1CPMU1:GND_TRIG #PWR0811
+L ETH1CPMU1:GND_TRIG #PWR0806
 U 1 1 5EBDBFF4
 P 5000 4050
-F 0 "#PWR0811" H 5000 3800 50  0001 C CNN
+F 0 "#PWR0806" H 5000 3800 50  0001 C CNN
 F 1 "GND_TRIG" H 5005 3877 50  0000 C CNN
 F 2 "" H 5000 4050 50  0001 C CNN
@@
 $EndComp
 $Comp
-L ETH1CPMU1:GND_TRIG #PWR0815
+L ETH1CPMU1:GND_TRIG #PWR0818
 U 1 1 5EBDCCC1
 P 7950 6100
-F 0 "#PWR0815" H 7950 5850 50  0001 C CNN
+F 0 "#PWR0818" H 7950 5850 50  0001 C CNN
 F 1 "GND_TRIG" H 7955 5927 50  0000 C CNN
 F 2 "" H 7950 6100 50  0001 C CNN
@@
 $EndComp
 $Comp
-L ETH1CPMU1:GND_TRIG #PWR0816
+L ETH1CPMU1:GND_TRIG #PWR0820
 U 1 1 5EBDD668
 P 9100 6100
-F 0 "#PWR0816" H 9100 5850 50  0001 C CNN
+F 0 "#PWR0820" H 9100 5850 50  0001 C CNN
 F 1 "GND_TRIG" H 9105 5927 50  0000 C CNN
 F 2 "" H 9100 6100 50  0001 C CNN
@@
 $EndComp
 $Comp
-L ETH1CPMU1:GND_TRIG #PWR0817
+L ETH1CPMU1:GND_TRIG #PWR0821
 U 1 1 5EBDD8F0
 P 9850 6100
-F 0 "#PWR0817" H 9850 5850 50  0001 C CNN
+F 0 "#PWR0821" H 9850 5850 50  0001 C CNN
 F 1 "GND_TRIG" H 9855 5927 50  0000 C CNN
 F 2 "" H 9850 6100 50  0001 C CNN
@@
 $EndComp
 $Comp
-L ETH1CPMU1:GND_TRIG #PWR0814
+L ETH1CPMU1:GND_TRIG #PWR0819
 U 1 1 5EBDF6F2
 P 8550 4950
-F 0 "#PWR0814" H 8550 4700 50  0001 C CNN
+F 0 "#PWR0819" H 8550 4700 50  0001 C CNN
 F 1 "GND_TRIG" H 8555 4777 50  0000 C CNN
 F 2 "" H 8550 4950 50  0001 C CNN
@@
 $EndComp
 $Comp
-L ETH1CPMU1:GND_TRIG #PWR0805
+L ETH1CPMU1:GND_TRIG #PWR0811
 U 1 1 5EBE030C
 P 5800 1400
-F 0 "#PWR0805" H 5800 1150 50  0001 C CNN
+F 0 "#PWR0811" H 5800 1150 50  0001 C CNN
 F 1 "GND_TRIG" H 5805 1227 50  0000 C CNN
 F 2 "" H 5800 1400 50  0001 C CNN
@@
 $EndComp
 $Comp
-L ETH1CPMU1:GND_TRIG #PWR0806
+L ETH1CPMU1:GND_TRIG #PWR0815
 U 1 1 5EBE0F56
 P 6550 1400
-F 0 "#PWR0806" H 6550 1150 50  0001 C CNN
+F 0 "#PWR0815" H 6550 1150 50  0001 C CNN
 F 1 "GND_TRIG" H 6555 1227 50  0000 C CNN
 F 2 "" H 6550 1400 50  0001 C CNN
@@
 $EndComp
 $Comp
-L ETH1CPMU1:+5V_TRIG #PWR0802
+L ETH1CPMU1:+5V_TRIG #PWR0810
 U 1 1 5EBE2413
 P 5800 900
-F 0 "#PWR0802" H 5800 750 50  0001 C CNN
+F 0 "#PWR0810" H 5800 750 50  0001 C CNN
 F 1 "+5V_TRIG" H 5815 1073 50  0000 C CNN
 F 2 "" H 5800 900 50  0001 C CNN
@@
 $EndComp
 $Comp
-L ETH1CPMU1:+5V_TRIG #PWR0803
+L ETH1CPMU1:+5V_TRIG #PWR0814
 U 1 1 5EBE29CC
 P 6550 900
-F 0 "#PWR0803" H 6550 750 50  0001 C CNN
+F 0 "#PWR0814" H 6550 750 50  0001 C CNN
 F 1 "+5V_TRIG" H 6565 1073 50  0000 C CNN
 F 2 "" H 6550 900 50  0001 C CNN
@@
 $EndComp
 $Comp
-L ETH1CPMU1:+5V_TRIG #PWR0808
+L ETH1CPMU1:+5V_TRIG #PWR0805
 U 1 1 5EBE2D84
 P 5000 2650
-F 0 "#PWR0808" H 5000 2500 50  0001 C CNN
+F 0 "#PWR0805" H 5000 2500 50  0001 C CNN
 F 1 "+5V_TRIG" H 5015 2823 50  0000 C CNN
 F 2 "" H 5000 2650 50  0001 C CNN
@@
 $EndComp
 $Comp
-L ETH1CPMU1:+5V_TRIG #PWR0813
+L ETH1CPMU1:+5V_TRIG #PWR0816
 U 1 1 5EBE6C8E
 P 6650 4500
-F 0 "#PWR0813" H 6650 4350 50  0001 C CNN
+F 0 "#PWR0816" H 6650 4350 50  0001 C CNN
 F 1 "+5V_TRIG" V 6650 4650 50  0000 L CNN
 F 2 "" H 6650 4500 50  0001 C CNN
@@
 $EndComp
 $Comp
-L ETH1CPMU1:+5V_TRIG #PWR0812
+L ETH1CPMU1:+5V_TRIG #PWR0817
 U 1 1 5EBE9033
 P 7950 4200
-F 0 "#PWR0812" H 7950 4050 50  0001 C CNN
+F 0 "#PWR0817" H 7950 4050 50  0001 C CNN
 F 1 "+5V_TRIG" H 7965 4373 50  0000 C CNN
 F 2 "" H 7950 4200 50  0001 C CNN
@@
 $EndComp
 $Comp
-L Diode:BAV99 D802
+L Diode:BAV99 D801
 U 1 1 5DD77A27
 P 7950 5450
-F 0 "D802" V 8200 5100 50  0000 L CNN
+F 0 "D801" V 8200 5100 50  0000 L CNN
 F 1 "BAV99" V 8100 5050 50  0000 L CNN
 F 2 "Package_TO_SOT_SMD:SOT-23" H 7950 4950 50  0001 C CNN
@@
 	7950 5750 7950 6100
 $Comp
-L ETH1CPMU1:74AC125 U801
+L ETH1CPMU1:74AC125 U802
 U 5 1 5E72A776
 P 5150 7100
-F 0 "U801" H 4750 7200 50  0000 C CNN
+F 0 "U802" H 4750 7200 50  0000 C CNN
 F 1 "74AC125" H 4750 7050 50  0000 C CNN
 F 2 "Package_SO:TSSOP-14_4.4x5mm_P0.65mm" H 5150 7100 50  0001 C CNN
@@
 $EndComp
 $Comp
-L ETH1CPMU1:+5V_TRIG #PWR0818
+L ETH1CPMU1:+5V_TRIG #PWR0807
 U 1 1 5E72EC8D
 P 5150 6750
-F 0 "#PWR0818" H 5150 6600 50  0001 C CNN
+F 0 "#PWR0807" H 5150 6600 50  0001 C CNN
 F 1 "+5V_TRIG" H 5165 6923 50  0000 C CNN
 F 2 "" H 5150 6750 50  0001 C CNN
@@
 $EndComp
 $Comp
-L ETH1CPMU1:GND_TRIG #PWR0819
+L ETH1CPMU1:GND_TRIG #PWR0808
 U 1 1 5E7300C2
 P 5150 7450
-F 0 "#PWR0819" H 5150 7200 50  0001 C CNN
+F 0 "#PWR0808" H 5150 7200 50  0001 C CNN
 F 1 "GND_TRIG" H 5155 7277 50  0000 C CNN
 F 2 "" H 5150 7450 50  0001 C CNN
@@
 $EndComp
 $Comp
-L ETH1CPMU1:GND_TRIG #PWR0820
+L ETH1CPMU1:GND_TRIG #PWR0812
 U 1 1 5DE91DF7
 P 6050 7450
-F 0 "#PWR0820" H 6050 7200 50  0001 C CNN
+F 0 "#PWR0812" H 6050 7200 50  0001 C CNN
 F 1 "GND_TRIG" H 6055 7277 50  0000 C CNN
 F 2 "" H 6050 7450 50  0001 C CNN
@@
 $EndComp
 $Comp
-L ETH1CPMU1:+5V_TRIG #PWR0821
+L ETH1CPMU1:+5V_TRIG #PWR0813
 U 1 1 5DE9761E
 P 6500 7450
-F 0 "#PWR0821" H 6500 7300 50  0001 C CNN
+F 0 "#PWR0813" H 6500 7300 50  0001 C CNN
 F 1 "+5V_TRIG" H 6515 7623 50  0000 C CNN
 F 2 "" H 6500 7450 50  0001 C CNN
