File: hardware/project/ETH1CPMU1/ETH1CPMU1.kicad_pcb (KiCad board)
At the start: 2 copper layers, 160 x 100 mm, 436 parts, among them J1301 Conn_02x05, J1401 Conn_02x05, J301 Conn_02x05, J302 Conn_02x01, K1101 HE3621A0510, K1102 HE3621A0510, K1103 HE3621A0510, K1104 HE3621A0510, K1105 HE3621A0510, K1106 HE3621A0510, K1107 HE3621A0510, K1108 HE3621A0510, K801 TQ2SA-5V, Q1101 BC847, Q1102 BC847, Q1103 BC847, Q1104 BC847, Q1105 BC847, Q1106 BC847, Q1107 BC847, Q1108 BC847, U1001 74AC125, U1002 ADuM5402, U1102 DG419LEUA, U1103 AD5520, U1201 INA159, U1202 ADG1414BRU, U1203 ADS8363, U1204 INA159, U1301 STM32H743ZI, U1501 ADuM3151, U301 STM32F765ZGT6, U402 LAN8742A, U501 LM1117IMP-3.3/NOPB, U503 MAX5902, U602 LM1117IMP-3.3/NOPB, U603 MC7815BD2TG, U604 LM1117IMP-3.3/NOPB, U606 LT8330_S6, U607 MC7915BD2TG, U608 LM1117IMP-5.0/NOPB, U610 LT8330_S6, U701 REF02AU, U702 AD8676, U703 AD8676, U704 AD8675, U705 AD5791, U801 AD5453YRMZ, U802 LT1468, U803 LT1468, U804 AD9835, U806 74AHCT1G08, U807 REF192, U808 TL071, U809 DG419LEUA, U810 TL072, U811 ADS7818, U812 AD5689BRUZ, U813 TL071, U814 TL072, U901 REF192, U902 TL071, U903 AD5689BRUZ, U904 TL071, Y1301 NX3225GD-8MHZ-STD-CRA-3, Y1401 NX3225GD-8MHZ-STD-CRA-3, Y301 NX3225GD-8MHZ-STD-CRA-3, Y401 NX5032GA-25.000M-LN-CD-1

Commit message: Schematic and PCB design.
Parts:
- added C607: 1u/HC, Capacitor_SMD:C_1206_3216Metric_Pad1.42x1.75mm_HandSolder, F.Cu at (181.5, 148.0)
- added C620: 1u/HC, Capacitor_SMD:C_1206_3216Metric_Pad1.42x1.75mm_HandSolder, F.Cu at (190.5, 147.0)
- added J201: C64AC, ETH1CPMU1:Socket_DIN41612-CaseC1-AC-Male-64Pin-2rows, F.Cu at (222.0, 90.0)
- added L1001: CW252016-R33G, ETH1CPMU1:CW252016, F.Cu at (206.2, 87.0)
- added L601: 7448013501, ETH1CPMU1:7448013501, F.Cu at (90.8, 132.2)
- added Q501: IRFR5410, ETH1CPMU1:TO-252-2_Rectifier, F.Cu at (205.2, 134.0)
- added TP601: 5006, TestPoint:TestPoint_Loop_D2.60mm_Drill1.6mm_Beaded, F.Cu at (153.9, 63.0)
- added TP701: 5006, TestPoint:TestPoint_Loop_D2.60mm_Drill1.6mm_Beaded, F.Cu at (145.7, 62.9)
- added U1101: THS6012, ETH1CPMU1:PowerPAD, F.Cu at (178.5, 49.2)
- added U1302: 24LC08B-E/MS, Package_SO:MSOP-8_3x3mm_P0.65mm, B.Cu at (138.8, 110.0)
- added U1401: STM32F413RGT6Tx, Package_QFP:LQFP-64_10x10mm_P0.5mm, F.Cu at (137.9, 75.9)
- added U1402: 24LC08B-E/MS, Package_SO:MSOP-8_3x3mm_P0.65mm, F.Cu at (235.7, 12.7)
- added U302: 24LC08B-E/MS, Package_SO:MSOP-8_3x3mm_P0.65mm, B.Cu at (165.5, 117.2)
- added U401: LC03-3.3, ETH1CPMU1:SO8E, F.Cu at (211.3, 102.5)
- added U403: LC03-3.3, ETH1CPMU1:SO8E, F.Cu at (211.3, 108.6)
- added U502: TSR1-2450, ETH1CPMU1:TSR1, F.Cu at (204.2, 123.5)
- added U601: THL15-2415WI, ETH1CPMU1:THL15, F.Cu at (92.8, 110.2)
- added U605: TSR2-2450, ETH1CPMU1:TSR2, F.Cu at (100.8, 88.2)
- added U609: TSR1-2490, ETH1CPMU1:TSR1, F.Cu at (83.8, 90.2)
- added U805: ECS-3225SMV-500-GP-TR, ETH1CPMU1:ECS, F.Cu at (164.8, 71.0)
- C1003, D1003, F501, R1005: moved to B.Cu
- C501, C502: footprint Capacitor_SMD:C_2220_5650Metric_Pad1.97x5.40mm_HandSolder -> Capacitor_SMD:C_1206_3216Metric_Pad1.42x1.75mm_HandSolder
- C503, C504: value 22u/16V -> 10u/16V; footprint Capacitor_SMD:C_2220_5650Metric_Pad1.97x5.40mm_HandSolder -> Capacitor_SMD:C_1206_3216Metric_Pad1.42x1.75mm_HandSolder; moved to B.Cu
- C605, C612, C613, C623, C624: value 22u/16V -> 10u/16V; footprint Capacitor_SMD:C_2220_5650Metric_Pad1.97x5.40mm_HandSolder -> Capacitor_SMD:C_1206_3216Metric_Pad1.42x1.75mm_HandSolder
- C608, C609, C610, C611, C621, C622: footprint Capacitor_SMD:C_1210_3225Metric_Pad1.42x2.65mm_HandSolder -> Capacitor_SMD:C_1206_3216Metric_Pad1.42x1.75mm_HandSolder
- RV701: value 10k -> 3314J-1-103E; footprint Resistor_SMD:R_0603_1608Metric_Pad1.05x0.95mm_HandSolder -> Potentiometer_SMD:Potentiometer_Bourns_3314J_Vertical
- U806: footprint Package_TO_SOT_SMD:SOT-23-5_HandSoldering -> Package_TO_SOT_SMD:SOT-353_SC-70-5_Handsoldering
- moved J1301 348.3 mm to (121.8, 125.0), turned to 180 degrees
- moved U903 337.7 mm to (115.8, 65.8)
- moved U1203 290.5 mm to (132.2, 91.9)
- moved C608 272.1 mm to (88.0, 76.5)
- moved U608 269.1 mm to (54.5, 79.2)
- moved C603 258.6 mm to (105.5, 132.2), turned to 90 degrees
- moved C602 258.4 mm to (101.5, 132.3), turned to 90 degrees
- moved C503 249.5 mm to (193.5, 126.5), turned to 180 degrees
- moved C1004 249.1 mm to (195.9, 81.8)
- moved C1003 246.5 mm to (189.8, 86.2), turned to 270 degrees
- moved U610 243.2 mm to (97.5, 69.8)
- moved C504 243.1 mm to (193.5, 124.0), turned to 180 degrees
- moved D1002 242.7 mm to (197.5, 91.8), turned to 180 degrees
- moved U806 240.2 mm to (167.2, 86.8)
- moved U1001 237.5 mm to (196.2, 86.8)
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- renumbered R1303 to R1301, R1304 to R1302, R1301 to R1303, R1302 to R1304
Connections:
- C1001 pad 2: AGNDF -> GND
- C1002 pad 2: AGNDF -> GND
- C1003 pad 1: +3.3VP -> +5V_TRIG
- C1003 pad 2: AGNDF -> GND_TRIG
- C1004 pad 1: +3.3VP -> +5V_TRIG
- C1004 pad 2: AGNDF -> GND_TRIG
- C1005 pad 1: +3.3VP -> +5V_TRIG
- C1005 pad 2: AGNDF -> GND_TRIG
- C1403 pad 2: (no net) -> Net-(C1403-Pad2)
- C1501 pad 2: AGNDF -> GND
- C301 pad 2: AGNDF -> GND
- C302 pad 2: AGNDF -> GND
- C303 pad 2: AGNDF -> GND
- C304 pad 2: AGNDF -> GND
- C305 pad 2: AGNDF -> GND
- C306 pad 2: AGNDF -> GND
- C307 pad 2: AGNDF -> GND
- C308 pad 2: AGNDF -> GND
- C309 pad 2: AGNDF -> GND
- C310 pad 2: AGNDF -> GND
- C311 pad 2: AGNDF -> GND
- C312 pad 2: AGNDF -> GND
- C313 pad 2: AGNDF -> GND
- C314 pad 2: AGNDF -> GND
- C315 pad 2: AGNDF -> GND
- C316 pad 2: AGNDF -> GND
- C317 pad 2: AGNDF -> GND
- C318 pad 2: AGNDF -> GND
- C319 pad 2: AGNDF -> GND
- C320 pad 2: AGNDF -> GND
- C401 pad 2: AGNDF -> GND
- C402 pad 2: AGNDF -> GND
- C403 pad 2: AGNDF -> GND
- C404 pad 2: AGNDF -> GND
- C405 pad 2: AGNDF -> GND
- C406 pad 2: AGNDF -> GND
- C407 pad 2: AGNDF -> GND
- C408 pad 2: AGNDF -> GND
- C409 pad 2: AGNDF -> GND
- C410 pad 2: AGNDF -> GND
- C412 pad 2: AGNDF -> GND
- C413 pad 2: AGNDF -> GND
- C414 pad 2: AGNDF -> GND
- C501 pad 2: AGNDF -> GND
- C502 pad 2: AGNDF -> GND
- C503 pad 2: AGNDF -> GND
- C504 pad 2: AGNDF -> GND
- C601 pad 2: (no net) -> Net-(C601-Pad2)
- C602 pad 2: AGNDF -> GND
- C603 pad 2: AGNDF -> GND
- C606 pad 2: (no net) -> Net-(C606-Pad2)
- D1001 pad 2: AGNDF -> GND_TRIG
- D1002 pad 1: AGNDF -> GND_TRIG
- D1003 pad 2: AGNDF -> GND_TRIG
- D502 pad 2: AGNDF -> GND
- D503 pad 1: AGNDF -> GND
- F501 pad 2: (no net) -> +24V
- J1401 pad 2: (no net) -> /MCU3/TMS_SWDIO
- J1401 pad 4: (no net) -> /MCU3/TCK_SWCLK
- J301 pad 3: AGNDF -> GND
- J301 pad 5: AGNDF -> GND
- J302 pad 2: AGNDF -> GND
- K1104 pad 4: (no net) -> /Connector/A
- K1105 pad 4: (no net) -> /Connector/B
- K1107 pad 4: (no net) -> /Connector/C
- K1108 pad 4: (no net) -> /Connector/E
- L401 pad 11: (no net) -> Net-(L401-Pad11)
- L401 pad 14: (no net) -> Net-(L401-Pad14)
- L401 pad 16: (no net) -> Net-(L401-Pad16)
- L401 pad 9: (no net) -> Net-(L401-Pad9)
- R1001 pad 1: +3.3VP -> +5V_TRIG
- R1004 pad 2: (no net) -> Net-(L1001-Pad2)
- R1005 pad 2: AGNDF -> GND_TRIG
- R1102 pad 1: (no net) -> Net-(R1102-Pad1)
- R1402 pad 1: (no net) -> Net-(R1402-Pad1)
- R1403 pad 2: (no net) -> /MCU3/EEPROM_SDA
- R1404 pad 2: (no net) -> /MCU3/EEPROM_SCL
- R304 pad 2: AGNDF -> GND
- R407 pad 2: AGNDF -> GND
- R409 pad 1: AGNDF -> GND
- R413 pad 2: AGNDF -> GND
- R414 pad 2: AGNDF -> GND
- R415 pad 2: AGNDF -> GND
- R416 pad 2: AGNDF -> GND
- U1001 pad 13: +3.3VP -> +5V_TRIG
- U1001 pad 14: +3.3VP -> +5V_TRIG
- U1001 pad 7: AGNDF -> GND_TRIG
- U1002 pad 10: +3.3VP -> +5V_TRIG
- U1002 pad 15: AGNDF -> GND_TRIG
- U1002 pad 16: +3.3VP -> +5V_TRIG
- U1002 pad 2: AGNDF -> GND
- U1002 pad 8: AGNDF -> GND
- U1002 pad 9: AGNDF -> GND_TRIG
- U1301 pad 53: (no net) -> /MCU2/EEPROM_WP
- U1501 pad 10: AGNDF -> GND
- U1501 pad 2: AGNDF -> GND
- U301 pad 107: AGNDF -> GND
- U301 pad 120: AGNDF -> GND
- U301 pad 130: AGNDF -> GND
- U301 pad 16: AGNDF -> GND
- U301 pad 31: AGNDF -> GND
- U301 pad 38: AGNDF -> GND
- U301 pad 51: AGNDF -> GND
- U301 pad 53: (no net) -> /MCU1/EEPROM_WP
- U301 pad 61: AGNDF -> GND
- U301 pad 83: AGNDF -> GND
- U301 pad 94: AGNDF -> GND
- U402 pad 25: AGNDF -> GND
- U501 pad 1: AGNDF -> GND
- U503 pad 3: (no net) -> Net-(Q501-Pad1)
- U503 pad 4: AGNDF -> GND
Other:
- outline, holes or cut-outs redrawn
- copper layers 2 -> 4
- rule pad_to_mask_clearance: 0.051 -> 0
- rule solder_mask_min_width: 0.25 -> 0.1

Commit message: Schematic design
Parts:
- added C1405: 100n, Capacitor_SMD:C_0603_1608Metric_Pad1.05x0.95mm_HandSolder, F.Cu at (153.2, 97.5)
- added C1406: 100n, Capacitor_SMD:C_0603_1608Metric_Pad1.05x0.95mm_HandSolder, F.Cu at (153.2, 100.0)
- added C1407: 100n, Capacitor_SMD:C_0603_1608Metric_Pad1.05x0.95mm_HandSolder, F.Cu at (157.6, 97.5)
- added C1408: 100n, Capacitor_SMD:C_0603_1608Metric_Pad1.05x0.95mm_HandSolder, F.Cu at (157.6, 100.0)
- added C1409: 100n, Capacitor_SMD:C_0603_1608Metric_Pad1.05x0.95mm_HandSolder, F.Cu at (161.9, 97.5)
- added C1410: 100n, Capacitor_SMD:C_0603_1608Metric_Pad1.05x0.95mm_HandSolder, F.Cu at (161.9, 100.0)
- added C841: 100n, Capacitor_SMD:C_0603_1608Metric_Pad1.05x0.95mm_HandSolder, F.Cu at (141.0, 154.5)
- added C842: 100n, Capacitor_SMD:C_0603_1608Metric_Pad1.05x0.95mm_HandSolder, F.Cu at (149.9, 147.8)
- added R838: 10k, Resistor_SMD:R_0603_1608Metric_Pad1.05x0.95mm_HandSolder, F.Cu at (141.0, 157.0)
- added R839: 10k, Resistor_SMD:R_0603_1608Metric_Pad1.05x0.95mm_HandSolder, F.Cu at (145.3, 154.5)
- added R840: 70k, Resistor_SMD:R_0603_1608Metric_Pad1.05x0.95mm_HandSolder, F.Cu at (153.5, 143.0)
- added R841: 10k, Resistor_SMD:R_0603_1608Metric_Pad1.05x0.95mm_HandSolder, F.Cu at (153.5, 145.5)
- added R842: 10k, Resistor_SMD:R_0603_1608Metric_Pad1.05x0.95mm_HandSolder, F.Cu at (157.8, 143.0)
- added R843: 10k, Resistor_SMD:R_0603_1608Metric_Pad1.05x0.95mm_HandSolder, F.Cu at (157.8, 145.5)
- added U815: TXB0104D, Package_SO:SOIC-14_3.9x8.7mm_P1.27mm, F.Cu at (134.6, 151.6)
- U809: value DG419LEUA -> DG408DY; footprint Package_SO:MSOP-8_3x3mm_P0.65mm -> Package_SO:TSSOP-16_4.4x5mm_P0.65mm
- moved U809 284.2 mm to (143.3, 149.9)
- moved R501 0.50 mm to (214.8, 131.8)
- moved U503 0.10 mm to (214.8, 134.8)
Connections:
- R819 pad 1: (no net) -> /AC source/DDS_MEAS_DATA
- R835 pad 2: (no net) -> /AC source/DDS_DAC_RSTSEL
- U1301 pad 111: (no net) -> /DAC/DAC_SCLK
- U1301 pad 113: (no net) -> /DAC/DAC_SDIN
- U1301 pad 114: (no net) -> /DAC/DAC_~LDAC
- U1401 pad 11: (no net) -> /AC source/DDS_MEAS_DATA
- U1401 pad 14: (no net) -> /AC source/DDS_DAC_RSTSEL
- U1401 pad 15: (no net) -> /AC source/DDS_MDAC_DIN
- U1401 pad 16: (no net) -> /AC source/DDS_DAC_~LDAC
- U1401 pad 17: (no net) -> /AC source/DDS_DAC_~RESET
- U1401 pad 21: (no net) -> /AC source/DDS_DAC_SCLK
- U1401 pad 22: (no net) -> /AC source/DDS_DAC_SDO
- U1401 pad 23: (no net) -> /AC source/DDS_DAC_SDIN
- U1401 pad 26: (no net) -> /AC source/DDS_FGEN_SCLK
- U1401 pad 27: (no net) -> /AC source/DDS_FGEN_~FSYNC
- U1401 pad 28: (no net) -> /AC source/DDS_FGEN_FSELECT
- U1401 pad 29: (no net) -> /AC source/DDS_MEAS_CLK
- U1401 pad 33: (no net) -> /AC source/DDS_MDAC_~SYNC
- U1401 pad 34: (no net) -> /AC source/DDS_MDAC_SCLK
- U1401 pad 38: (no net) -> /AC source/DDS_MEAS_A0
- U1401 pad 39: (no net) -> /AC source/DDS_MEAS_A1
- U1401 pad 40: (no net) -> /AC source/DDS_MEAS_A2
- U1401 pad 41: (no net) -> /AC source/DDS_FGEN_PSEL0
- U1401 pad 42: (no net) -> /AC source/DDS_FGEN_PSEL1
- U1401 pad 43: (no net) -> /AC source/DDS_FGEN_SDATA
- U1401 pad 50: (no net) -> /AC source/DDS_DAC_~SYNC
- U1401 pad 57: (no net) -> /MCU3/EEPROM_WP
- U1401 pad 58: (no net) -> /MCU3/EEPROM_SCL
- U1401 pad 59: (no net) -> /MCU3/EEPROM_SDA
- U1401 pad 62: (no net) -> /AC source/DDS_MEAS_CONV
- U1402 pad 7: (no net) -> /MCU3/EEPROM_WP
- U801 pad 3: (no net) -> /AC source/DDS_MDAC_SCLK
- U801 pad 4: (no net) -> /AC source/DDS_MDAC_DIN
- U801 pad 5: (no net) -> /AC source/DDS_MDAC_~SYNC
- U804 pad 10: (no net) -> /AC source/DDS_FGEN_FSELECT
- U804 pad 11: (no net) -> /AC source/DDS_FGEN_PSEL1
- U804 pad 12: (no net) -> /AC source/DDS_FGEN_PSEL0
- U804 pad 7: (no net) -> /AC source/DDS_FGEN_SCLK
- U804 pad 8: (no net) -> /AC source/DDS_FGEN_SDATA
- U809 pad 2: /AC source/MEAS_AMPL -> Net-(R838-Pad1)
- U809 pad 3: AGNDF -> -15VF
- U809 pad 4: +15VF -> AGNDF
- U809 pad 5: +3.3VP -> /AC source/MEAS_AMPL
- U809 pad 6: (no net) -> Net-(R840-Pad1)
- U809 pad 7: -15VF -> Net-(R842-Pad2)
- U809 pad 8: /AC source/MEAS_OUT -> Net-(U809-Pad8)
- U810 pad 3: Net-(U809-Pad1) -> Net-(U809-Pad8)
- U811 pad 5: (no net) -> /AC source/DDS_MEAS_CONV
- U811 pad 7: (no net) -> /AC source/DDS_MEAS_CLK
- U812 pad 12: (no net) -> /AC source/DDS_DAC_SCLK
- U812 pad 14: (no net) -> /AC source/DDS_DAC_SDIN
- U812 pad 8: (no net) -> /AC source/DDS_DAC_SDO
- U812 pad 9: (no net) -> /AC source/DDS_DAC_~LDAC
- U903 pad 12: (no net) -> /DAC/DAC_SCLK
- U903 pad 14: (no net) -> /DAC/DAC_SDIN
- U903 pad 9: (no net) -> /DAC/DAC_~LDAC

Commit message: PCB design.
Parts:
- removed C1115: 10u, Capacitor_SMD:C_1206_3216Metric_Pad1.42x1.75mm_HandSolder
- removed C813: 100n, Capacitor_SMD:C_0603_1608Metric_Pad1.05x0.95mm_HandSolder
- removed the C907 at (455.9, 133.7)
- removed the C908 at (468.5, 120.5)
- removed FB601, FB602: 742792031, Inductor_SMD:L_0805_2012Metric_Pad1.15x1.40mm_HandSolder
- removed the R1202 at (437.4, 128.8)
- removed the R1203 at (422.9, 133.1)
- removed U808, U813: TL071, Package_SO:SOIC-8_3.9x4.9mm_P1.27mm
- removed the U902 at (457.8, 120.0)
- removed the U904 at (457.3, 126.7)
- added C1110: 100n, Capacitor_SMD:C_0603_1608Metric_Pad1.05x0.95mm_HandSolder, B.Cu at (164.0, 97.2)
- added C1211: 100n, Capacitor_SMD:C_0603_1608Metric_Pad1.05x0.95mm_HandSolder, B.Cu at (126.1, 102.9)
- added C1313: 100n, Capacitor_SMD:C_0603_1608Metric_Pad1.05x0.95mm_HandSolder, B.Cu at (139.8, 80.6)
- added C1415: 10u, Capacitor_SMD:C_0805_2012Metric_Pad1.15x1.40mm_HandSolder, F.Cu at (153.8, 55.9)
- added C1507: 1u, Capacitor_SMD:C_0603_1608Metric_Pad1.05x0.95mm_HandSolder, B.Cu at (139.7, 114.7)
- added C320: 100n, Capacitor_SMD:C_0603_1608Metric_Pad1.05x0.95mm_HandSolder, B.Cu at (171.3, 129.4)
- added C902: 1n, Capacitor_SMD:C_0603_1608Metric_Pad1.05x0.95mm_HandSolder, B.Cu at (157.0, 81.5)
- added FB1501: 742792031, Inductor_SMD:L_0805_2012Metric_Pad1.15x1.40mm_HandSolder, B.Cu at (139.7, 111.0)
- added R902: 100, Resistor_SMD:R_0603_1608Metric_Pad1.05x0.95mm_HandSolder, F.Cu at (157.4, 81.5)
- added U1102: TL072, Package_SO:SOIC-8_3.9x4.9mm_P1.27mm, F.Cu at (169.5, 97.2)
- added U1309: TL072, Package_SO:SOIC-8_3.9x4.9mm_P1.27mm, F.Cu at (124.5, 75.4)
- added U903: INA159, Package_SO:MSOP-8_3x3mm_P0.65mm, F.Cu at (161.8, 81.5)
- C1001: renamed from C1501; moved to B.Cu
- C1002: renamed from C1502; moved to B.Cu
- C1101: renamed from C901; moved to B.Cu
- C1102: renamed from C902; moved to B.Cu
- C1103: renamed from C903; moved to B.Cu
- C1104: renamed from C904; moved to B.Cu
- C1105: renamed from C905; moved to B.Cu
- C1106: renamed from C906; moved to B.Cu
- C1107: renamed from C909; moved to B.Cu
- C1108: renamed from C910; moved to B.Cu
- C1109: renamed from C911; moved to B.Cu
- C1201: renamed from C1401; moved to B.Cu
- C1202: renamed from C1402; moved to B.Cu
- C1203: renamed from C1403; moved to B.Cu
- C1204: renamed from C1404; moved to B.Cu
- C1205: renamed from C1405; moved to B.Cu
- C1206: renamed from C1406; moved to B.Cu
- C1207: renamed from C1407; moved to B.Cu
- C1208: renamed from C1408; moved to B.Cu
- C1209: renamed from C1409; moved to B.Cu
- C1210: renamed from C1410; moved to B.Cu
- C1301: renamed from C801; moved to B.Cu
- C1302: renamed from C802; moved to B.Cu
- C1303: renamed from C803; moved to B.Cu
- C1304: renamed from C804; moved to B.Cu
- C1314: renamed from C815; moved to B.Cu
- C1315: renamed from C816; moved to B.Cu
- C1316: renamed from C819; moved to B.Cu
- C1317: renamed from C820; moved to B.Cu
- C1318: renamed from C814; moved to B.Cu
- C1319: renamed from C817; moved to B.Cu
- C1320: renamed from C818; moved to B.Cu
- C1322: renamed from C822; moved to B.Cu
- C1323: renamed from C823; moved to B.Cu
- C1324: renamed from C824; moved to B.Cu
- C1325: renamed from C826; moved to B.Cu
- C1326: renamed from C828; moved to B.Cu
- C1327: renamed from C825; moved to B.Cu
- C1329: renamed from C829; moved to B.Cu
- C1330: renamed from C830; moved to B.Cu
- C1331: renamed from C831; moved to B.Cu
- C1332: renamed from C832; moved to B.Cu
- C1333: renamed from C833; moved to B.Cu
- C1334: renamed from C834; moved to B.Cu
- C1335: renamed from C835; moved to B.Cu
- C1338: renamed from C838; moved to B.Cu
- C1339: renamed from C839; moved to B.Cu
- C1340: renamed from C840; moved to B.Cu
- C1341: renamed from C841; moved to B.Cu
- C1342: renamed from C842; moved to B.Cu
- C1401: renamed from C1101; moved to B.Cu
- C1402: renamed from C1102; moved to B.Cu
- C1403: renamed from C1103; moved to B.Cu
- C1404: renamed from C1104; moved to B.Cu
- C1405: renamed from C1105; moved to B.Cu
- C1406: renamed from C1106; moved to B.Cu
- C1407: renamed from C1107; moved to B.Cu
- C1408: renamed from C1108; moved to B.Cu
- C1409: renamed from C1109; moved to B.Cu
- C1410: renamed from C1110; moved to B.Cu
- C1411: renamed from C1111; moved to B.Cu
- C1412: renamed from C1112; moved to B.Cu
- C1413: renamed from C1113; moved to B.Cu
- C1414: renamed from C1114; moved to B.Cu
- C1416: renamed from C1116; moved to B.Cu
- C1417: renamed from C1117; footprint Capacitor_SMD:C_1206_3216Metric_Pad1.42x1.75mm_HandSolder -> Capacitor_SMD:C_0805_2012Metric_Pad1.15x1.40mm_HandSolder; moved to B.Cu
- C1418: renamed from C1118; moved to B.Cu
- C1419: renamed from C1119; footprint Capacitor_SMD:C_1206_3216Metric_Pad1.42x1.75mm_HandSolder -> Capacitor_SMD:C_0805_2012Metric_Pad1.15x1.40mm_HandSolder; moved to B.Cu
- C1420: renamed from C1120; moved to B.Cu
- C1421: renamed from C1121; moved to B.Cu
- C1422: renamed from C1122; moved to B.Cu
- C1423: renamed from C1123; footprint Capacitor_SMD:C_1206_3216Metric_Pad1.42x1.75mm_HandSolder -> Capacitor_SMD:C_0805_2012Metric_Pad1.15x1.40mm_HandSolder
- C1424: renamed from C1124; moved to B.Cu
- C1425: renamed from C1125; footprint Capacitor_SMD:C_1206_3216Metric_Pad1.42x1.75mm_HandSolder -> Capacitor_SMD:C_0805_2012Metric_Pad1.15x1.40mm_HandSolder; moved to B.Cu
- C1426: renamed from C1126; moved to B.Cu
- C1501: renamed from C1301; moved to B.Cu
- C1502: renamed from C1302; moved to B.Cu
- C1503: renamed from C1303; moved to B.Cu
- C1504: renamed from C1304; moved to B.Cu
- C1505: renamed from C1305; moved to B.Cu
- C1506: renamed from C1306; moved to B.Cu
- C1508: renamed from C1307; moved to B.Cu
- C1509: renamed from C1308; moved to B.Cu
- C1510: renamed from C1309; moved to B.Cu
- C1511: renamed from C1310; moved to B.Cu
- C1512: renamed from C1311; moved to B.Cu
- C1513: renamed from C1312; moved to B.Cu
- C1514: renamed from C1313; moved to B.Cu
- C1515: renamed from C1314; moved to B.Cu
- C1516: renamed from C1315; moved to B.Cu
- C1517: renamed from C1316; moved to B.Cu
- C1518: renamed from C1317; moved to B.Cu
- C1519: renamed from C1318; moved to B.Cu
- C301, C302, C303, C304, C305, C306, C307, C308, C309, C310, C311, C312, C313, C314, C315, C316, C317, C318, C319, C401, C405, C406, C407, C408, C410, C411, C412, C413, C414, C601, C602, C603, C604, C605, C606, C607, C610, C611, C612, C613, C614, C619, C620, C622, C623, C624, C625, C630, C704, C706, C708, C710, C712, C714, C716, C718, C720, C722, D601, D602, FB301, R301, R302, R304, R401, R402, R403, R404, R409, R410, R411, R414, R415, R416, R417, R418, R419, R420, R421, R601, R607, Y301: moved to B.Cu
- C321: renamed from C320; moved to B.Cu
- C627, C628: footprint Capacitor_SMD:C_0805_2012Metric_Pad1.15x1.40mm_HandSolder -> Capacitor_SMD:C_1206_3216Metric_Pad1.42x1.75mm_HandSolder
- C703, C705, C707, C709, C711, C713, C715, C717, C719: footprint Capacitor_SMD:C_1206_3216Metric_Pad1.42x1.75mm_HandSolder -> Capacitor_SMD:C_0805_2012Metric_Pad1.15x1.40mm_HandSolder; moved to B.Cu
- C721: footprint Capacitor_SMD:C_1206_3216Metric_Pad1.42x1.75mm_HandSolder -> Capacitor_SMD:C_0805_2012Metric_Pad1.15x1.40mm_HandSolder
- C801: renamed from C1001; moved to B.Cu
- C802: renamed from C1002; moved to B.Cu
- C804: renamed from C1004; moved to B.Cu
- C805: renamed from C1005; moved to B.Cu
- C901: renamed from C1201; moved to B.Cu
- C903: renamed from C1202; moved to B.Cu
- C904: renamed from C1203; moved to B.Cu
- C905: renamed from C1204; footprint Capacitor_SMD:C_1206_3216Metric_Pad1.42x1.75mm_HandSolder -> Capacitor_SMD:C_0805_2012Metric_Pad1.15x1.40mm_HandSolder; moved to B.Cu
- C906: renamed from C1205; moved to B.Cu
- C907: renamed from C1206; footprint Capacitor_SMD:C_1206_3216Metric_Pad1.42x1.75mm_HandSolder -> Capacitor_SMD:C_0805_2012Metric_Pad1.15x1.40mm_HandSolder; moved to B.Cu
- C908: renamed from C1207; moved to B.Cu
- C909: renamed from C1208; footprint Capacitor_SMD:C_1206_3216Metric_Pad1.42x1.75mm_HandSolder -> Capacitor_SMD:C_0805_2012Metric_Pad1.15x1.40mm_HandSolder
- C910: renamed from C1209; moved to B.Cu
- C911: renamed from C1210; footprint Capacitor_SMD:C_1206_3216Metric_Pad1.42x1.75mm_HandSolder -> Capacitor_SMD:C_0805_2012Metric_Pad1.15x1.40mm_HandSolder; moved to B.Cu
- C912: renamed from C1211; moved to B.Cu
- C913: renamed from C1212; footprint Capacitor_SMD:C_1206_3216Metric_Pad1.42x1.75mm_HandSolder -> Capacitor_SMD:C_0805_2012Metric_Pad1.15x1.40mm_HandSolder; moved to B.Cu
- C914: renamed from C1213; moved to B.Cu
- C915: renamed from C1214; footprint Capacitor_SMD:C_1206_3216Metric_Pad1.42x1.75mm_HandSolder -> Capacitor_SMD:C_0805_2012Metric_Pad1.15x1.40mm_HandSolder; moved to B.Cu
- C916: renamed from C1215; moved to B.Cu
- C917: renamed from C1216; footprint Capacitor_SMD:C_1206_3216Metric_Pad1.42x1.75mm_HandSolder -> Capacitor_SMD:C_0805_2012Metric_Pad1.15x1.40mm_HandSolder; moved to B.Cu
- D1301: renamed from D801; moved to B.Cu
- D1302: renamed from D802; moved to B.Cu
- R1102: renamed from R902; moved to B.Cu
- R1104: renamed from R904; moved to B.Cu
- R1105: renamed from R905; moved to B.Cu
- R1106: renamed from R906; moved to B.Cu
- R1108: renamed from R908; moved to B.Cu
- R1109: renamed from R909; moved to B.Cu
- R1111: renamed from R911; moved to B.Cu
- R1112: renamed from R912; moved to B.Cu
- R1113: renamed from R913; moved to B.Cu
- R1201: renamed from R1401; moved to B.Cu
- R1202: renamed from R1402; moved to B.Cu
- R1203: renamed from R1403; moved to B.Cu
- R1204: renamed from R1404; moved to B.Cu
- R1301: renamed from R801; moved to B.Cu
- R1302: renamed from R802; moved to B.Cu
- R1303: renamed from R803; moved to B.Cu
- R1304: renamed from R804; moved to B.Cu
- R1305: renamed from R805; moved to B.Cu
- R1307: renamed from R807; moved to B.Cu
- R1310: renamed from R810; moved to B.Cu
- R1311: renamed from R811; moved to B.Cu
- R1312: renamed from R839; moved to B.Cu
- R1313: renamed from R812; moved to B.Cu
- R1314: renamed from R814; moved to B.Cu
- R1315: renamed from R815; moved to B.Cu
- R1316: renamed from R816; moved to B.Cu
- R1317: renamed from R817; moved to B.Cu
- R1319: renamed from R813; moved to B.Cu
- R1320: renamed from R824; moved to B.Cu
- R1321: renamed from R825; moved to B.Cu
- R1322: renamed from R826; moved to B.Cu
- R1323: renamed from R818; moved to B.Cu
- R1324: renamed from R819; moved to B.Cu
- R1325: renamed from R820; moved to B.Cu
- R1326: renamed from R821; moved to B.Cu
- R1327: renamed from R822; moved to B.Cu
- R1328: renamed from R840; moved to B.Cu
- R1329: renamed from R829; moved to B.Cu
- R1330: renamed from R823; moved to B.Cu
- R1331: renamed from R827; moved to B.Cu
- R1332: renamed from R841; moved to B.Cu
- R1333: renamed from R828; moved to B.Cu
- R1334: renamed from R831; moved to B.Cu
- R1335: renamed from R842; moved to B.Cu
- R1336: renamed from R833; moved to B.Cu
- R1337: renamed from R834; moved to B.Cu
- R1338: renamed from R835; moved to B.Cu
- R1339: renamed from R843; moved to B.Cu
- R1340: renamed from R836; moved to B.Cu
- R1341: renamed from R837; moved to B.Cu
- R1343: renamed from R832; moved to B.Cu
- R1403: renamed from R1103; moved to B.Cu
- R1404: renamed from R1104; moved to B.Cu
- R1405: renamed from R1105; moved to B.Cu
- R1406: renamed from R1106; moved to B.Cu
- R1414: renamed from R1114; moved to B.Cu
- R1415: renamed from R1115; moved to B.Cu
- R1416: renamed from R1116; moved to B.Cu
- R1417: renamed from R1117; moved to B.Cu
- R1502: renamed from R1302; moved to B.Cu
- R1503: renamed from R1303; moved to B.Cu
- R1504: renamed from R1304; moved to B.Cu
- R801: renamed from R1001; moved to B.Cu
- R903: renamed from R1204; moved to B.Cu
- R904: renamed from R1205; moved to B.Cu
- Y1201: renamed from Y1401; moved to B.Cu
- Y1501: renamed from Y1301; moved to B.Cu
- moved C1505 364.7 mm to (114.7, 129.9)
- moved C1513 360.5 mm to (121.5, 122.0)
- moved R1501 359.2 mm to (114.7, 129.9), turned to 180 degrees
- moved C1519 356.2 mm to (124.3, 112.4), turned to 270 degrees
- moved C1514 356.1 mm to (121.5, 129.3)
- moved C1508 354.6 mm to (126.2, 127.4), turned to 90 degrees
- moved C1511 352.7 mm to (121.5, 116.6)
- moved C1503 350.9 mm to (121.8, 112.4), turned to 270 degrees
- moved C1515 349.0 mm to (119.3, 112.4), turned to 270 degrees
- moved C1512 347.8 mm to (131.2, 112.4), turned to 270 degrees
- moved C1518 346.7 mm to (131.3, 127.4), turned to 90 degrees
- moved C1504 346.1 mm to (121.5, 126.7)
- moved R1503 345.4 mm to (126.6, 112.4), turned to 270 degrees
- moved R1502 345.1 mm to (134.9, 127.4), turned to 90 degrees
- moved C1506 345.0 mm to (136.8, 112.4), turned to 270 degrees
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- renumbered C805 to C1305, C806 to C1306, C807 to C1307, C808 to C1308, C809 to C1309, C810 to C1310, C811 to C1311, C812 to C1312, C821 to C1321, C827 to C1328, C836 to C1336, C837 to C1337, C1003 to C803, C1006 to C806, D1001 to D801, D1002 to D802, D1003 to D803, J1401 to J1201, J1301 to J1501, K801 to K1301, K1101 to K1401, K1102 to K1402, K1103 to K1403, K1104 to K1404, K1105 to K1405, K1106 to K1406, K1107 to K1407, K1108 to K1408, L801 to L1301, L802 to L1302, L803 to L1303, L1001 to L801, Q1101 to Q1401, Q1102 to Q1402, Q1103 to Q1403, Q1104 to Q1404, Q1105 to Q1405, Q1106 to Q1406, Q1107 to Q1407, Q1108 to Q1408, R901 to R1101, R903 to R1103, R907 to R1107, R910 to R1110, R806 to R1306, R808 to R1308, R809 to R1309, R838 to R1318, R830 to R1342, R1101 to R1401, R1102 to R1402, R1107 to R1407, R1108 to R1408, R1109 to R1409, R1110 to R1410, R1111 to R1411, R1112 to R1412, R1113 to R1413, R1301 to R1501, R1002 to R802, R1003 to R803, R1004 to R804, R1005 to R805, R1201 to R901, R1206 to R905, U1501 to U1001, U901 to U1101, U903 to U1103, U1401 to U1201, U1402 to U1202, U801 to U1301, U802 to U1302, U803 to U1303, U804 to U1304, U805 to U1305, U806 to U1306, U815 to U1307, U807 to U1308, U809 to U1310, U810 to U1311, U811 to U1312, U812 to U1313, U814 to U1314, U1101 to U1401, U1102 to U1402, U1103 to U1403, U1301 to U1501, U1302 to U1502, U1001 to U801, U1002 to U802, U1201 to U901, U1202 to U902, U1203 to U904, U1204 to U905
Connections:
- C1104 pad 1: Net-(C904-Pad1) -> /DAC/PMU_CPH
- C1106 pad 1: Net-(C906-Pad1) -> /DAC/PMU_CLH
- C1316 pad 1: Net-(C819-Pad1) -> Net-(C1316-Pad1)
- C1317 pad 2: Net-(C820-Pad2) -> Net-(C1317-Pad2)
- C1319 pad 1: Net-(C817-Pad1) -> Net-(C1319-Pad1)
- C1320 pad 1: Net-(C817-Pad1) -> Net-(C1319-Pad1)
- C1323 pad 1: Net-(C823-Pad1) -> Net-(C1323-Pad1)
- C1325 pad 1: Net-(C826-Pad1) -> Net-(C1325-Pad1)
- C1326 pad 2: Net-(C828-Pad2) -> Net-(C1326-Pad2)
- C1329 pad 1: +3.3VF -> +3.3VP
- C1330 pad 1: +3.3VF -> +3.3VP
- C1331 pad 1: +3.3VF -> +3.3VP
- C618 pad 1: Net-(C618-Pad1) -> +15VF
- C629 pad 1: Net-(C629-Pad1) -> -15VF
- D1302 pad 1: Net-(C820-Pad2) -> Net-(C1317-Pad2)
- D1302 pad 2: (no net) -> Net-(D1302-Pad2)
- D1302 pad 3: Net-(D802-Pad3) (its old number) -> (no net)
- D1302 pad 4: Net-(C820-Pad2) -> (no net)
- D1302 pad 5: (no net) -> Net-(C1317-Pad2)
- D1302 pad 6: Net-(D802-Pad3) (its old number) -> Net-(D1302-Pad2)
- J201 pad A5: Net-(J201-PadA5) -> /Connector/C
- J201 pad C5: Net-(J201-PadA5) -> /Connector/C
- R1103 pad 1: Net-(C904-Pad1) -> /DAC/PMU_CPH
- R1110 pad 1: Net-(C906-Pad1) -> /DAC/PMU_CLH
- R1111 pad 2: (no net) -> /DAC/DAC_RSTSEL
- R1315 pad 2: Net-(D802-Pad3) (its old number) -> Net-(D1302-Pad2)
- R1316 pad 1: Net-(C820-Pad2) -> Net-(C1317-Pad2)
- R1317 pad 2: Net-(C819-Pad1) -> Net-(C1316-Pad1)
- R1322 pad 2: Net-(C819-Pad1) -> Net-(C1316-Pad1)
- R1323 pad 2: Net-(C817-Pad1) -> Net-(C1319-Pad1)
- R1325 pad 2: Net-(R820-Pad2) -> Net-(R1325-Pad2)
- R1327 pad 1: Net-(C823-Pad1) -> Net-(C1323-Pad1)
- R1329 pad 1: Net-(C826-Pad1) -> Net-(C1325-Pad1)
- R1331 pad 1: Net-(R820-Pad2) -> Net-(R1325-Pad2)
- R1331 pad 2: Net-(R827-Pad2) -> Net-(R1331-Pad2)
- R1333 pad 2: Net-(R827-Pad2) -> Net-(R1331-Pad2)
- R1336 pad 1: Net-(C828-Pad2) -> Net-(C1326-Pad2)
- R1337 pad 2: Net-(C828-Pad2) -> Net-(C1326-Pad2)
- R1341 pad 1: Net-(C828-Pad2) -> Net-(C1326-Pad2)
- U1103 pad 8: (no net) -> /DAC/DAC_SDO
- U1201 pad 20: (no net) -> /MCU2/MCU3_NSS
- U1201 pad 51: (no net) -> /MCU2/MCU3_SCLK
- U1201 pad 52: (no net) -> /MCU2/MCU3_MISO
- U1201 pad 53: (no net) -> /MCU2/MCU3_MOSI
- U1310 pad 8: Net-(U809-Pad8) -> Net-(U1309-Pad3)
- U1311 pad 1: Net-(R820-Pad2) -> Net-(C1316-Pad1)
- U1311 pad 2: Net-(R827-Pad2) -> Net-(C1316-Pad1)
- U1311 pad 3: Net-(U809-Pad8) -> Net-(C1317-Pad2)
- U1311 pad 5: Net-(C823-Pad1) -> Net-(C1325-Pad1)
- U1311 pad 6: Net-(C817-Pad1) -> Net-(C1326-Pad2)
- U1311 pad 7: Net-(C817-Pad1) -> /AC source/V_OFFSET
- U1313 pad 3: Net-(D802-Pad3) (its old number) -> Net-(D1302-Pad2)
- U1403 pad 1: (no net) -> /DAC/PMU_CPH
- U1403 pad 58: (no net) -> /ADC/PMU_MEASOUT
- U1403 pad 63: (no net) -> /DAC/PMU_CLH
- U1501 pad 102: (no net) -> /DAC/DAC_RSTSEL
- U1501 pad 103: (no net) -> /DAC/DAC_~LDAC
- U1501 pad 104: (no net) -> /DAC/DAC_~RESET
- U1501 pad 110: (no net) -> /DAC/DAC_~SYNC
- U1501 pad 112: (no net) -> /DAC/DAC_SDO
- U1501 pad 114: /DAC/DAC_~LDAC -> (no net)
- U1501 pad 123: (no net) -> /MCU2/MCU3_MOSI
- U1501 pad 124: (no net) -> /MCU2/MCU3_MISO
- U1501 pad 125: (no net) -> /MCU2/MCU3_NSS
- U1501 pad 126: (no net) -> /MCU2/MCU3_SCLK
- U1501 pad 140: /ADC/ADC_MUX_~SYNC -> (no net)
- U1501 pad 31: Net-(U1301-Pad31) -> AGNDF
- U1501 pad 32: Net-(U1301-Pad31) -> /MCU2/MCU_VDDA
- U1501 pad 33: (no net) -> /MCU2/MCU_VDDA
- U1501 pad 46: (no net) -> /ADC/ADC_CONVST
- U1501 pad 73: (no net) -> /ADC/ADC_MUX_~SYNC
- U301 pad 104: (no net) -> /MCU1/MCU_DEFAULT
- U603 pad 3: Net-(C618-Pad1) -> +15VF
- U607 pad 3: Net-(C629-Pad1) -> -15VF
- U901 pad 1: Net-(U1201-Pad1) -> Net-(U901-Pad1)
- U901 pad 8: Net-(U1201-Pad1) -> Net-(U901-Pad1)
- U904 pad 16: (no net) -> +3.3VF
- U904 pad 17: (no net) -> AGNDF
- U904 pad 19: (no net) -> /ADC/ADC_CONVST
- U904 pad 6: Net-(U1201-Pad1) -> Net-(U901-Pad1)
- U904 pad 8: Net-(R1203-Pad2) -> Net-(U901-Pad1)
- U904 pad 9: Net-(U1201-Pad1) -> Net-(U901-Pad1)

Commit message: PCB design
Parts:
- added C1343: 100n, Capacitor_SMD:C_0603_1608Metric_Pad1.05x0.95mm_HandSolder, B.Cu at (122.0, 78.7)
- C1336, C1337, R305: moved to B.Cu
- moved TP601 69.8 mm to (149.2, 47.1)
- moved TP701 4.95 mm to (154.8, 47.1)
- moved U502 3.72 mm to (200.5, 122.7), turned to 270 degrees
- moved J1501 3.14 mm to (112.4, 120.1)
- moved C1505 3.14 mm to (113.0, 127.3)
- moved R1501 3.14 mm to (113.0, 127.3)
- moved C801 2.29 mm to (184.0, 87.2)
- moved C802 2.29 mm to (186.3, 87.2)
- moved D803 2.29 mm to (211.7, 87.5)
- moved L801 2.29 mm to (211.8, 87.5)
- moved R801 2.29 mm to (200.9, 88.8)
- moved U801 2.29 mm to (200.8, 88.0)
- moved C803 2.29 mm to (196.1, 87.0)
- moved C804 2.29 mm to (196.1, 91.7)
- moved C805 2.29 mm to (200.9, 86.4)
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Other:
- copper layers 4 -> 6
- net class Signals added: clearance 0.127, trace_width 0.127, via_dia 0.4, via_drill 0.2
- rule trace_min: 0.2 -> 0.1
- rule via_min_drill: 0.3 -> 0.2
