File: hardware/project/ETH1CPMU1/ETH1CPMU1.kicad_pcb (KiCad board)
At the start: 6 copper layers, 160 x 100 mm, 472 parts, among them J1201 Conn_02x05, J1501 Conn_02x05, J201 C64AC, J301 Conn_02x05, J302 Conn_02x01, K1301 TQ2SA-5V, K1401 HE3621A0510, K1402 HE3621A0510, K1403 HE3621A0510, K1404 HE3621A0510, K1405 HE3621A0510, K1406 HE3621A0510, K1407 HE3621A0510, K1408 HE3621A0510, Q1401 BC847, Q1402 BC847, Q1403 BC847, Q1404 BC847, Q1405 BC847, Q1406 BC847, Q1407 BC847, Q1408 BC847, Q501 IRFR5410, U1001 ADuM3151, U1101 REF192, U1102 TL072, U1103 AD5689BRUZ, U1201 STM32F413RGT6Tx, U1202 24LC08B-E/MS, U1301 AD5453YRMZ, U1302 LT1468, U1303 LT1468, U1304 AD9835, U1305 ECS-3225SMV-500-GP-TR, U1306 74AHCT1G08, U1307 TXB0104D, U1308 REF192, U1309 TL072, U1310 DG408DY, U1311 TL072, U1312 ADS7818, U1313 AD5689BRUZ, U1314 TL072, U1401 THS6012, U1402 DG419LEUA, U1403 AD5520, U1501 STM32H743ZI, U1502 24LC08B-E/MS, U301 STM32F765ZGT6, U302 24LC08B-E/MS, U401 LC03-3.3, U402 LAN8742A, U403 LC03-3.3, U501 LM1117IMP-3.3/NOPB, U502 TSR1-2450, U503 MAX5902, U601 THL15-2415WI, U602 LM1117IMP-3.3/NOPB, U603 MC7815BD2TG, U604 LM1117IMP-3.3/NOPB, U605 TSR2-2450, U606 LT8330_S6, U607 MC7915BD2TG, U608 LM1117IMP-5.0/NOPB, U609 TSR1-2490, U610 LT8330_S6, U701 REF02AU, U702 AD8676, U703 AD8676, U704 AD8675, U705 AD5791, U801 74AC125, U802 ADuM5402, U901 INA159, U902 ADG1414BRU, U903 INA159, U904 ADS8363, U905 INA159, Y1201 NX3225GD-8MHZ-STD-CRA-3, Y1501 NX3225GD-8MHZ-STD-CRA-3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

Commit message: PCB design
Parts:
- removed the C1110 at (164.0, 97.2)
- removed the R1104 at (158.9, 100.1)
- removed R1105: 10k, Resistor_SMD:R_0603_1608Metric_Pad1.05x0.95mm_HandSolder
- removed R1108, R1111, R1112: R, Resistor_SMD:R_0603_1608Metric_Pad1.05x0.95mm_HandSolder
- removed the U1102 at (169.5, 97.2)
- removed U1103: AD5689BRUZ, Package_SO:TSSOP-16_4.4x5mm_P0.65mm
- removed the U703 at (169.3, 75.1)
- added C1242: 10p, Capacitor_SMD:C_0603_1608Metric_Pad1.05x0.95mm_HandSolder, B.Cu at (138.8, 50.8)
- added C1401: C, Capacitor_SMD:C_0603_1608Metric_Pad1.05x0.95mm_HandSolder, F.Cu at (175.3, 80.1)
- added C1402: C, Capacitor_SMD:C_0603_1608Metric_Pad1.05x0.95mm_HandSolder, F.Cu at (175.1, 61.7)
- added C1403: C, Capacitor_SMD:C_0603_1608Metric_Pad1.05x0.95mm_HandSolder, F.Cu at (175.1, 98.6)
- added C1404: 100n, Capacitor_SMD:C_0603_1608Metric_Pad1.05x0.95mm_HandSolder, B.Cu at (168.9, 97.0)
- added C1405: 100n, Capacitor_SMD:C_0603_1608Metric_Pad1.05x0.95mm_HandSolder, B.Cu at (168.9, 59.9)
- added C1406: 100n, Capacitor_SMD:C_0603_1608Metric_Pad1.05x0.95mm_HandSolder, B.Cu at (168.9, 78.4)
- added C1407: 100n, Capacitor_SMD:C_0603_1608Metric_Pad1.05x0.95mm_HandSolder, B.Cu at (171.4, 97.0)
- added C1408: 100n, Capacitor_SMD:C_0603_1608Metric_Pad1.05x0.95mm_HandSolder, B.Cu at (171.4, 59.9)
- added C1409: 100n, Capacitor_SMD:C_0603_1608Metric_Pad1.05x0.95mm_HandSolder, B.Cu at (171.4, 78.4)
- added C1410: 10p, Capacitor_SMD:C_0603_1608Metric_Pad1.05x0.95mm_HandSolder, B.Cu at (178.1, 83.1)
- added C1411: 10p, Capacitor_SMD:C_0603_1608Metric_Pad1.05x0.95mm_HandSolder, B.Cu at (178.1, 86.6)
- added C1412: 10p, Capacitor_SMD:C_0603_1608Metric_Pad1.05x0.95mm_HandSolder, B.Cu at (178.1, 90.2)
- added C1413: 10p, Capacitor_SMD:C_0603_1608Metric_Pad1.05x0.95mm_HandSolder, B.Cu at (178.1, 93.7)
- added C1414: 10p, Capacitor_SMD:C_0603_1608Metric_Pad1.05x0.95mm_HandSolder, B.Cu at (178.1, 75.9)
- added C1415: 10p, Capacitor_SMD:C_0603_1608Metric_Pad1.05x0.95mm_HandSolder, B.Cu at (178.1, 79.5)
- added C1416: 100n, Capacitor_SMD:C_0603_1608Metric_Pad1.05x0.95mm_HandSolder, B.Cu at (168.9, 70.4)
- added C1417: 100n, Capacitor_SMD:C_0603_1608Metric_Pad1.05x0.95mm_HandSolder, B.Cu at (171.4, 70.4)
- added C1508: 220n, Capacitor_SMD:C_0603_1608Metric_Pad1.05x0.95mm_HandSolder, B.Cu at (152.3, 99.6)
- added C1509: 220n, Capacitor_SMD:C_0603_1608Metric_Pad1.05x0.95mm_HandSolder, B.Cu at (152.3, 97.0)
- added C1512: 1n, Capacitor_SMD:C_0603_1608Metric_Pad1.05x0.95mm_HandSolder, B.Cu at (165.0, 101.2)
- added C1513: 1n, Capacitor_SMD:C_0603_1608Metric_Pad1.05x0.95mm_HandSolder, B.Cu at (165.0, 96.5)
- added Q1201: BC847, Package_TO_SOT_SMD:SOT-23, B.Cu at (135.4, 50.8)
- added Q1401: BC847, Package_TO_SOT_SMD:SOT-23, F.Cu at (178.8, 83.1)
- added Q1402: BC847, Package_TO_SOT_SMD:SOT-23, F.Cu at (178.8, 86.6)
- added Q1403: BC847, Package_TO_SOT_SMD:SOT-23, F.Cu at (178.8, 90.2)
- added Q1404: BC847, Package_TO_SOT_SMD:SOT-23, F.Cu at (178.8, 93.7)
- added Q1405: BC847, Package_TO_SOT_SMD:SOT-23, F.Cu at (178.8, 75.9)
- added Q1406: BC847, Package_TO_SOT_SMD:SOT-23, F.Cu at (178.8, 79.5)
- added R1241: 10k, Resistor_SMD:R_0603_1608Metric_Pad1.05x0.95mm_HandSolder, B.Cu at (132.0, 50.8)
- added R1401: R, Resistor_SMD:R_0603_1608Metric_Pad1.05x0.95mm_HandSolder, F.Cu at (175.3, 76.6)
- added R1402: R, Resistor_SMD:R_0603_1608Metric_Pad1.05x0.95mm_HandSolder, F.Cu at (175.1, 58.2)
- added R1403: R, Resistor_SMD:R_0603_1608Metric_Pad1.05x0.95mm_HandSolder, F.Cu at (175.1, 95.0)
- added R1404: 100k, Resistor_SMD:R_0603_1608Metric_Pad1.05x0.95mm_HandSolder, F.Cu at (173.2, 83.7)
- added R1405: 100k, Resistor_SMD:R_0603_1608Metric_Pad1.05x0.95mm_HandSolder, F.Cu at (169.8, 83.7)
- added R1406: 100k, Resistor_SMD:R_0603_1608Metric_Pad1.05x0.95mm_HandSolder, F.Cu at (173.2, 65.3)
- added R1407: 100k, Resistor_SMD:R_0603_1608Metric_Pad1.05x0.95mm_HandSolder, F.Cu at (169.8, 65.3)
- added R1408: 100k, Resistor_SMD:R_0603_1608Metric_Pad1.05x0.95mm_HandSolder, F.Cu at (173.4, 102.1)
- added R1409: 100k, Resistor_SMD:R_0603_1608Metric_Pad1.05x0.95mm_HandSolder, F.Cu at (169.8, 102.1)
- added R1410: 50, Resistor_SMD:R_0603_1608Metric_Pad1.05x0.95mm_HandSolder, F.Cu at (175.3, 90.4)
- added R1411: 50, Resistor_SMD:R_0603_1608Metric_Pad1.05x0.95mm_HandSolder, F.Cu at (175.1, 72.1)
- added R1412: 100k, Resistor_SMD:R_0603_1608Metric_Pad1.05x0.95mm_HandSolder, F.Cu at (175.3, 86.9)
- added R1413: 100k, Resistor_SMD:R_0603_1608Metric_Pad1.05x0.95mm_HandSolder, F.Cu at (175.1, 68.6)
- added R1414: 10k, Resistor_SMD:R_0603_1608Metric_Pad1.05x0.95mm_HandSolder, B.Cu at (179.6, 83.1)
- added R1415: 10k, Resistor_SMD:R_0603_1608Metric_Pad1.05x0.95mm_HandSolder, B.Cu at (179.6, 86.6)
- added R1416: 10k, Resistor_SMD:R_0603_1608Metric_Pad1.05x0.95mm_HandSolder, B.Cu at (179.6, 90.2)
- added R1417: 10k, Resistor_SMD:R_0603_1608Metric_Pad1.05x0.95mm_HandSolder, B.Cu at (179.6, 93.7)
- added R1418: 10k, Resistor_SMD:R_0603_1608Metric_Pad1.05x0.95mm_HandSolder, B.Cu at (179.6, 75.9)
- added R1419: 10k, Resistor_SMD:R_0603_1608Metric_Pad1.05x0.95mm_HandSolder, B.Cu at (179.6, 79.5)
- added R1503: 1k, Resistor_SMD:R_0603_1608Metric_Pad1.05x0.95mm_HandSolder, F.Cu at (152.3, 99.6)
- added R1504: 1k, Resistor_SMD:R_0603_1608Metric_Pad1.05x0.95mm_HandSolder, F.Cu at (152.3, 97.0)
- added R1509: 24k9, Resistor_SMD:R_0603_1608Metric_Pad1.05x0.95mm_HandSolder, F.Cu at (156.6, 102.0)
- added R1510: 33k2, Resistor_SMD:R_0603_1608Metric_Pad1.05x0.95mm_HandSolder, F.Cu at (165.0, 99.7)
- added R1511: 24k9, Resistor_SMD:R_0603_1608Metric_Pad1.05x0.95mm_HandSolder, B.Cu at (156.6, 102.0)
- added R1512: 33k2, Resistor_SMD:R_0603_1608Metric_Pad1.05x0.95mm_HandSolder, F.Cu at (165.0, 95.0)
- added R1515: 100k, Resistor_SMD:R_0603_1608Metric_Pad1.05x0.95mm_HandSolder, F.Cu at (165.0, 101.2)
- added R1516: 100k, Resistor_SMD:R_0603_1608Metric_Pad1.05x0.95mm_HandSolder, F.Cu at (165.0, 96.5)
- added R906: 0, Resistor_SMD:R_0603_1608Metric_Pad1.05x0.95mm_HandSolder, F.Cu at (161.0, 87.4)
- added R907: 0, Resistor_SMD:R_0603_1608Metric_Pad1.05x0.95mm_HandSolder, F.Cu at (164.8, 87.4)
- added U1401: PGA103, Package_SO:SOIC-8_3.9x4.9mm_P1.27mm, F.Cu at (170.8, 78.4)
- added U1402: PGA103, Package_SO:SOIC-8_3.9x4.9mm_P1.27mm, F.Cu at (170.8, 59.9)
- added U1403: PGA103, Package_SO:SOIC-8_3.9x4.9mm_P1.27mm, F.Cu at (170.8, 96.8)
- added U1404: OPA602, Package_SO:SOIC-8_3.9x4.9mm_P1.27mm, F.Cu at (170.8, 88.6)
- added U1405: OPA602, Package_SO:SOIC-8_3.9x4.9mm_P1.27mm, F.Cu at (170.8, 70.4)
- added U1502: TL074, Package_SO:SOIC-14_3.9x8.7mm_P1.27mm, F.Cu at (158.9, 95.6)
- added U1503: AD5324, Package_SO:MSOP-10_3x3mm_P0.5mm, F.Cu at (146.2, 100.5)
- added U702: AD8676, Package_SO:SOIC-8_3.9x4.9mm_P1.27mm, F.Cu at (162.9, 72.8)
- C1212: renamed from C1336; moved to F.Cu
- C1215: renamed from C1337; moved to F.Cu
- C1302: renamed from C1415; moved to B.Cu
- C1315: renamed from C1423; moved to B.Cu
- R1505: renamed from R1102; moved to F.Cu
- R1506: renamed from R1106; moved to F.Cu
- moved C1312 20.2 mm to (170.8, 45.0), turned to 0 degrees
- moved R1505 19.9 mm to (152.3, 102.0), turned to 180 degrees
- moved C1302 19.3 mm to (170.8, 46.9), turned to 0 degrees
- moved R1507 18.5 mm to (152.3, 102.0), turned to 180 degrees
- moved C1511 14.5 mm to (160.8, 102.0)
- moved R1514 14.5 mm to (160.8, 102.0)
- moved C1501 14.4 mm to (158.9, 94.7), turned to 0 degrees
- moved C1506 13.4 mm to (152.3, 92.2)
- moved R1501 13.4 mm to (152.3, 92.2)
- moved C1316 12.1 mm to (165.7, 55.1), turned to 0 degrees
- moved C1507 11.7 mm to (152.3, 94.6)
- moved R1502 11.7 mm to (152.3, 94.6)
- moved C1504 10.4 mm to (146.2, 99.4), turned to 0 degrees
- moved TP701 8.83 mm to (149.1, 53.8)
- moved C908 8.52 mm to (161.2, 78.0)
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- renumbered C1205 to C1101, C1206 to C1102, C1207 to C1103, C1208 to C1104, C1209 to C1105, C1210 to C1106, C1211 to C1107, C1203 to C1108, C1204 to C1109, C1201 to C1110, C1202 to C1111, C1329 to C1201, C1314 to C1202, C1330 to C1203, C1331 to C1204, C1315 to C1205, C1332 to C1206, C1333 to C1207, C1334 to C1208, C1335 to C1209, C1316 to C1210, C1325 to C1211, C1317 to C1213, C1304 to C1214, C1313 to C1216, C1326 to C1217, C1338 to C1218, C1309 to C1219, C1305 to C1220, C1310 to C1221, C1306 to C1222, C1311 to C1223, C1307 to C1224, C1312 to C1225, C1339 to C1226, C1340 to C1227, C1308 to C1228, C1341 to C1229, C1327 to C1230, C1342 to C1231, C1303 to C1232, C1321 to C1233, C1343 to C1234, C1322 to C1235, C1319 to C1236, C1320 to C1237, C1328 to C1238, C1301 to C1239, C1323 to C1240, C1324 to C1241, C1318 to C1243, C1302 to C1244, C1414 to C1301, C1416 to C1303, C1417 to C1304, C1418 to C1305, C1409 to C1306, C1410 to C1307, C1411 to C1308, C1419 to C1309, C1420 to C1310, C1421 to C1311, C1422 to C1312, C1404 to C1313, C1401 to C1314, C1424 to C1316, C1425 to C1317, C1426 to C1318, C1403 to C1319, C1405 to C1320, C1407 to C1321, C1412 to C1322, C1402 to C1323, C1406 to C1324, C1408 to C1325, C1413 to C1326, C1107 to C1501, C1102 to C1502, C1108 to C1503, C1109 to C1504, C1103 to C1505, C1101 to C1506, C1105 to C1507, C1104 to C1510, C1106 to C1511, C1508 to C1601, C1501 to C1602, C1509 to C1603, C1502 to C1604, C1510 to C1605, C1503 to C1606, C1504 to C1607, C1511 to C1608, C1512 to C1609, C1506 to C1610, C1513 to C1611, C1514 to C1612, C1515 to C1613, C1516 to C1614, C1517 to C1615, C1518 to C1616, C1519 to C1617, C1507 to C1618, C1505 to C1619, C307 to C301, C308 to C302, C309 to C303, C301 to C304, C310 to C305, C302 to C306, C303 to C307, C311 to C308, C304 to C309, C312 to C310, C306 to C311, C313 to C312, C314 to C313, C315 to C314, C316 to C315, C317 to C316, C318 to C317, C319 to C318, C320 to C319, C321 to C320, C305 to C321, C413 to C401, C401 to C402, C408 to C403, C414 to C404, C402 to C405, C409 to C406, C403 to C407, C404 to C408, C405 to C409, C406 to C410, C407 to C411, C410 to C412, C412 to C413, C411 to C414, C602 to C601, C614 to C602, C625 to C603, C603 to C604, C619 to C605, C630 to C606, C620 to C608, C601 to C609, C606 to C610, C615 to C611, C626 to C612, C604 to C613, C616 to C614, C627 to C615, C617 to C616, C628 to C617, C629 to C619, C608 to C620, C609 to C621, C621 to C622, C610 to C623, C622 to C624, C611 to C625, C612 to C626, C623 to C627, C605 to C628, C613 to C629, C624 to C630, C703 to C701, C711 to C702, C704 to C703, C712 to C704, C713 to C706, C706 to C707, C714 to C708, C707 to C709, C715 to C710, C708 to C711, C716 to C712, C709 to C713, C717 to C714, C710 to C715, C718 to C716, C701 to C717, C702 to C718, C904 to C901, C908 to C902, C905 to C903, C909 to C904, C906 to C905, C910 to C906, C911 to C908, C912 to C909, C913 to C910, C914 to C911, C915 to C912, C916 to C913, C901 to C914, C902 to C915, C903 to C916, D1302 to D1201, D1301 to D1202, D502 to D501, D503 to D502, D501 to D503, D602 to D601, D601 to D602, D802 to D801, D801 to D802, FB1501 to FB1601, J1201 to J1101, J1501 to J1601, J302 to J301, J301 to J302, K1301 to K1201, K1403 to K1301, K1404 to K1302, K1405 to K1303, K1406 to K1304, K1407 to K1305, K1408 to K1306, K1401 to K1307, K1402 to K1308, L1301 to L1201, L1302 to L1202, L1303 to L1203, L604 to L603, L603 to L604, Q1402 to Q1301, Q1403 to Q1302, Q1405 to Q1303, Q1407 to Q1304, Q1401 to Q1305, Q1404 to Q1306, Q1406 to Q1307, Q1408 to Q1308, R1203 to R1101, R1204 to R1102, R1202 to R1103, R1201 to R1104, R1320 to R1201, R1338 to R1202, R1334 to R1203, R1340 to R1204, R1321 to R1205, R1311 to R1206, R1313 to R1207, R1314 to R1208, R1305 to R1209, R1315 to R1210, R1316 to R1211, R1329 to R1212, R1310 to R1213, R1336 to R1214, R1341 to R1215, R1337 to R1216, R1308 to R1217, R1317 to R1218, R1322 to R1219, R1328 to R1220, R1332 to R1221, R1309 to R1222, R1339 to R1223, R1318 to R1224, R1335 to R1225, R1306 to R1226, R1333 to R1227, R1312 to R1228, R1331 to R1229, R1342 to R1230, R1303 to R1231, R1325 to R1232, R1343 to R1233, R1330 to R1234, R1326 to R1235, R1301 to R1236, R1307 to R1237, R1327 to R1238, R1304 to R1239, R1323 to R1240, R1302 to R1242, R1319 to R1243, R1324 to R1244, R1402 to R1301, R1407 to R1302, R1401 to R1303, R1408 to R1304, R1409 to R1305, R1410 to R1306, R1411 to R1307, R1412 to R1308, R1413 to R1309, R1404 to R1310, R1405 to R1311, R1414 to R1312, R1416 to R1313, R1403 to R1314, R1406 to R1315, R1415 to R1316, R1417 to R1317, R1101 to R1501, R1107 to R1502, R1109 to R1507, R1113 to R1508, R1103 to R1513, R1110 to R1514, R1503 to R1601, R1504 to R1602, R1502 to R1603, R1501 to R1604, R305 to R303, R303 to R305, R405 to R401, R406 to R402, R407 to R403, R408 to R404, R412 to R405, R417 to R406, R418 to R407, R419 to R408, R420 to R409, R421 to R410, R413 to R411, R409 to R412, R414 to R413, R415 to R414, R401 to R415, R402 to R416, R403 to R417, R404 to R418, R416 to R419, R410 to R420, R411 to R421, R603 to R602, R605 to R603, R607 to R604, R602 to R605, R604 to R606, R606 to R607, R707 to R702, R705 to R703, R703 to R705, R702 to R707, R802 to R801, R803 to R802, R801 to R803, R905 to R903, R903 to R904, R904 to R905, U1201 to U1101, U1202 to U1102, U1305 to U1201, U1308 to U1202, U1306 to U1203, U1313 to U1204, U1304 to U1205, U1311 to U1206, U1309 to U1207, U1307 to U1208, U1310 to U1209, U1301 to U1210, U1314 to U1211, U1302 to U1212, U1303 to U1213, U1312 to U1214, U1402 to U1301, U1403 to U1302, U1401 to U1303, U1101 to U1501, U1502 to U1601, U1501 to U1602, U302 to U301, U301 to U302, U402 to U401, U401 to U402, U503 to U501, U501 to U503, U606 to U601, U610 to U602, U601 to U603, U603 to U604, U607 to U605, U605 to U606, U609 to U607, U602 to U608, U604 to U609, U608 to U610, U702 to U703, U705 to U704, U704 to U705, U802 to U801, U801 to U802, U904 to U901, U901 to U902, U905 to U904, U902 to U905, Y1201 to Y1101, Y1501 to Y1601
Connections:
- U1101 pad 37: (no net) -> /AC source/AC_RELAY
- U1302 pad 58: /ADC/PMU_MEASOUT -> /PGA/PMU_MEASOUT
- U1302 pad 60: /ADC/PMU_MEASIOUT -> /PGA/PMU_MEASIOUT
- U1302 pad 61: /ADC/PMU_MEASVOUT -> /PGA/PMU_MEASVOUT
- U1602 pad 102: /DAC/DAC_RSTSEL -> (no net)
- U1602 pad 103: /DAC/DAC_~LDAC -> (no net)
- U1602 pad 104: /DAC/DAC_~RESET -> (no net)
- U1602 pad 112: /DAC/DAC_SDO -> (no net)
- U1602 pad 113: /DAC/DAC_SDIN -> /DAC/DAC_DIN
- U1602 pad 114: (no net) -> /MCU2/G1A0_CTR
- U1602 pad 115: (no net) -> /MCU2/G1A1_CTR
- U1602 pad 116: (no net) -> /MCU2/G2A0_CTR
- U1602 pad 117: (no net) -> /MCU2/G2A1_CTR
- U1602 pad 118: (no net) -> /MCU2/G3A0_CTR
- U1602 pad 119: (no net) -> /MCU2/G3A1_CTR
- U903 pad 3: /ADC/PMU_MEASOUT -> /ADC/PMU_MEAS_GAIN
- U905 pad 13: /ADC/PMU_MEASIOUT -> /ADC/PMU_MEASI_GAIN
- U905 pad 6: /ADC/PMU_MEASVOUT -> /ADC/PMU_MEASV_GAIN
Other:
- board text added: "1"
- board text added: "2"
- board text added: "3"
- board text added: "4"
- board text added: "5"
- board text added: "6"

Commit message: PCB design
Parts:
- moved C1314 2.09 mm to (170.2, 53.3)
- moved R1303 2.09 mm to (170.2, 53.3)
- moved R1301 2.09 mm to (170.2, 49.8)
- moved C1312 1.53 mm to (169.3, 45.1)
- moved C1302 1.52 mm to (169.3, 46.9)
- moved C1512 1.02 mm to (165.0, 102.2)
- moved R1515 1.02 mm to (165.0, 102.2)
- moved C1513 0.89 mm to (165.0, 97.4)
- moved R1516 0.89 mm to (165.0, 97.4)
- moved C1510 0.76 mm to (165.0, 92.6)
- moved R1513 0.76 mm to (165.0, 92.6)
- moved C604 0.52 mm to (87.8, 131.4)
- moved C601 0.52 mm to (87.8, 134.6)
- moved L601 0.52 mm to (87.8, 132.1)
- moved C1612 0.38 mm to (123.7, 127.9)
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Other:
- board text added: "ETH1CPMU1 PROTOTYPE V 1.0 DEFAULT IP: 192.168.1.123 DEFAULT TCP/IP PORT: 2000 SHORT J301 FOR DEFAULT CONFIGURATION"

Commit message: PCB design
Parts:
- added C1418: 100n, Capacitor_SMD:C_0603_1608Metric_Pad1.05x0.95mm_HandSolder, B.Cu at (169.8, 88.6)
- added C1419: 100n, Capacitor_SMD:C_0603_1608Metric_Pad1.05x0.95mm_HandSolder, B.Cu at (172.3, 88.6)
- R1219: moved to F.Cu
- moved C313 23.5 mm to (157.1, 131.2), turned to 270 degrees
- moved FB301 19.2 mm to (159.5, 112.6), turned to 270 degrees
- moved C307 18.1 mm to (160.5, 128.3)
- moved C320 18.1 mm to (158.8, 109.7), turned to 180 degrees
- moved C316 16.0 mm to (156.8, 112.6), turned to 270 degrees
- moved C319 15.7 mm to (176.8, 112.6), turned to 270 degrees
- moved C309 15.3 mm to (173.7, 127.6), turned to 90 degrees
- moved C312 13.1 mm to (167.5, 122.9)
- moved R302 11.4 mm to (160.5, 121.9), turned to 0 degrees
- moved R304 11.2 mm to (175.5, 116.0), turned to 180 degrees
- moved R301 10.7 mm to (160.5, 120.4), turned to 0 degrees
- moved C321 10.4 mm to (185.7, 116.5)
- moved R305 10.4 mm to (185.7, 116.5)
- moved Y301 8.70 mm to (165.6, 112.5), turned to 180 degrees
- moved C310 8.38 mm to (167.5, 119.4), turned to 90 degrees
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Connections:
- D1201 pad 3: (no net) -> Net-(D1201-Pad3)
- D1201 pad 4: (no net) -> Net-(D1201-Pad4)
- J1101 pad 6: (no net) -> Net-(J1101-Pad6)
- J1101 pad 7: (no net) -> Net-(J1101-Pad7)
- J1101 pad 8: (no net) -> Net-(J1101-Pad8)
- J1101 pad 9: (no net) -> Net-(J1101-Pad9)
- J1601 pad 6: (no net) -> Net-(J1601-Pad6)
- J1601 pad 7: (no net) -> Net-(J1601-Pad7)
- J1601 pad 8: (no net) -> Net-(J1601-Pad8)
- J1601 pad 9: (no net) -> Net-(J1601-Pad9)
- J201 pad A1: (no net) -> Net-(J201-PadA1)
- J201 pad A10: (no net) -> Net-(J201-PadA10)
- J201 pad A11: (no net) -> Net-(J201-PadA11)
- J201 pad A12: (no net) -> Net-(J201-PadA12)
- J201 pad A13: (no net) -> Net-(J201-PadA13)
- J201 pad A14: (no net) -> Net-(J201-PadA14)
- J201 pad A15: (no net) -> Net-(J201-PadA15)
- J201 pad A17: (no net) -> Net-(J201-PadA17)
- J201 pad A19: (no net) -> Net-(J201-PadA19)
- J201 pad A23: (no net) -> Net-(J201-PadA23)
- J201 pad A24: (no net) -> Net-(J201-PadA24)
- J201 pad A25: (no net) -> Net-(J201-PadA25)
- J201 pad A26: (no net) -> Net-(J201-PadA26)
- J201 pad A29: (no net) -> Net-(J201-PadA29)
- J201 pad A30: (no net) -> Net-(J201-PadA30)
- J201 pad A8: (no net) -> Net-(J201-PadA8)
- J201 pad A9: (no net) -> Net-(J201-PadA9)
- J201 pad C1: (no net) -> Net-(J201-PadC1)
- J201 pad C10: (no net) -> Net-(J201-PadC10)
- J201 pad C11: (no net) -> Net-(J201-PadC11)
- J201 pad C12: (no net) -> Net-(J201-PadC12)
- J201 pad C13: (no net) -> Net-(J201-PadC13)
- J201 pad C14: (no net) -> Net-(J201-PadC14)
- J201 pad C15: (no net) -> Net-(J201-PadC15)
- J201 pad C17: (no net) -> Net-(J201-PadC17)
- J201 pad C19: (no net) -> Net-(J201-PadC19)
- J201 pad C23: (no net) -> Net-(J201-PadC23)
- J201 pad C24: (no net) -> Net-(J201-PadC24)
- J201 pad C25: (no net) -> Net-(J201-PadC25)
- J201 pad C26: (no net) -> Net-(J201-PadC26)
- J201 pad C29: (no net) -> Net-(J201-PadC29)
- J201 pad C30: (no net) -> Net-(J201-PadC30)
- J201 pad C8: (no net) -> Net-(J201-PadC8)
- J201 pad C9: (no net) -> Net-(J201-PadC9)
- J302 pad 7: (no net) -> Net-(J302-Pad7)
- J302 pad 9: (no net) -> Net-(J302-Pad9)
- K1201 pad 5: (no net) -> Net-(K1201-Pad5)
- K1201 pad 6: (no net) -> Net-(K1201-Pad6)
- U1101 pad 10: (no net) -> Net-(U1101-Pad10)
- U1101 pad 2: (no net) -> Net-(U1101-Pad2)
- U1101 pad 24: (no net) -> Net-(U1101-Pad24)
- U1101 pad 25: (no net) -> Net-(U1101-Pad25)
- U1101 pad 3: (no net) -> Net-(U1101-Pad3)
- U1101 pad 35: (no net) -> Net-(U1101-Pad35)
- U1101 pad 36: (no net) -> Net-(U1101-Pad36)
- U1101 pad 4: (no net) -> Net-(U1101-Pad4)
- U1101 pad 44: (no net) -> Net-(U1101-Pad44)
- U1101 pad 45: (no net) -> Net-(U1101-Pad45)
- U1101 pad 54: (no net) -> Net-(U1101-Pad54)
- U1101 pad 55: (no net) -> Net-(U1101-Pad55)
- U1101 pad 56: (no net) -> Net-(U1101-Pad56)
- U1101 pad 61: (no net) -> Net-(U1101-Pad61)
- U1101 pad 8: (no net) -> Net-(U1101-Pad8)
- U1101 pad 9: (no net) -> Net-(U1101-Pad9)
- U1202 pad 1: (no net) -> Net-(U1202-Pad1)
- U1202 pad 5: (no net) -> Net-(U1202-Pad5)
- U1202 pad 7: (no net) -> Net-(U1202-Pad7)
- U1202 pad 8: (no net) -> Net-(U1202-Pad8)
- U1204 pad 2: (no net) -> Net-(U1204-Pad2)
- U1204 pad 6: (no net) -> Net-(U1204-Pad6)
- U1205 pad 3: (no net) -> Net-(U1205-Pad3)
- U1208 pad 10: (no net) -> Net-(U1208-Pad10)
- U1208 pad 5: (no net) -> Net-(U1208-Pad5)
- U1208 pad 6: (no net) -> Net-(U1208-Pad6)
- U1208 pad 9: (no net) -> Net-(U1208-Pad9)
- U1209 pad 10: (no net) -> Net-(U1209-Pad10)
- U1209 pad 11: (no net) -> Net-(U1209-Pad11)
- U1209 pad 12: (no net) -> Net-(U1209-Pad12)
- U1209 pad 9: (no net) -> Net-(U1209-Pad9)
- U1212 pad 1: (no net) -> Net-(U1212-Pad1)
- U1212 pad 5: (no net) -> Net-(U1212-Pad5)
- U1212 pad 8: (no net) -> Net-(U1212-Pad8)
- U1213 pad 1: (no net) -> Net-(U1213-Pad1)
- U1213 pad 5: (no net) -> Net-(U1213-Pad5)
- U1213 pad 8: (no net) -> Net-(U1213-Pad8)
- U1302 pad 31: (no net) -> Net-(U1302-Pad31)
- U1302 pad 35: (no net) -> Net-(U1302-Pad35)
- U1303 pad 10: (no net) -> Net-(U1303-Pad10)
- U1303 pad 11: (no net) -> Net-(U1303-Pad11)
- U1303 pad 12: (no net) -> Net-(U1303-Pad12)
- U1303 pad 13: (no net) -> Net-(U1303-Pad13)
- U1303 pad 14: (no net) -> Net-(U1303-Pad14)
- U1303 pad 15: (no net) -> Net-(U1303-Pad15)
- U1303 pad 16: (no net) -> Net-(U1303-Pad16)
- U1303 pad 17: (no net) -> Net-(U1303-Pad17)
- U1303 pad 19: (no net) -> Net-(U1303-Pad19)
- U1303 pad 6: (no net) -> Net-(U1303-Pad6)
- U1303 pad 7: (no net) -> Net-(U1303-Pad7)
- U1303 pad 8: (no net) -> Net-(U1303-Pad8)
- U1303 pad 9: (no net) -> Net-(U1303-Pad9)
- U1403 pad 3: (no net) -> Net-(U1403-Pad3)
- U1404 pad 1: (no net) -> Net-(U1404-Pad1)
- U1404 pad 5: (no net) -> Net-(U1404-Pad5)
- U1404 pad 8: (no net) -> Net-(U1404-Pad8)
- U1405 pad 1: (no net) -> Net-(U1405-Pad1)
- U1405 pad 5: (no net) -> Net-(U1405-Pad5)
- U1405 pad 8: (no net) -> Net-(U1405-Pad8)
- U1501 pad 1: (no net) -> Net-(U1501-Pad1)
- U1501 pad 5: (no net) -> Net-(U1501-Pad5)
- U1501 pad 7: (no net) -> Net-(U1501-Pad7)
- U1501 pad 8: (no net) -> Net-(U1501-Pad8)
- U1602 pad 10: (no net) -> Net-(U1602-Pad10)
- U1602 pad 100: (no net) -> Net-(U1602-Pad100)
- U1602 pad 101: (no net) -> Net-(U1602-Pad101)
- U1602 pad 102: (no net) -> Net-(U1602-Pad102)
- U1602 pad 103: (no net) -> Net-(U1602-Pad103)
- U1602 pad 104: (no net) -> Net-(U1602-Pad104)
- U1602 pad 11: (no net) -> Net-(U1602-Pad11)
- U1602 pad 112: (no net) -> Net-(U1602-Pad112)
- U1602 pad 12: (no net) -> Net-(U1602-Pad12)
- U1602 pad 122: (no net) -> Net-(U1602-Pad122)
- U1602 pad 127: (no net) -> Net-(U1602-Pad127)
- U1602 pad 128: (no net) -> Net-(U1602-Pad128)
- U1602 pad 129: (no net) -> Net-(U1602-Pad129)
- U1602 pad 13: (no net) -> Net-(U1602-Pad13)
- U1602 pad 132: (no net) -> Net-(U1602-Pad132)
- U1602 pad 133: (no net) -> Net-(U1602-Pad133)
- U1602 pad 134: (no net) -> Net-(U1602-Pad134)
- U1602 pad 135: (no net) -> Net-(U1602-Pad135)
- U1602 pad 136: (no net) -> Net-(U1602-Pad136)
- U1602 pad 137: (no net) -> Net-(U1602-Pad137)
- U1602 pad 139: (no net) -> Net-(U1602-Pad139)
- U1602 pad 140: (no net) -> Net-(U1602-Pad140)
- U1602 pad 141: (no net) -> Net-(U1602-Pad141)
- U1602 pad 142: (no net) -> Net-(U1602-Pad142)
- U1602 pad 2: (no net) -> Net-(U1602-Pad2)
- U1602 pad 22: (no net) -> Net-(U1602-Pad22)
- U1602 pad 26: (no net) -> Net-(U1602-Pad26)
- U1602 pad 27: (no net) -> Net-(U1602-Pad27)
- U1602 pad 28: (no net) -> Net-(U1602-Pad28)
- U1602 pad 29: (no net) -> Net-(U1602-Pad29)
- U1602 pad 34: (no net) -> Net-(U1602-Pad34)
- U1602 pad 35: (no net) -> Net-(U1602-Pad35)
- U1602 pad 36: (no net) -> Net-(U1602-Pad36)
- U1602 pad 37: (no net) -> Net-(U1602-Pad37)
- U1602 pad 47: (no net) -> Net-(U1602-Pad47)
- U1602 pad 48: (no net) -> Net-(U1602-Pad48)
- U1602 pad 49: (no net) -> Net-(U1602-Pad49)
- U1602 pad 50: (no net) -> Net-(U1602-Pad50)
- U1602 pad 56: (no net) -> Net-(U1602-Pad56)
- U1602 pad 57: (no net) -> Net-(U1602-Pad57)
- U1602 pad 70: (no net) -> Net-(U1602-Pad70)
- U1602 pad 74: (no net) -> Net-(U1602-Pad74)
- U1602 pad 87: (no net) -> Net-(U1602-Pad87)
- U1602 pad 96: (no net) -> Net-(U1602-Pad96)
- U1602 pad 97: (no net) -> Net-(U1602-Pad97)
- U1602 pad 98: (no net) -> Net-(U1602-Pad98)
- U1602 pad 99: (no net) -> Net-(U1602-Pad99)
- U302 pad 1: (no net) -> Net-(U302-Pad1)
- U302 pad 10: (no net) -> Net-(U302-Pad10)
- U302 pad 100: (no net) -> Net-(U302-Pad100)
- U302 pad 101: (no net) -> Net-(U302-Pad101)
- U302 pad 102: (no net) -> Net-(U302-Pad102)
- U302 pad 103: (no net) -> Net-(U302-Pad103)
- U302 pad 11: (no net) -> Net-(U302-Pad11)
- U302 pad 111: (no net) -> Net-(U302-Pad111)
- U302 pad 112: (no net) -> Net-(U302-Pad112)
- U302 pad 113: (no net) -> Net-(U302-Pad113)
- U302 pad 114: (no net) -> Net-(U302-Pad114)
- U302 pad 115: (no net) -> Net-(U302-Pad115)
- U302 pad 116: (no net) -> Net-(U302-Pad116)
- U302 pad 117: (no net) -> Net-(U302-Pad117)
- U302 pad 118: (no net) -> Net-(U302-Pad118)
- U302 pad 119: (no net) -> Net-(U302-Pad119)
- U302 pad 12: (no net) -> Net-(U302-Pad12)
- U302 pad 122: (no net) -> Net-(U302-Pad122)
- U302 pad 123: (no net) -> Net-(U302-Pad123)
- U302 pad 124: (no net) -> Net-(U302-Pad124)
- U302 pad 125: (no net) -> Net-(U302-Pad125)
- U302 pad 127: (no net) -> Net-(U302-Pad127)
- U302 pad 13: (no net) -> Net-(U302-Pad13)
- U302 pad 132: (no net) -> Net-(U302-Pad132)
- U302 pad 134: (no net) -> Net-(U302-Pad134)
- U302 pad 135: (no net) -> Net-(U302-Pad135)
- U302 pad 136: (no net) -> Net-(U302-Pad136)
- U302 pad 137: (no net) -> Net-(U302-Pad137)
- U302 pad 139: (no net) -> Net-(U302-Pad139)
- U302 pad 14: (no net) -> Net-(U302-Pad14)
- U302 pad 140: (no net) -> Net-(U302-Pad140)
- U302 pad 141: (no net) -> Net-(U302-Pad141)
- U302 pad 142: (no net) -> Net-(U302-Pad142)
- U302 pad 15: (no net) -> Net-(U302-Pad15)
- U302 pad 2: (no net) -> Net-(U302-Pad2)
- U302 pad 29: (no net) -> Net-(U302-Pad29)
- U302 pad 3: (no net) -> Net-(U302-Pad3)
- U302 pad 34: (no net) -> Net-(U302-Pad34)
- U302 pad 37: (no net) -> Net-(U302-Pad37)
- U302 pad 4: (no net) -> Net-(U302-Pad4)
- U302 pad 40: (no net) -> Net-(U302-Pad40)
- U302 pad 41: (no net) -> Net-(U302-Pad41)
- U302 pad 42: (no net) -> Net-(U302-Pad42)
- U302 pad 46: (no net) -> Net-(U302-Pad46)
- U302 pad 47: (no net) -> Net-(U302-Pad47)
- U302 pad 48: (no net) -> Net-(U302-Pad48)
- U302 pad 49: (no net) -> Net-(U302-Pad49)
- U302 pad 5: (no net) -> Net-(U302-Pad5)
- U302 pad 50: (no net) -> Net-(U302-Pad50)
- U302 pad 56: (no net) -> Net-(U302-Pad56)
- U302 pad 57: (no net) -> Net-(U302-Pad57)
- U302 pad 58: (no net) -> Net-(U302-Pad58)
- U302 pad 59: (no net) -> Net-(U302-Pad59)
- U302 pad 60: (no net) -> Net-(U302-Pad60)
- U302 pad 63: (no net) -> Net-(U302-Pad63)
- U302 pad 64: (no net) -> Net-(U302-Pad64)
- U302 pad 65: (no net) -> Net-(U302-Pad65)
- U302 pad 66: (no net) -> Net-(U302-Pad66)
- U302 pad 67: (no net) -> Net-(U302-Pad67)
- U302 pad 68: (no net) -> Net-(U302-Pad68)
- U302 pad 69: (no net) -> Net-(U302-Pad69)
- U302 pad 7: (no net) -> Net-(U302-Pad7)
- U302 pad 70: (no net) -> Net-(U302-Pad70)
- U302 pad 73: (no net) -> Net-(U302-Pad73)
- U302 pad 77: (no net) -> Net-(U302-Pad77)
- U302 pad 78: (no net) -> Net-(U302-Pad78)
- U302 pad 79: (no net) -> Net-(U302-Pad79)
- U302 pad 8: (no net) -> Net-(U302-Pad8)
- U302 pad 80: (no net) -> Net-(U302-Pad80)
- U302 pad 81: (no net) -> Net-(U302-Pad81)
- U302 pad 82: (no net) -> Net-(U302-Pad82)
- U302 pad 85: (no net) -> Net-(U302-Pad85)
- U302 pad 86: (no net) -> Net-(U302-Pad86)
- U302 pad 87: (no net) -> Net-(U302-Pad87)
- U302 pad 88: (no net) -> Net-(U302-Pad88)
- U302 pad 89: (no net) -> Net-(U302-Pad89)
- U302 pad 9: (no net) -> Net-(U302-Pad9)
- U302 pad 90: (no net) -> Net-(U302-Pad90)
- U302 pad 91: (no net) -> Net-(U302-Pad91)
- U302 pad 92: (no net) -> Net-(U302-Pad92)
- U302 pad 93: (no net) -> Net-(U302-Pad93)
- U302 pad 96: (no net) -> Net-(U302-Pad96)
- U302 pad 97: (no net) -> Net-(U302-Pad97)
- U302 pad 98: (no net) -> Net-(U302-Pad98)
- U302 pad 99: (no net) -> Net-(U302-Pad99)
- U402 pad 2: (no net) -> Net-(U402-Pad2)
- U402 pad 3: (no net) -> Net-(U402-Pad3)
- U402 pad 6: (no net) -> Net-(U402-Pad6)
- U402 pad 7: (no net) -> Net-(U402-Pad7)
- U403 pad 2: (no net) -> Net-(U403-Pad2)
- U403 pad 3: (no net) -> Net-(U403-Pad3)
- U403 pad 6: (no net) -> Net-(U403-Pad6)
- U403 pad 7: (no net) -> Net-(U403-Pad7)
- U501 pad 5: (no net) -> Net-(U501-Pad5)
- U603 pad 4: (no net) -> Net-(U603-Pad4)
- U603 pad 6: (no net) -> Net-(U603-Pad6)
- U701 pad 1: (no net) -> Net-(U701-Pad1)
- U701 pad 3: (no net) -> Net-(U701-Pad3)
- U701 pad 7: (no net) -> Net-(U701-Pad7)
- U701 pad 8: (no net) -> Net-(U701-Pad8)
- U704 pad 1: (no net) -> Net-(U704-Pad1)
- U704 pad 20: (no net) -> Net-(U704-Pad20)
- U705 pad 1: (no net) -> Net-(U705-Pad1)
- U705 pad 5: (no net) -> Net-(U705-Pad5)
- U705 pad 8: (no net) -> Net-(U705-Pad8)
- U801 pad 11: (no net) -> Net-(U801-Pad11)
- U801 pad 6: (no net) -> Net-(U801-Pad6)
- U801 pad 7: (no net) -> Net-(U801-Pad7)
- U901 pad 14: (no net) -> Net-(U901-Pad14)
- U901 pad 15: (no net) -> Net-(U901-Pad15)
- U901 pad 24: (no net) -> Net-(U901-Pad24)
- U901 pad 26: (no net) -> Net-(U901-Pad26)
- U901 pad 31: (no net) -> Net-(U901-Pad31)
- U901 pad 32: (no net) -> Net-(U901-Pad32)
Routing:
- net +3V3: track 0.00 -> 77.0 mm, vias 0 -> 40
- net +24VDD: track 0.00 -> 69.0 mm, vias 0 -> 42
- net +15VF: track 0.00 -> 60.7 mm, vias 0 -> 26
- net -15VF: track 0.00 -> 51.4 mm, vias 0 -> 21
- net Net-(K1301-Pad3): track 0.00 -> 41.0 mm
- net Net-(K1303-Pad3): track 0.00 -> 32.4 mm
- net +5VF: track 0.00 -> 31.9 mm, vias 0 -> 13
- net Net-(C1313-Pad2): track 0.00 -> 30.4 mm, vias 0 -> 1
- net Net-(K1305-Pad3): track 0.00 -> 23.9 mm
- net Net-(C502-Pad1): track 0.00 -> 21.0 mm, vias 0 -> 18
- net VCCQ: track 0.00 -> 19.7 mm, vias 0 -> 6
- net +5V: track 0.00 -> 19.4 mm, vias 0 -> 16
- net +3.3VF: track 0.00 -> 18.3 mm, vias 0 -> 11
- net Net-(K1302-Pad3): track 0.00 -> 16.1 mm
- net +24V: track 0.00 -> 16.0 mm, vias 0 -> 14
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- added copper zone on B.Cu, net +24V
- added copper zone on F.Cu, net +24V
- added copper zone on Power, net +24V
- added copper zone on Power+GND, net +24V
- added copper zone on B.Cu, net +24VDD
- added copper zone on F.Cu, net +24VDD
- added copper zone on Power, net +24VDD
- added copper zone on Power+GND, net +24VDD
- added copper zone on B.Cu, net +3V3
- added copper zone on F.Cu, net +3V3
- added copper zone on Power, net +3V3
- added copper zone on B.Cu, net +5V
- added copper zone on F.Cu, net +5V
- added copper zone on Power, net +5V
- added copper zone on GND, net AGNDF
- added copper zone on B.Cu, net Earth
- added copper zone on F.Cu, net Earth
- added copper zone on GND, net Earth
- added copper zone on B.Cu, net GND
- added copper zone on F.Cu, net GND
- added copper zone on GND, net GND
- added copper zone on B.Cu, net GND_TRIG
- added copper zone on F.Cu, net GND_TRIG
- added copper zone on GND, net GND_TRIG
- added copper zone on B.Cu, net Net-(C414-Pad1)
- added copper zone on B.Cu, net Net-(C502-Pad1)
- added copper zone on F.Cu, net Net-(C502-Pad1)
- added copper zone on Power, net Net-(C502-Pad1)
- added copper zone on B.Cu, net Net-(D501-Pad1)
- added copper zone on F.Cu, net Net-(D501-Pad1)
- added copper zone on Power, net Net-(D501-Pad1)
- added copper zone on Power+GND, net VCCQ
Other:
- net class Default: clearance 0.2 -> 0.127; trace_width 0.25 -> 0.127; via_dia 0.8 -> 0.5; via_drill 0.4 -> 0.2
- net class Signals removed
- rule trace_clearance: 0.2 -> 0.127
