File: hardware/project/ETH1CPMU1/Connector.sch (KiCad schematic (older format))
At the start: 1 part, among them J201 C64AC

Commit message: Schematic design
Changed lines of the file:
@@
 $Descr A4 11693 8268
 encoding utf-8
-Sheet 2 12
+Sheet 2 14
 Title ""
 Date ""
@@
 Wire Wire Line
 	5200 1400 5200 1350
-Text Label 5000 1200 0    50   ~ 0
-A
-Text Label 5000 1400 0    50   ~ 0
-B
-Text Label 5000 1600 0    50   ~ 0
-C
-Text Label 5000 1800 0    50   ~ 0
-D
-Text Label 5000 2000 0    50   ~ 0
-E
-Text Label 5000 2200 0    50   ~ 0
-F
 Wire Wire Line
 	5250 5150 5200 5150
@@
 Wire Wire Line
 	5200 3950 5250 3950
+Text HLabel 5000 1200 0    50   BiDi ~ 0
+A
+Text HLabel 5000 1400 0    50   BiDi ~ 0
+B
+Text HLabel 5000 1600 0    50   BiDi ~ 0
+C
+Text HLabel 5000 1800 0    50   BiDi ~ 0
+D
+Text HLabel 5000 2000 0    50   BiDi ~ 0
+E
+Text HLabel 5000 2200 0    50   BiDi ~ 0
+F
 $EndSCHEMATC

Commit message: Schematic and PCB design.
Connections:
- net D: no longer names the net of J201.A5 (5A), J201.C5 (5C)
- no-connect marks 26 -> 34
Changed lines of the file:
@@
 	5250 1850 5200 1850
-Wire Wire Line
-	5200 1850 5200 1800
 Wire Wire Line
 	5200 1750 5250 1750
@@
 	5200 2000 5200 1950
 Wire Wire Line
-	5200 1800 5000 1800
-Wire Wire Line
 	5200 1600 5000 1600
 Connection ~ 5200 1600
 Wire Wire Line
 	5200 1600 5200 1550
-Connection ~ 5200 1800
-Wire Wire Line
-	5200 1800 5200 1750
 Wire Wire Line
 	5200 1400 5000 1400
@@
 Text HLabel 5000 1600 0    50   BiDi ~ 0
 C
-Text HLabel 5000 1800 0    50   BiDi ~ 0
-D
 Text HLabel 5000 2000 0    50   BiDi ~ 0
 E
 Text HLabel 5000 2200 0    50   BiDi ~ 0
 F
+NoConn ~ 5250 5350
+NoConn ~ 5250 5450
+NoConn ~ 5250 5550
+NoConn ~ 5250 5650
+NoConn ~ 5250 5750
+NoConn ~ 5250 5850
+NoConn ~ 5250 5950
+NoConn ~ 5250 6050
+Wire Wire Line
+	5200 1750 5200 1850
 $EndSCHEMATC

Commit message: PCB design.
Connections:
- net C: now also J201.A5 (5A), J201.C5 (5C)
Changed lines of the file:
@@
 	5200 2000 5200 1950
 Wire Wire Line
-	5200 1600 5000 1600
+	5200 1600 5100 1600
 Connection ~ 5200 1600
 Wire Wire Line
@@
 NoConn ~ 5250 6050
 Wire Wire Line
-	5200 1750 5200 1850
+	5200 1750 5200 1800
+Wire Wire Line
+	5200 1800 5100 1800
+Wire Wire Line
+	5100 1800 5100 1600
+Connection ~ 5200 1800
+Wire Wire Line
+	5200 1800 5200 1850
+Connection ~ 5100 1600
+Wire Wire Line
+	5100 1600 5000 1600
 $EndSCHEMATC

Commit message: PCB design
Connections:
- net C: no longer J201.A5 (5A), J201.C5 (5C)
- net J: now reaches J201.A10 (10A)
- net J: now also J201.C10 (10C)
- net K: now reaches J201.A11 (11A)
- net K: now also J201.C11 (11C)
- net L: now reaches J201.A12 (12A)
- net L: now also J201.C12 (12C)
- net M: now reaches J201.A13 (13A)
- net M: now also J201.C13 (13C)
- net G: now reaches J201.A8 (8A)
- net G: now also J201.C8 (8C)
- net I: now reaches J201.A9 (9A)
- net I: now also J201.C9 (9C)
- new net D: J201.A5 (5A), J201.C5 (5C)
- no-connect marks 34 -> 22
Changed lines of the file:
@@
 Wire Wire Line
 	5200 2000 5200 1950
-Wire Wire Line
-	5200 1600 5100 1600
 Connection ~ 5200 1600
 Wire Wire Line
@@
 NoConn ~ 5250 4550
 NoConn ~ 5250 4650
-NoConn ~ 5250 2350
-NoConn ~ 5250 2450
-NoConn ~ 5250 2550
-NoConn ~ 5250 2650
-NoConn ~ 5250 2750
-NoConn ~ 5250 2850
-NoConn ~ 5250 2950
-NoConn ~ 5250 3050
-NoConn ~ 5250 3150
-NoConn ~ 5250 3250
-NoConn ~ 5250 3350
-NoConn ~ 5250 3450
 NoConn ~ 5250 3550
 NoConn ~ 5250 3650
@@
 NoConn ~ 5250 6050
 Wire Wire Line
+	5000 1600 5200 1600
+Wire Wire Line
 	5200 1750 5200 1800
 Wire Wire Line
-	5200 1800 5100 1800
-Wire Wire Line
-	5100 1800 5100 1600
+	5200 1800 5000 1800
 Connection ~ 5200 1800
 Wire Wire Line
 	5200 1800 5200 1850
-Connection ~ 5100 1600
-Wire Wire Line
-	5100 1600 5000 1600
+Text Label 5000 1800 0    50   ~ 0
+D
+Wire Wire Line
+	5250 2450 5200 2450
+Wire Wire Line
+	5200 2450 5200 2400
+Wire Wire Line
+	5200 2350 5250 2350
+Wire Wire Line
+	5200 2400 5000 2400
+Connection ~ 5200 2400
+Wire Wire Line
+	5200 2400 5200 2350
+Text Label 5000 2400 0    50   ~ 0
+G
+Wire Wire Line
+	5250 2650 5200 2650
+Wire Wire Line
+	5200 2650 5200 2600
+Wire Wire Line
+	5200 2550 5250 2550
+Wire Wire Line
+	5200 2600 5000 2600
+Connection ~ 5200 2600
+Wire Wire Line
+	5200 2600 5200 2550
+Text Label 5000 2600 0    50   ~ 0
+I
+Wire Wire Line
+	5250 3450 5200 3450
+Wire Wire Line
+	5200 3450 5200 3400
+Wire Wire Line
+	5200 3350 5250 3350
+Wire Wire Line
+	5250 3250 5200 3250
+Wire Wire Line
+	5200 3250 5200 3200
+Wire Wire Line
+	5200 3150 5250 3150
+Wire Wire Line
+	5250 3050 5200 3050
+Wire Wire Line
+	5200 3050 5200 3000
+Wire Wire Line
+	5200 2950 5250 2950
+Wire Wire Line
+	5250 2850 5200 2850
+Wire Wire Line
+	5200 2850 5200 2800
+Wire Wire Line
+	5200 2750 5250 2750
+Wire Wire Line
+	5200 2800 5000 2800
+Connection ~ 5200 2800
+Wire Wire Line
+	5200 2800 5200 2750
+Wire Wire Line
+	5200 3000 5000 3000
+Connection ~ 5200 3000
+Wire Wire Line
+	5200 3000 5200 2950
+Wire Wire Line
+	5200 3200 5000 3200
+Connection ~ 5200 3200
+Wire Wire Line
+	5200 3200 5200 3150
+Wire Wire Line
+	5200 3400 5000 3400
+Connection ~ 5200 3400
+Wire Wire Line
+	5200 3400 5200 3350
+Text Label 5000 2800 0    50   ~ 0
+J
+Text Label 5000 3000 0    50   ~ 0
+K
+Text Label 5000 3200 0    50   ~ 0
+L
+Text Label 5000 3400 0    50   ~ 0
+M
 $EndSCHEMATC
