File: hardware/project/ETH1CPMU1/PMU.sch (KiCad schematic (older format))
At the start: 62 parts, among them K1401 HE3621A0510, K1402 HE3621A0510, K1403 HE3621A0510, K1404 HE3621A0510, K1405 HE3621A0510, K1406 HE3621A0510, K1407 HE3621A0510, K1408 HE3621A0510, Q1401 BC847, Q1402 BC847, Q1403 BC847, Q1404 BC847, Q1405 BC847, Q1406 BC847, Q1407 BC847, Q1408 BC847, U1401 THS6012, U1402 DG419LEUA, U1403 AD5520

Commit message: PCB design
Parts:
- renumbered C1414 to C1301, C1415 to C1302, C1416 to C1303, C1417 to C1304, C1418 to C1305, C1409 to C1306, C1410 to C1307, C1411 to C1308, C1419 to C1309, C1420 to C1310, C1421 to C1311, C1422 to C1312, C1404 to C1313, C1401 to C1314, C1423 to C1315, C1424 to C1316, C1425 to C1317, C1426 to C1318, C1403 to C1319, C1405 to C1320, C1407 to C1321, C1412 to C1322, C1402 to C1323, C1406 to C1324, C1408 to C1325, C1413 to C1326, K1403 to K1301, K1404 to K1302, K1405 to K1303, K1406 to K1304, K1407 to K1305, K1408 to K1306, K1401 to K1307, K1402 to K1308, Q1402 to Q1301, Q1403 to Q1302, Q1405 to Q1303, Q1407 to Q1304, Q1401 to Q1305, Q1404 to Q1306, Q1406 to Q1307, Q1408 to Q1308, R1402 to R1301, R1407 to R1302, R1401 to R1303, R1408 to R1304, R1409 to R1305, R1410 to R1306, R1411 to R1307, R1412 to R1308, R1413 to R1309, R1404 to R1310, R1405 to R1311, R1414 to R1312, R1416 to R1313, R1403 to R1314, R1406 to R1315, R1415 to R1316, R1417 to R1317, U1402 to U1301, U1403 to U1302, U1401 to U1303

Commit message: PCB design
Connections:
- net +3.3VF renamed +3.3VP
Changed lines of the file:
@@
-	1    0    0    -1
-$EndComp
-$Comp
-L ETH1CPMU1:+3.3VF #PWR01310
-U 1 1 5E174F9C
-P 3800 2050
-F 0 "#PWR01310" H 3800 1900 50  0001 C CNN
-F 1 "+3.3VF" H 3815 2223 50  0000 C CNN
-F 2 "" H 3800 2050 50  0001 C CNN
-F 3 "" H 3800 2050 50  0001 C CNN
-	1    3800 2050
 	1    0    0    -1
 $EndComp
@@
 Wire Wire Line
 	3150 9950 2900 9950
-$Comp
-L ETH1CPMU1:+3.3VF #PWR01306
-U 1 1 5E18B6A7
-P 3150 9900
-F 0 "#PWR01306" H 3150 9750 50  0001 C CNN
-F 1 "+3.3VF" H 3165 10073 50  0000 C CNN
-F 2 "" H 3150 9900 50  0001 C CNN
-F 3 "" H 3150 9900 50  0001 C CNN
-	1    3150 9900
-	1    0    0    -1
-$EndComp
 $Comp
 L ETH1CPMU1:AGNDF #PWR01308
@@
 Text HLabel 1800 3450 0    50   Input ~ 0
 AC_FOURCE
-$Comp
-L ETH1CPMU1:+3.3VF #PWR01321
-U 1 1 5E2C33FA
-P 5700 9500
-F 0 "#PWR01321" H 5700 9350 50  0001 C CNN
-F 1 "+3.3VF" H 5715 9673 50  0000 C CNN
-F 2 "" H 5700 9500 50  0001 C CNN
-F 3 "" H 5700 9500 50  0001 C CNN
-	1    5700 9500
-	1    0    0    -1
-$EndComp
 Wire Wire Line
 	5700 9500 5700 9550
@@
 F 3 "~" H 3950 10150 50  0001 C CNN
 	1    3950 10150
-	1    0    0    -1
-$EndComp
-$Comp
-L ETH1CPMU1:+3.3VF #PWR01311
-U 1 1 5E333BDD
-P 3950 9900
-F 0 "#PWR01311" H 3950 9750 50  0001 C CNN
-F 1 "+3.3VF" H 3965 10073 50  0000 C CNN
-F 2 "" H 3950 9900 50  0001 C CNN
-F 3 "" H 3950 9900 50  0001 C CNN
-	1    3950 9900
 	1    0    0    -1
 $EndComp
@@
 Wire Wire Line
 	3250 2650 3300 2650
+$Comp
+L power:+3.3VP #PWR0101
+U 1 1 5E074E3D
+P 3800 2050
+F 0 "#PWR0101" H 3950 2000 50  0001 C CNN
+F 1 "+3.3VP" H 3820 2193 50  0000 C CNN
+F 2 "" H 3800 2050 50  0001 C CNN
+F 3 "" H 3800 2050 50  0001 C CNN
+	1    3800 2050
+	1    0    0    -1
+$EndComp
+$Comp
+L power:+3.3VP #PWR0102
+U 1 1 5E075067
+P 3150 9900
+F 0 "#PWR0102" H 3300 9850 50  0001 C CNN
+F 1 "+3.3VP" H 3170 10043 50  0000 C CNN
+F 2 "" H 3150 9900 50  0001 C CNN
+F 3 "" H 3150 9900 50  0001 C CNN
+	1    3150 9900
+	1    0    0    -1
+$EndComp
+$Comp
+L power:+3.3VP #PWR0103
+U 1 1 5E079009
+P 3950 9900
+F 0 "#PWR0103" H 4100 9850 50  0001 C CNN
+F 1 "+3.3VP" H 3970 10043 50  0000 C CNN
+F 2 "" H 3950 9900 50  0001 C CNN
+F 3 "" H 3950 9900 50  0001 C CNN
+	1    3950 9900
+	1    0    0    -1
+$EndComp
+$Comp
+L power:+3.3VP #PWR0104
+U 1 1 5E079EB9
+P 5700 9500
+F 0 "#PWR0104" H 5850 9450 50  0001 C CNN
+F 1 "+3.3VP" H 5720 9643 50  0000 C CNN
+F 2 "" H 5700 9500 50  0001 C CNN
+F 3 "" H 5700 9500 50  0001 C CNN
+	1    5700 9500
+	1    0    0    -1
+$EndComp
 $EndSCHEMATC
