File: hardware/project/ETH1CPMU1/ADC.sch (KiCad schematic (older format))
At the start: 29 parts, among them U901 ADS8363, U902 INA159, U903 INA159, U904 INA159, U905 ADG1414BRU

Commit message: PCB design
Connections:
- net +3.3VF renamed +3.3VP
Changed lines of the file:
@@
 Wire Wire Line
 	2050 7350 2300 7350
-$Comp
-L ETH1CPMU1:+3.3VF #PWR0907
-U 1 1 5E654E98
-P 2050 6900
-F 0 "#PWR0907" H 2050 6750 50  0001 C CNN
-F 1 "+3.3VF" H 2065 7073 50  0000 C CNN
-F 2 "" H 2050 6900 50  0001 C CNN
-F 3 "" H 2050 6900 50  0001 C CNN
-	1    2050 6900
-	1    0    0    -1
-$EndComp
 Wire Wire Line
 	2050 6900 2050 6950
@@
 Wire Wire Line
 	1050 7350 1300 7350
-$Comp
-L ETH1CPMU1:+3.3VF #PWR0903
-U 1 1 5E68C8C2
-P 1050 6900
-F 0 "#PWR0903" H 1050 6750 50  0001 C CNN
-F 1 "+3.3VF" H 1065 7073 50  0000 C CNN
-F 2 "" H 1050 6900 50  0001 C CNN
-F 3 "" H 1050 6900 50  0001 C CNN
-	1    1050 6900
-	1    0    0    -1
-$EndComp
 Wire Wire Line
 	1050 6900 1050 6950
@@
 Wire Wire Line
 	9300 1150 9300 1200
-$Comp
-L ETH1CPMU1:+3.3VF #PWR0935
-U 1 1 5E1C16F5
-P 9300 1150
-F 0 "#PWR0935" H 9300 1000 50  0001 C CNN
-F 1 "+3.3VF" H 9315 1323 50  0000 C CNN
-F 2 "" H 9300 1150 50  0001 C CNN
-F 3 "" H 9300 1150 50  0001 C CNN
-	1    9300 1150
-	1    0    0    -1
-$EndComp
 Wire Wire Line
 	9550 3100 9550 3050
@@
 Wire Wire Line
 	2300 3650 2350 3650
-$Comp
-L ETH1CPMU1:+3.3VF #PWR0910
-U 1 1 5DE1F585
-P 2300 3650
-F 0 "#PWR0910" H 2300 3500 50  0001 C CNN
-F 1 "+3.3VF" V 2300 3900 50  0000 C CNN
-F 2 "" H 2300 3650 50  0001 C CNN
-F 3 "" H 2300 3650 50  0001 C CNN
-	1    2300 3650
-	0    -1   -1   0
-$EndComp
 Wire Wire Line
 	2300 3550 2350 3550
@@
 F 3 "" H 3350 2450 50  0001 C CNN
 	1    3350 2450
-	1    0    0    -1
-$EndComp
-$Comp
-L ETH1CPMU1:+3.3VF #PWR0912
-U 1 1 5DD3B37F
-P 3050 2450
-F 0 "#PWR0912" H 3050 2300 50  0001 C CNN
-F 1 "+3.3VF" H 3065 2623 50  0000 C CNN
-F 2 "" H 3050 2450 50  0001 C CNN
-F 3 "" H 3050 2450 50  0001 C CNN
-	1    3050 2450
 	1    0    0    -1
 $EndComp
@@
 Text HLabel 7950 1000 2    50   Input ~ 0
 PMU_MEASV_GAIN
+$Comp
+L power:+3.3VP #PWR0108
+U 1 1 5E0B81B2
+P 9300 1150
+F 0 "#PWR0108" H 9450 1100 50  0001 C CNN
+F 1 "+3.3VP" H 9320 1293 50  0000 C CNN
+F 2 "" H 9300 1150 50  0001 C CNN
+F 3 "" H 9300 1150 50  0001 C CNN
+	1    9300 1150
+	1    0    0    -1
+$EndComp
+$Comp
+L power:+3.3VP #PWR0109
+U 1 1 5E0B84ED
+P 3050 2450
+F 0 "#PWR0109" H 3200 2400 50  0001 C CNN
+F 1 "+3.3VP" H 3070 2593 50  0000 C CNN
+F 2 "" H 3050 2450 50  0001 C CNN
+F 3 "" H 3050 2450 50  0001 C CNN
+	1    3050 2450
+	1    0    0    -1
+$EndComp
+$Comp
+L power:+3.3VP #PWR0110
+U 1 1 5E0B9BE8
+P 2050 6900
+F 0 "#PWR0110" H 2200 6850 50  0001 C CNN
+F 1 "+3.3VP" H 2070 7043 50  0000 C CNN
+F 2 "" H 2050 6900 50  0001 C CNN
+F 3 "" H 2050 6900 50  0001 C CNN
+	1    2050 6900
+	1    0    0    -1
+$EndComp
+$Comp
+L power:+3.3VP #PWR0111
+U 1 1 5E0BB973
+P 1050 6900
+F 0 "#PWR0111" H 1200 6850 50  0001 C CNN
+F 1 "+3.3VP" H 1070 7043 50  0000 C CNN
+F 2 "" H 1050 6900 50  0001 C CNN
+F 3 "" H 1050 6900 50  0001 C CNN
+	1    1050 6900
+	1    0    0    -1
+$EndComp
+$Comp
+L power:+3.3VP #PWR?
+U 1 1 5E13DA46
+P 2300 3650
+F 0 "#PWR?" H 2450 3600 50  0001 C CNN
+F 1 "+3.3VP" V 2300 3750 50  0000 L CNN
+F 2 "" H 2300 3650 50  0001 C CNN
+F 3 "" H 2300 3650 50  0001 C CNN
+	1    2300 3650
+	0    -1   -1   0
+$EndComp
 $EndSCHEMATC
