File: hardware/project/ETH1CPMU1/MCU_Main.sch (KiCad schematic (older format))
At the start: 31 parts, among them J301 Conn_02x05, J302 Conn_02x01, U301 STM32F765ZGT6, U302 24LC08B-E/MS, Y301 NX3225GD-8MHZ-STD-CRA-3

Commit message: PCB design.
Parts:
- added C320: 100n, Capacitor_SMD:C_0603_1608Metric_Pad1.05x0.95mm_HandSolder, symbol Device:C
- renumbered C320 to C321
Connections:
- net +3V3: now also C320.1
- net GND: now also C320.2
- net MCU_DEFAULT: now also U301.104 (PA12,TIM1_ETR,SPI2_SCK,I2S2_CK,UART4_TX,USART1_RTS,SAI2_FS_B,CAN1_TX,OTG_FS_DP,LCD_R5,EVENTOUT)
- no-connect marks 88 -> 87
Other:
- moved on the sheet: C321, FB301, J301, J302, R305

Commit message: PCB design
Parts:
- renumbered C307 to C301, C308 to C302, C309 to C303, C301 to C304, C310 to C305, C302 to C306, C303 to C307, C311 to C308, C304 to C309, C312 to C310, C306 to C311, C313 to C312, C314 to C313, C315 to C314, C316 to C315, C317 to C316, C318 to C317, C319 to C318, C320 to C319, C321 to C320, C305 to C321, J302 to J301, J301 to J302, R305 to R303, R303 to R305, U302 to U301, U301 to U302

Commit message: PCB designed
Connections:
- net MCU1_GPIO_OUT1: now also U302.60 (PE9,TIM1_CH1,DFSDM1_CKOUT,UART7_RTS,QUADSPI_BK2_IO2,FMC_D6,EVENTOUT); no longer U302.22 (PF10,QUADSPI_CLK,DCMI_D11,LCD_DE,EVENTOUT,ADC3_IN8)
- net MCU1_GPIO_OUT2: now also U302.59 (PE8,TIM1_CH1N,DFSDM1_CKIN2,UART7_TX,QUADSPI_BK2_IO1,FMC_D5,EVENTOUT); no longer U302.26 (PC0,DFSDM1_CKIN0,DFSDM1_DATIN4,SAI2_FS_B,OTG_HS_ULPI_STP,FMC_SDNWE,LCD_R5,EVENTOUT,ADC1_IN10,ADC2_IN10,ADC3_IN10)
- net MCU1_MCLK: now also U302.65 (PE12,TIM1_CH3N,SPI4_SCK,DFSDM1_DATIN5,SAI2_SCK_B,FMC_D9,LCD_B4,EVENTOUT); no longer U302.19 (PF7,TIM11_CH1,SPI5_SCK,SAI1_MCLK_B,UART7_TX,QUADSPI_BK1_IO2,EVENTOUT,ADC3_IN5)
- net MCU1_MISO: now also U302.66 (PE13,TIM1_CH3,SPI4_MISO,DFSDM1_CKIN5,SAI2_FS_B,FMC_D10,LCD_DE,EVENTOUT); no longer U302.20 (PF8,SPI5_MISO,SAI1_SCK_B,UART7_RTS,TIM13_CH1,QUADSPI_BK1_IO0,EVENTOUT,ADC3_IN6)
- net MCU1_MOSI: now also U302.67 (PE14,TIM1_CH4,SPI4_MOSI,SAI2_MCLK_B,FMC_D11,LCD_CLK,EVENTOUT); no longer U302.21 (PF9,SPI5_MOSI,SAI1_FS_B,UART7_CTS,TIM14_CH1,QUADSPI_BK1_IO1,EVENTOUT,ADC3_IN7)
- net MCU1_STATUS_IN: now also U302.63 (PE10,TIM1_CH2N,DFSDM1_DATIN4,UART7_CTS,QUADSPI_BK2_IO3,FMC_D7,EVENTOUT); no longer U302.28 (PC2,DFSDM1_CKIN1,SPI2_MISO,DFSDM1_CKOUT,OTG_HS_ULPI_DIR,ETH_MII_TXD2,FMC_SDNE0,EVENTOUT,ADC1_IN12,ADC2_IN12,ADC3_IN12)
- net MCU1_~MSS: now also U302.64 (PE11,TIM1_CH2,SPI4_NSS,DFSDM1_CKIN4,SAI2_SD_B,FMC_D8,LCD_G3,EVENTOUT); no longer U302.18 (PF6,TIM10_CH1,SPI5_NSS,SAI1_SD_B,UART7_RX,QUADSPI_BK1_IO3,EVENTOUT,ADC3_IN4)
- net MCU_DEFAULT: now also U302.47 (PB1,TIM1_CH3N,TIM3_CH4,TIM8_CH3N,DFSDM1_DATIN1,LCD_R6,OTG_HS_ULPI_D2,ETH_MII_RXD3,LCD_G0,EVENTOUT,ADC1_IN9,ADC2_IN9); no longer U302.104 (PA12,TIM1_ETR,SPI2_SCK,I2S2_CK,UART4_TX,USART1_RTS,SAI2_FS_B,CAN1_TX,OTG_FS_DP,LCD_R5,EVENTOUT)
- net TRIG_EN: now also U302.12 (PF2,I2C2_SMBA,FMC_A2,EVENTOUT); no longer U302.74 (PB13,TIM1_CH1N,SPI2_SCK,I2S2_CK,DFSDM1_CKIN1,USART3_CTS,UART5_TX,CAN2_TX,OTG_HS_ULPI_D6,ETH_MII_TXD1,ETH_RMII_TXD1,EVENTOUT,OTG_HS_VBUS)
- net TRIG_IN: now also U302.10 (PF0,I2C2_SDA,FMC_A0,EVENTOUT); no longer U302.76 (PB15,RTC_REFIN,TIM1_CH3N,TIM8_CH3N,USART1_RX,SPI2_MOSI,I2S2_SD,DFSDM1_CKIN2,UART4_CTS,TIM12_CH2,SDMMC2_D1,OTG_HS_DP,EVENTOUT)
- net TRIG_OUT: now also U302.11 (PF1,I2C2_SCL,FMC_A1,EVENTOUT); no longer U302.75 (PB14,TIM1_CH2N,TIM8_CH2N,USART1_TX,SPI2_MISO,DFSDM1_DATIN2,USART3_RTS,UART4_RTS,TIM12_CH1,SDMMC2_D0,OTG_HS_DM,EVENTOUT)
Changed lines of the file:
@@
 Text Notes 10200 11150 0    50   ~ 0
 PROGRAMMING CONNECTOR\nDESIGNED FOR JLINK
-$Comp
-L ETH1CPMU1:STM32F765ZGT6 U302
-U 1 1 5DC8ECD0
-P 8900 4900
-F 0 "U302" H 3450 8800 50  0000 C CNN
-F 1 "STM32F765ZGT6" H 14050 8800 50  0000 C CNN
-F 2 "ETH1CPMU1:TQFP-144_20x20mm_P0.5mm" H 24800 6400 50  0001 C CNN
-F 3 "" H 24800 6400 50  0001 C CNN
-	1    8900 4900
-	1    0    0    -1
-$EndComp
 Wire Wire Line
 	14600 2250 14650 2250
@@
 Wire Wire Line
 	700  9650 700  9550
-Text HLabel 14650 7550 2    50   Output ~ 0
+Text HLabel 3150 1650 0    50   Output ~ 0
 TRIG_EN
-Text HLabel 14650 7650 2    50   Output ~ 0
+Text HLabel 3150 1550 0    50   Output ~ 0
 TRIG_OUT
-Text HLabel 14650 7750 2    50   Input ~ 0
+Text HLabel 3150 1450 0    50   Input ~ 0
 TRIG_IN
 Wire Wire Line
 	14600 8250 15250 8250
 Wire Wire Line
-	14650 7550 14600 7550
-Wire Wire Line
-	14650 7650 14600 7650
-Wire Wire Line
-	14600 7750 14650 7750
-Text HLabel 3150 5050 0    50   Input ~ 0
+	3150 1650 3200 1650
+Wire Wire Line
+	3150 1550 3200 1550
+Wire Wire Line
+	3200 1450 3150 1450
+Text HLabel 14650 5550 2    50   Input ~ 0
 MCU1_STATUS_IN
-Text HLabel 3150 4850 0    50   Output ~ 0
+Text HLabel 14650 5350 2    50   Output ~ 0
 MCU1_GPIO_OUT2
-Text HLabel 3150 2450 0    50   Output ~ 0
+Text HLabel 14650 5450 2    50   Output ~ 0
 MCU1_GPIO_OUT1
 Wire Wire Line
-	3150 2450 3200 2450
-Wire Wire Line
-	3200 4850 3150 4850
-Wire Wire Line
-	3150 5050 3200 5050
-Wire Wire Line
-	3200 2050 3150 2050
-Wire Wire Line
-	3150 2150 3200 2150
-Wire Wire Line
-	3200 2250 3150 2250
-Wire Wire Line
-	3150 2350 3200 2350
-Text HLabel 3150 2050 0    50   Output ~ 0
+	14650 5450 14600 5450
+Wire Wire Line
+	14600 5350 14650 5350
+Wire Wire Line
+	14650 5550 14600 5550
+Wire Wire Line
+	14600 5650 14650 5650
+Wire Wire Line
+	14600 5850 14650 5850
+Wire Wire Line
+	14650 5950 14600 5950
+Text HLabel 14650 5650 2    50   Output ~ 0
 MCU1_~MSS
-Text HLabel 3150 2250 0    50   Input ~ 0
+Text HLabel 14650 5850 2    50   Input ~ 0
 MCU1_MISO
-Text HLabel 3150 2350 0    50   Output ~ 0
+Text HLabel 14650 5950 2    50   Output ~ 0
 MCU1_MOSI
-Text HLabel 3150 2150 0    50   Output ~ 0
-MCU1_MCLK
 NoConn ~ 3200 5850
 NoConn ~ 3200 5950
@@
 NoConn ~ 3200 2650
 NoConn ~ 3200 3150
-NoConn ~ 3200 1450
-NoConn ~ 3200 1550
-NoConn ~ 3200 1650
 NoConn ~ 3200 3450
 NoConn ~ 3200 3550
@@
 NoConn ~ 14600 5150
 NoConn ~ 14600 5250
-NoConn ~ 14600 5350
-NoConn ~ 14600 5450
-NoConn ~ 14600 5550
-NoConn ~ 14600 5650
-NoConn ~ 14600 5750
-NoConn ~ 14600 5850
-NoConn ~ 14600 5950
 NoConn ~ 14600 6050
 NoConn ~ 14600 6250
-NoConn ~ 14600 6350
 NoConn ~ 14600 6450
 NoConn ~ 14600 6650
@@
 	3700 10900 4200 10900
 Wire Wire Line
-	3200 4350 2650 4350
-Text Label 2650 4350 0    50   ~ 0
+	14600 6350 15150 6350
+Text Label 15150 6350 2    50   ~ 0
 MCU_DEFAULT
+Text HLabel 14650 5750 2    50   Output ~ 0
+MCU1_MCLK
+Wire Wire Line
+	14650 5750 14600 5750
+$Comp
+L ETH1CPMU1:STM32F765ZGT6 U302
+U 1 1 5DC8ECD0
+P 8900 4900
+F 0 "U302" H 3450 8800 50  0000 C CNN
+F 1 "STM32F765ZGT6" H 14050 8800 50  0000 C CNN
+F 2 "ETH1CPMU1:TQFP-144_20x20mm_P0.5mm" H 24800 6400 50  0001 C CNN
+F 3 "" H 24800 6400 50  0001 C CNN
+	1    8900 4900
+	1    0    0    -1
+$EndComp
+NoConn ~ 3200 2450
+NoConn ~ 3200 2350
+NoConn ~ 3200 2250
+NoConn ~ 3200 2150
+NoConn ~ 3200 2050
+NoConn ~ 3200 4850
+NoConn ~ 3200 5050
+NoConn ~ 14600 7550
+NoConn ~ 14600 7650
+NoConn ~ 14600 7750
+NoConn ~ 3200 4350
 $EndSCHEMATC
